File: hardware/schematic/v1.0/_restore_backup_2026-07-31T10-43-38-896/GPSDO.kicad_sch (KiCad schematic)
At the start: 59 parts, among them J1 USB_C_Receptacle_USB2.0_16P, Q1 NMOS, SW1 SW_Push, U1 STM32G431KBUx, U2 OCXO-10M, U3 SKG123N, U4 IPEX1, U5 BQ25890, U6 TPS7A8901, U7 CH340E, Y1 Crystal_GND24

Commit message: Update KiCad schematic files and history
Parts:
- removed C21: 0.1uF, Capacitor_SMD:C_0603_1608Metric, symbol Device:C
- removed R19: 10K, Resistor_SMD:R_0603_1608Metric, symbol Device:R
- removed SW1: SW_Push, Capacitor_SMD:C_0201_0603Metric, symbol Switch:SW_Push
- U2: footprint Counter:OCXO_19x19mm -> (none)
Connections:
- net RESET: no longer names the net of U1.4 (PG10)
Other:
- note removed: "Optional RESET"
- moved on the sheet: C10, C11, C6, C7, C8, C9, JP1, R10, R11, R8, R9, U6
