File: hardware/schematic/v1.0/GPSDO_Rev1.0/MCU.kicad_sch (KiCad schematic)
At the start: 0 parts

Commit message: sch update
Parts:
- added U1: TDC7200PWR, GPSDO_Rev1.0:TDC7200PWR, symbol GPSDO_Rev1.0:TDC7200PWR
Changed lines of the file:
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@@
 	(generator_version "10.0")
 	(paper "A4")
+	(symbol
+		(lib_id "GPSDO_Rev1.0:TDC7200PWR")
+		(at 210.82 124.46 0)
+		(unit 1)
+		(body_style 1)
+		(exclude_from_sim no)
+		(in_bom yes)
+		(on_board yes)
+		(in_pos_files yes)
+		(dnp no)
+		(fields_autoplaced yes)
+		(property "Reference" "U1"
+			(at 210.82 109.22 0)
+			(show_name no)
+			(do_not_autoplace no)
+			(effects
+				(font
+					(size 1.27 1.27)
+				)
+			)
+		)
+		(property "Value" "TDC7200PWR"
+			(at 210.82 111.76 0)
+			(show_name no)
+			(do_not_autoplace no)
+			(effects
+				(font
+					(size 1.27 1.27)
+				)
+			)
+		)
+		(property "Footprint" "GPSDO_Rev1.0:TDC7200PWR"
+			(at 210.82 124.46 0)
+			(hide yes)
+			(show_name no)
+			(do_not_autoplace no)
+			(effects
+				(font
+					(size 1.27 1.27)
+				)
+			)
+		)
+		(property "Datasheet" "https://www.lcsc.com/datasheet/lcsc_datasheet_2303011701_Texas-Instruments-TDC7200PWR_C2653139.pdf"
+			(at 210.82 124.46 0)
+			(hide yes)
+			(show_name no)
+			(do_not_autoplace no)
+			(effects
+				(font
+					(size 1.27 1.27)
+				)
+			)
+		)
+		(property "Description" "-40℃~+85℃ 0.5uA 20MHz 2V~3.6V SPI TSSOP-14 ADCs/DACs - Special Purpose ROHS"
+			(at 210.82 124.46 0)
+			(hide yes)
+			(show_name no)
+			(do_not_autoplace no)
+			(effects
+				(font
+					(size 1.27 1.27)
+				)
+			)
+		)
+		(property "LCSC" "C2653139"
+			(at 210.82 124.46 0)
+			(hide yes)
+			(show_name no)
+			(do_not_autoplace no)
+			(effects
+				(font
+					(size 1.27 1.27)
+				)
+			)
+		)
+		(property "Manufacturer" "Texas Instruments"
+			(at 210.82 124.46 0)
+			(hide yes)
+			(show_name no)
+			(do_not_autoplace no)
+			(effects
+				(font
+					(size 1.27 1.27)
+				)
+			)
+		)
+		(property "Manufacturer Part" "TDC7200PWR"
+			(at 210.82 124.46 0)
+			(hide yes)
+			(show_name no)
+			(do_not_autoplace no)
+			(effects
+				(font
+					(size 1.27 1.27)
+				)
+			)
+		)
+		(pin "5"
+		)
+		(pin "6"
+		)
+		(pin "10"
+		)
+		(pin "13"
+		)
+		(pin "9"
+		)
+		(pin "1"
+		)
+		(pin "2"
+		)
+		(pin "3"
+		)
+		(pin "4"
+		)
+		(pin "7"
+		)
+		(pin "8"
+		)
+		(pin "11"
+		)
+		(pin "12"
+		)
+		(pin "14"
+		)
+		(instances
+			(project "GPSDO_Rev1.0"
+				(path "/7fcb1340-2836-48b1-8b47-374fa7e6ca96/a223c499-b8b9-41df-ac1a-b6212c61923a"
+					(reference "U1")
+					(unit 1)
+				)
+			)
+		)
+	)
 )

Commit message: sch update
Parts:
- added C10, C9: 1uF, GPSDO_Rev1.0:C_0603_1608Metric, symbol GPSDO_Rev1.0:C
- added C12: 100nF, GPSDO_Rev1.0:C_0402_1005Metric, symbol GPSDO_Rev1.0:C
- added JP1: SolderJumper_2_Bridged, Jumper:SolderJumper-2_P1.3mm_Bridged_RoundedPad1.0x1.5mm, symbol Jumper:SolderJumper_2_Bridged
- added R10: 100K, GPSDO_Rev1.0:R_0402_1005Metric, symbol GPSDO_Rev1.0:R
- added U9: STM32G431KBUx, GPSDO_Rev1.0:QFN-32-1EP_5x5mm_P0.5mm_EP3.45x3.45mm, symbol GPSDO_Rev1.0:STM32G431KBUx
Connections:
- net TDC_ENABLE: now reaches U1.1 (ENABLE)
- net MCU_SPI2_MOSI: now reaches U1.10 (DIN)
- net MCU_SPI2_NSS: now reaches U1.11 (CSB)
- net MCU_SPI2_SCK: now reaches U1.12 (SCLK)
- net at U1.13 (VREG): now also C9.1
- net +3.3V: now reaches U1.14 (VDD)
- net +3.3V: now also C10.1, C12.1, R10.1
- net 1PPS: now reaches U1.3 (START)
- net at U1.4 (STOP): now also JP1.2 (B)
- net 10MHZ_TDC: now reaches U1.5 (CLOCK)
- net 10MHZ_TDC: now also JP1.1 (A)
- net GND: now reaches U1.7 (GND)
- net GND: now also C10.2, C12.2, C9.2
- net at U1.8 (INTB): now also R10.2
- net MCU_SPI2_MISO: now reaches U1.9 (DOUT)
- new net: U9.16 (VSS), U9.32 (VSS), U9.33 (VSS)
- no-connect marks 0 -> 2
Other:
- note added: "BOOT0"
- note added: "Time-to-Digital Converter"
- moved on the sheet: U1

Commit message: pdf and sch update
Parts:
- added C13, C14, C15: 100nF, GPSDO_Rev1.0:C_0402_1005Metric, symbol GPSDO_Rev1.0:C
- added R11, R14: 5.1K, GPSDO_Rev1.0:R_0402_1005Metric, symbol GPSDO_Rev1.0:R
- added U11: CH340E, GPSDO_Rev1.0:CH340E, symbol GPSDO_Rev1.0:CH340E
- added USB1: TYPE-C_16PIN_2MD_073, GPSDO_Rev1.0:TYPE-C_16PIN_2MD_073, symbol GPSDO_Rev1.0:TYPE-C_16PIN_2MD_073
Connections:
- net +3.3V: now also U9.1 (VDD), U9.15 (VDDA), U9.17 (VDD), C13.1, C14.1, C15.1, U11.10 (V3), U11.7 (VCC)
- net GND: now also U9.14 (VSSA), U9.16 (VSS), U9.31 (PB8), U9.32 (VSS), U9.33 (VSS), C13.2, C14.2, C15.2, R11.1, R14.1, U11.3 (GND), USB1.13 (EH), USB1.14 (EH), USB1.A1B12 (GND), USB1.B1A12 (GND)
- net PWM: now reaches U9.10 (PA5)
- net TXD: now reaches U9.19 (PA9)
- net 10MHZ_MCU: now reaches U9.2 (PF0)
- net RXD: now reaches U9.20 (PA10)
- net SWDIO: now reaches U9.23 (PA13)
- net SWCLK: now reaches U9.24 (PA14)
- net RX2: now reaches U9.27 (PB4)
- net RX2: now also U11.8 (TXD)
- net TX2: now reaches U9.7 (PA2)
- net TX2: now also U11.9 (RXD)
- new net: R11.2, USB1.A5 (CC1)
- new net: R14.2, USB1.B5 (CC2)
- new net USB_D+: U11.1 (UD+), USB1.A6 (Dp1), USB1.B6 (Dp2)
- new net USB_D-: U11.2 (UD-), USB1.A7 (Dn1), USB1.B7 (Dn2)
- new net VBUS: USB1.A4B9 (VBUS), USB1.B4A9 (VBUS)
- no-connect marks 2 -> 8
Other:
- note added: "32bit TIM"
- note added: "Microcontroller"
- note added: "USB Connector"
- moved on the sheet: U9
