File: hardware/schematic/v1.0/GPSDO_Rev1.0/MCU.kicad_sch (KiCad schematic)
At the start: 14 parts, among them U1 TDC7200PWR, U11 CH340E, U9 STM32G431KBUx

Commit message: sch update
Parts:
- added FB1, FB2: 100R, GPSDO_Rev1.0:L_0603_1608Metric, symbol GPSDO_Rev1.0:FerriteBead_Small
Connections:
- net +3.3V: now also FB1.2, FB2.2; no longer C10.1, C12.1, C13.1, C14.1, C15.1, R10.1, U1.14 (VDD), U9.1 (VDD), U9.15 (VDDA), U9.17 (VDD)
- new net: C10.1, C12.1, FB2.1, R10.1, U1.14 (VDD)
- new net: C13.1, C14.1, C15.1, FB1.1, U9.1 (VDD), U9.15 (VDDA), U9.17 (VDD)
Other:
- moved on the sheet: C13, C14, C15

Commit message: sch upate
Parts:
- added FB6: 100R, GPSDO_Rev1.0:L_0603_1608Metric, symbol GPSDO_Rev1.0:FerriteBead_Small
Connections:
- net +3.3V: now also FB6.2; no longer U11.10 (V3), U11.7 (VCC)
- new net: FB6.1, U11.10 (V3), U11.7 (VCC)
Changed lines of the file:
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@@
+	(wire
+		(pts
+			(xy 273.05 63.5) (xy 273.05 64.77)
+		)
+		(stroke
+			(width 0)
+			(type default)
+		)
+	)
 	(wire
 		(pts
@@
 	)
 	(symbol
-		(lib_id "power:+3.3V")
-		(at 273.05 69.85 0)
-		(unit 1)
-		(body_style 1)
-		(exclude_from_sim no)
-		(in_bom yes)
-		(on_board yes)
-		(in_pos_files yes)
-		(dnp no)
-		(fields_autoplaced yes)
-		(property "Reference" "#PWR015"
-			(at 273.05 73.66 0)
-			(hide yes)
-			(show_name no)
-			(do_not_autoplace no)
-			(effects
-				(font
-					(size 1.27 1.27)
-				)
-			)
-		)
-		(property "Value" "+3.3V"
-			(at 273.05 64.77 0)
-			(show_name no)
-			(do_not_autoplace no)
-			(effects
-				(font
-					(size 1.27 1.27)
-				)
-			)
-		)
-		(property "Footprint" ""
-			(at 273.05 69.85 0)
-			(hide yes)
-			(show_name no)
-			(do_not_autoplace no)
-			(effects
-				(font
-					(size 1.27 1.27)
-				)
-			)
-		)
-		(property "Datasheet" ""
-			(at 273.05 69.85 0)
-			(hide yes)
-			(show_name no)
-			(do_not_autoplace no)
-			(effects
-				(font
-					(size 1.27 1.27)
-				)
-			)
-		)
-		(property "Description" "Power symbol creates a global label with name \"+3.3V\""
-			(at 273.05 69.85 0)
-			(hide yes)
-			(show_name no)
-			(do_not_autoplace no)
-			(effects
-				(font
-					(size 1.27 1.27)
-				)
-			)
-		)
-		(pin "1"
-		)
-		(instances
-			(project "GPSDO_Rev1.0"
-				(path "/7fcb1340-2836-48b1-8b47-374fa7e6ca96/a223c499-b8b9-41df-ac1a-b6212c61923a"
-					(reference "#PWR015")
-					(unit 1)
-				)
-			)
-		)
-	)
-	(symbol
 		(lib_id "power:GND")
 		(at 72.39 78.74 0)
@@
 	)
 	(symbol
+		(lib_id "power:+3.3V")
+		(at 273.05 63.5 0)
+		(unit 1)
+		(body_style 1)
+		(exclude_from_sim no)
+		(in_bom yes)
+		(on_board yes)
+		(in_pos_files yes)
+		(dnp no)
+		(fields_autoplaced yes)
+		(property "Reference" "#PWR015"
+			(at 273.05 67.31 0)
+			(hide yes)
+			(show_name no)
+			(do_not_autoplace no)
+			(effects
+				(font
+					(size 1.27 1.27)
+				)
+			)
+		)
+		(property "Value" "+3.3V"
+			(at 273.05 58.42 0)
+			(show_name no)
+			(do_not_autoplace no)
+			(effects
+				(font
+					(size 1.27 1.27)
+				)
+			)
+		)
+		(property "Footprint" ""
+			(at 273.05 63.5 0)
+			(hide yes)
+			(show_name no)
+			(do_not_autoplace no)
+			(effects
+				(font
+					(size 1.27 1.27)
+				)
+			)
+		)
+		(property "Datasheet" ""
+			(at 273.05 63.5 0)
+			(hide yes)
+			(show_name no)
+			(do_not_autoplace no)
+			(effects
+				(font
+					(size 1.27 1.27)
+				)
+			)
+		)
+		(property "Description" "Power symbol creates a global label with name \"+3.3V\""
+			(at 273.05 63.5 0)
+			(hide yes)
+			(show_name no)
+			(do_not_autoplace no)
+			(effects
+				(font
+					(size 1.27 1.27)
+				)
+			)
+		)
+		(pin "1"
+		)
+		(instances
+			(project "GPSDO_Rev1.0"
+				(path "/7fcb1340-2836-48b1-8b47-374fa7e6ca96/a223c499-b8b9-41df-ac1a-b6212c61923a"
+					(reference "#PWR015")
+					(unit 1)
+				)
+			)
+		)
+	)
+	(symbol
 		(lib_id "power:GND")
 		(at 237.49 31.75 90)
@@
 					(unit 1)
 				)
+			)
+		)
+	)
+	(symbol
+		(lib_id "GPSDO_Rev1.0:FerriteBead_Small")
+		(at 273.05 67.31 180)
+		(unit 1)
+		(body_style 1)
+		(exclude_from_sim no)
+		(in_bom yes)
+		(on_board yes)
+		(in_pos_files yes)
+		(dnp no)
+		(property "Reference" "FB6"
+			(at 269.494 64.516 0)
+			(show_name no)
+			(do_not_autoplace no)
+			(effects
+				(font
+					(size 1.27 1.27)
+				)
+			)
+		)
+		(property "Value" "100R"
+			(at 268.986 68.834 0)
+			(show_name no)
+			(do_not_autoplace no)
+			(effects
+				(font
+					(size 1.27 1.27)
+				)
+			)
+		)
+		(property "Footprint" "GPSDO_Rev1.0:L_0603_1608Metric"
+			(at 274.828 67.31 90)
+			(hide yes)
+			(show_name no)
+			(do_not_autoplace no)
+			(effects
+				(font
+					(size 1.27 1.27)
+				)
+			)
+		)
+		(property "Datasheet" ""
+			(at 273.05 67.31 0)
+			(hide yes)
+			(show_name no)
+			(do_not_autoplace no)
+			(effects
+				(font
+					(size 1.27 1.27)
+				)
+			)
+		)
+		(property "Description" "Ferrite bead, small symbol"
+			(at 273.05 67.31 0)
+			(hide yes)
+			(show_name no)
+			(do_not_autoplace no)
+			(effects
+				(font
+					(size 1.27 1.27)
+				)
+			)
+		)
+		(pin "2"
+		)
+		(pin "1"
+		)
+		(instances
+			(project "GPSDO_Rev1.0"
+				(path "/7fcb1340-2836-48b1-8b47-374fa7e6ca96/a223c499-b8b9-41df-ac1a-b6212c61923a"
+					(reference "FB6")
+					(unit 1)
+				)

Commit message: sch update
Other:
- note added: "SWD Connector"
- moved on the sheet: C10, C12, C9, FB2, FB6, JP1, R10, R11, R14, U1, U11, USB1

Commit message: sch update
Parts:
- added C32, C33: 100nF, GPSDO_Rev1.0:C_0402_1005Metric, symbol GPSDO_Rev1.0:C
- added U15: STM32G431CBU6, GPSDO_Rev1.0:STM32G431CBU6, symbol GPSDO_Rev1.0:STM32G431CBU6
Connections:
- net MCU_SPI2_MISO is gone; now on net MCU_SPI1_MISO: U1.9 (DOUT)
- net MCU_SPI2_MOSI is gone; now on net MCU_SPI1_MOSI: U1.10 (DIN)
- net MCU_SPI2_NSS is gone; now on net MCU_SPI1_NSS: U1.11 (CSB)
- net 10MHZ_MCU: now also U15.5 (PF0-OSC_IN)
- net GND: now also C32.2, C33.2, U15.46 (PB8-BOOT0); no longer U9.14 (VSSA), U9.16 (VSS), U9.31 (PB8), U9.32 (VSS), U9.33 (VSS)
- net PWM: no longer U9.10 (PA5)
- net RX2: now also U15.11 (PA3); no longer U9.27 (PB4)
- net SWCLK: now also U15.37 (PA14); no longer U9.24 (PA14)
- net SWDIO: now also U15.36 (PA13); no longer U9.23 (PA13)
- net TX2: now also U15.10 (PA2); no longer U9.7 (PA2)
- net VBAT: now reaches C13.1, C14.1, C15.1, FB1.1
- net VBAT: now also C32.1, C33.1, U15.1 (VBAT), U15.21 (VDDA), U15.23 (VDD), U15.35 (VDD), U15.48 (VDD); no longer U9.1 (VDD), U9.15 (VDDA), U9.17 (VDD)
- net MCU_SPI1_MISO: now reaches U9.11 (PA6)
- net MCU_SPI1_MOSI: now reaches U9.12 (PA7)
- net MCU_SPI1_NSS: now reaches U9.9 (PA4)
- net MCU_SPI2_SCK renamed MCU_SPI1_SCK
- net MCU_SPI1_SCK: now also U9.10 (PA5)
- new net: U9.1 (VDD), U9.15 (VDDA), U9.17 (VDD)
- new net: U9.14 (VSSA), U9.16 (VSS), U9.32 (VSS), U9.33 (VSS)
- no-connect marks 8 -> 9
Other:
- moved on the sheet: U9

Commit message: sch update
Connections:
- net GND: now also U15.49 (VSS)
- net MCU_SPI1_MISO: no longer U1.9 (DOUT)
- net MCU_SPI1_MOSI: no longer U1.10 (DIN)
- net MCU_SPI1_NSS: no longer U1.11 (CSB)
- net MCU_SPI1_SCK: no longer U1.12 (SCLK)
- net TMP_SCL: now also U15.38 (PA15)
- net TMP_SDA: now also U15.45 (PB7)
- net TDC_SPI1_NSS: now reaches U15.12 (PA4)
- net TDC_SPI1_NSS: now also U1.11 (CSB)
- net TDC_SPI1_SCK: now reaches U15.13 (PA5)
- net TDC_SPI1_SCK: now also U1.12 (SCLK)
- net TDC_SPI1_MISO: now reaches U15.14 (PA6)
- net TDC_SPI1_MISO: now also U1.9 (DOUT)
- net TDC_SPI1_MOSI: now reaches U15.15 (PA7)
- net TDC_SPI1_MOSI: now also U1.10 (DIN)
- no-connect marks 9 -> 11
Changed lines of the file:
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@@
+	)
+	(no_connect
+		(at 59.69 130.81)
 	)
 	(no_connect
@@
 	)
 	(no_connect
+		(at 59.69 128.27)
+	)
+	(no_connect
 		(at 255.27 55.88)
 	)
@@
 		)
 	)
+	(wire
+		(pts
+			(xy 107.95 105.41) (xy 110.49 105.41)
+		)
+		(stroke
+			(width 0)
+			(type default)
+		)
+	)
 	(polyline
 		(pts
@@
 	(wire
 		(pts
+			(xy 107.95 82.55) (xy 121.92 82.55)
+		)
+		(stroke
+			(width 0)
+			(type default)
+		)
+	)
+	(wire
+		(pts
 			(xy 166.37 57.15) (xy 168.91 57.15)
 		)
@@
 	(wire
 		(pts
+			(xy 107.95 77.47) (xy 121.92 77.47)
+		)
+		(stroke
+			(width 0)
+			(type default)
+		)
+	)
+	(wire
+		(pts
 			(xy 93.98 50.8) (xy 101.6 50.8)
 		)
@@
 	(wire
 		(pts
+			(xy 107.95 85.09) (xy 121.92 85.09)
+		)
+		(stroke
+			(width 0)
+			(type default)
+		)
+	)
+	(wire
+		(pts
 			(xy 93.98 43.18) (xy 101.6 43.18)
 		)
@@
 	(wire
 		(pts
+			(xy 107.95 130.81) (xy 110.49 130.81)
+		)
+		(stroke
+			(width 0)
+			(type default)
+		)
+	)
+	(wire
+		(pts
 			(xy 255.27 50.8) (xy 261.62 50.8)
 		)
@@
 			(width 0)
 			(type dash)
+		)
+	)
+	(wire
+		(pts
+			(xy 107.95 80.01) (xy 121.92 80.01)
+		)
+		(stroke
+			(width 0)
+			(type default)
 		)
 	)
@@
 		)
 	)
+	(label "TDC_SPI1_SCK"
+		(at 109.22 80.01 0)
+		(effects
+			(font
+				(size 1.27 1.27)
+			)
+			(justify left bottom)
+		)
+	)
+	(label "TDC_SPI1_NSS"
+		(at 109.22 77.47 0)
+		(effects
+			(font
+				(size 1.27 1.27)
+			)
+			(justify left bottom)
+		)
+	)
 	(label "RX2"
 		(at 109.22 74.93 0)
@@
 		)
 	)
-	(label "MCU_SPI1_MISO"
+	(label "TDC_SPI1_MISO"
 		(at 213.36 110.49 0)
 		(effects
@@
 		)
 	)
-	(label "MCU_SPI1_MOSI"
+	(label "TDC_SPI1_MOSI"
 		(at 213.36 107.95 0)
 		(effects
@@
 		)
 	)
-	(label "MCU_SPI1_SCK"
+	(label "TDC_SPI1_MISO"
+		(at 109.22 82.55 0)
+		(effects
+			(font
+				(size 1.27 1.27)
+			)
+			(justify left bottom)
+		)
+	)
+	(label "TDC_SPI1_SCK"
 		(at 213.36 102.87 0)
+		(effects
+			(font
+				(size 1.27 1.27)
+			)
+			(justify left bottom)
+		)
+	)
+	(label "TDC_SPI1_MOSI"
+		(at 109.22 85.09 0)
 		(effects
 			(font
@@
 		)
 	)
-	(label "MCU_SPI1_NSS"
+	(label "TDC_SPI1_NSS"
 		(at 213.36 105.41 0)
 		(effects
@@
 			)
 			(justify left bottom)
+		)
+	)
+	(hierarchical_label "TMP_SDA"
+		(shape bidirectional)
+		(at 110.49 130.81 0)
+		(effects
+			(font
+				(size 1.27 1.27)
+			)
+			(justify left)
 		)
 	)
@@
 		(shape input)
 		(at -35.56 73.66 0)
+		(effects
+			(font
+				(size 1.27 1.27)
+			)
+			(justify left)
+		)
+	)
+	(hierarchical_label "TMP_SCL"
+		(shape output)
+		(at 110.49 105.41 0)
 		(effects
 			(font
@@
 	(symbol
 		(lib_id "power:GND")
-		(at 88.9 186.69 0)
+		(at 83.82 162.56 0)
 		(unit 1)
 		(body_style 1)
@@
 		(dnp no)
 		(property "Reference" "#PWR0146"
-			(at 88.9 193.04 0)
+			(at 83.82 168.91 0)
 			(hide yes)
 			(show_name no)
@@
 		)
 		(property "Value" "GND"
-			(at 88.9 189.738 90)
+			(at 83.82 165.608 90)
 			(hide yes)
 			(show_name no)
@@
 		)
 		(property "Footprint" ""
-			(at 88.9 186.69 0)
+			(at 83.82 162.56 0)
 			(hide yes)
 			(show_name no)
@@
 		)
 		(property "Datasheet" ""
-			(at 88.9 186.69 0)
+			(at 83.82 162.56 0)
 			(hide yes)
 			(show_name no)
@@
 		)
 		(property "Description" "Power symbol creates a global label with name \"GND\" , ground"
-			(at 88.9 186.69 0)
-			(hide yes)
-			(show_name no)
+			(at 83.82 162.56 0)
+			(hide yes)
+			(show_name no)

Commit message: sch update
Parts:
- added C42: 100nF, GPSDO_Rev1.0:C_0402_1005Metric, symbol GPSDO_Rev1.0:C
Connections:
- net GND: now also C42.1
- net PWM: now also U15.8 (PA0)
- net PULSE_GNSS: now reaches U15.24 (PB11)
- net USART1_TX: now reaches U15.31 (PA9)
- net USART1_TX: now also U11.9 (RXD)
- net USART1_RX: now reaches U15.32 (PA10)
- net USART1_RX: now also U11.8 (TXD)
- net NRST: now reaches U15.7 (PG10-NRST)
- net NRST: now also C42.2
- net RX2 renamed GNSS_UART_TXD
- net GNSS_UART_TXD: no longer U11.8 (TXD)
- net TX2 renamed GNSS_UART_RXD
- net GNSS_UART_RXD: no longer U11.9 (RXD)
- no-connect marks 11 -> 12
Other:
- moved on the sheet: C13, C14, C15, C32, C33, FB1, FB6, U15

Commit message: sch update
Parts:
- added J3: Conn_01x04_Socket, Connector_PinHeader_2.54mm:PinHeader_1x04_P2.54mm_Vertical, symbol Connector:Conn_01x04_Socket
Connections:
- net 1PPS is gone; now on net PULSE_GNSS: U1.3 (START)
- net GND: now also J3.2 (Pin_2)
- net NRST: now also J3.1 (Pin_1)
- net SWCLK: now also J3.3 (Pin_3)
- net SWDIO: now also J3.4 (Pin_4)
Changed lines of the file:
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@@
 		)
 	)
+	(wire
+		(pts
+			(xy 179.07 153.67) (xy 190.5 153.67)
+		)
+		(stroke
+			(width 0)
+			(type default)
+		)
+	)
 	(polyline
 		(pts
@@
 	(wire
 		(pts
+			(xy 179.07 146.05) (xy 190.5 146.05)
+		)
+		(stroke
+			(width 0)
+			(type default)
+		)
+	)
+	(wire
+		(pts
 			(xy 82.55 52.07) (xy 90.17 52.07)
 		)
@@
 	(wire
 		(pts
+			(xy 179.07 151.13) (xy 190.5 151.13)
+		)
+		(stroke
+			(width 0)
+			(type default)
+		)
+	)
+	(wire
+		(pts
 			(xy -64.77 73.66) (xy -63.5 73.66)
 		)
@@
 		)
 	)
+	(label "SWCLK"
+		(at 179.07 151.13 0)
+		(effects
+			(font
+				(size 1.27 1.27)
+			)
+			(justify left bottom)
+		)
+	)
 	(label "RESET"
 		(at -71.12 48.26 0)
@@
 		)
 	)
+	(label "NRST"
+		(at 179.07 146.05 0)
+		(effects
+			(font
+				(size 1.27 1.27)
+			)
+			(justify left bottom)
+		)
+	)
 	(label "USART1_RX"
 		(at 105.41 93.98 0)
@@
 		)
 	)
+	(label "SWDIO"
+		(at 179.07 153.67 0)
+		(effects
+			(font
+				(size 1.27 1.27)
+			)
+			(justify left bottom)
+		)
+	)
 	(label "MCU_SPI1_MOSI"
 		(at -36.83 66.04 0)
@@
 		)
 	)
+	(hierarchical_label "PULSE_GNSS"
+		(shape input)
+		(at 179.07 100.33 180)
+		(effects
+			(font
+				(size 1.27 1.27)
+			)
+			(justify right)
+		)
+	)
 	(hierarchical_label "GNSS_UART_RXD"
 		(shape output)
@@
 		)
 	)
-	(hierarchical_label "1PPS"
-		(shape input)
-		(at 179.07 100.33 180)
-		(effects
-			(font
-				(size 1.27 1.27)
-			)
-			(justify right)
-		)
-	)
 	(hierarchical_label "PULSE_GNSS"
 		(shape input)
@@
 	)
 	(symbol
+		(lib_id "Connector:Conn_01x04_Socket")
+		(at 195.58 148.59 0)
+		(unit 1)
+		(body_style 1)
+		(exclude_from_sim no)
+		(in_bom yes)
+		(on_board yes)
+		(in_pos_files yes)
+		(dnp no)
+		(fields_autoplaced yes)
+		(property "Reference" "J3"
+			(at 196.85 148.5899 0)
+			(show_name no)
+			(do_not_autoplace no)
+			(effects
+				(font
+					(size 1.27 1.27)
+				)
+				(justify left)
+			)
+		)
+		(property "Value" "Conn_01x04_Socket"
+			(at 196.85 151.1299 0)
+			(show_name no)
+			(do_not_autoplace no)
+			(effects
+				(font
+					(size 1.27 1.27)
+				)
+				(justify left)
+			)
+		)
+		(property "Footprint" "Connector_PinHeader_2.54mm:PinHeader_1x04_P2.54mm_Vertical"
+			(at 195.58 148.59 0)
+			(hide yes)
+			(show_name no)
+			(do_not_autoplace no)
+			(effects
+				(font
+					(size 1.27 1.27)
+				)
+			)
+		)
+		(property "Datasheet" ""
+			(at 195.58 148.59 0)
+			(hide yes)
+			(show_name no)
+			(do_not_autoplace no)
+			(effects
+				(font
+					(size 1.27 1.27)
+				)
+			)
+		)
+		(property "Description" "Generic connector, single row, 01x04, script generated"
+			(at 195.58 148.59 0)
+			(hide yes)
+			(show_name no)
+			(do_not_autoplace no)
+			(effects
+				(font
+					(size 1.27 1.27)
+				)
+			)
+		)
+		(pin "4"
+		)
+		(pin "1"
+		)
+		(pin "3"
+		)
+		(pin "2"
+		)
+		(instances
+			(project "GPSDO_Rev1.0"
+				(path "/7fcb1340-2836-48b1-8b47-374fa7e6ca96/a223c499-b8b9-41df-ac1a-b6212c61923a"
+					(reference "J3")
+					(unit 1)
+				)
+			)
+		)
+	)
+	(symbol
 		(lib_id "GPSDO_Rev1.0:TYPE-C_16PIN_2MD_073")
 		(at 194.31 48.26 0)
@@
 					(unit 1)
 				)
+			)
+		)
+	)
+	(symbol
+		(lib_id "power:GND")
+		(at 190.5 148.59 270)
+		(unit 1)
+		(body_style 1)
+		(exclude_from_sim no)
+		(in_bom yes)
+		(on_board yes)
+		(in_pos_files yes)
+		(dnp no)
+		(property "Reference" "#PWR0158"
+			(at 184.15 148.59 0)
+			(hide yes)
+			(show_name no)
+			(do_not_autoplace no)
+			(effects
+				(font
+					(size 1.27 1.27)
+				)
+			)
+		)
+		(property "Value" "GND"
+			(at 187.452 148.59 90)
+			(hide yes)
+			(show_name no)
+			(do_not_autoplace no)
+			(effects
+				(font
+					(size 1.27 1.27)
+				)
+				(justify right)
+			)
+		)
+		(property "Footprint" ""
+			(at 190.5 148.59 0)
+			(hide yes)
+			(show_name no)
+			(do_not_autoplace no)
+			(effects
+				(font
+					(size 1.27 1.27)
+				)
+			)
+		)
+		(property "Datasheet" ""
+			(at 190.5 148.59 0)
+			(hide yes)
+			(show_name no)
+			(do_not_autoplace no)
+			(effects
+				(font
+					(size 1.27 1.27)
+				)
+			)
+		)
+		(property "Description" "Power symbol creates a global label with name \"GND\" , ground"
+			(at 190.5 148.59 0)
+			(hide yes)
+			(show_name no)
+			(do_not_autoplace no)
+			(effects
+				(font
+					(size 1.27 1.27)
+				)
+			)
+		)
+		(pin "1"
+		)
+		(instances
+			(project "GPSDO_Rev1.0"
+				(path "/7fcb1340-2836-48b1-8b47-374fa7e6ca96/a223c499-b8b9-41df-ac1a-b6212c61923a"
+					(reference "#PWR0158")
+					(unit 1)
+				)

Commit message: sch update
Parts:
- added D3: GREEN, GPSDO_Rev1.0:LED_0603_1608Metric, symbol GPSDO_Rev1.0:LED
- added D4: YELLOW, GPSDO_Rev1.0:LED_0603_1608Metric, symbol GPSDO_Rev1.0:LED
- added D5: RED, GPSDO_Rev1.0:LED_0603_1608Metric, symbol GPSDO_Rev1.0:LED
- added R21, R24, R25: 2.2K, GPSDO_Rev1.0:R_0402_1005Metric, symbol GPSDO_Rev1.0:R
Connections:
- net GND: now also D3.1 (K), D4.1 (K), D5.1 (K)
- net PULSE_GNSS: now also U15.29 (PC6); no longer U15.24 (PB11)
- net LED_RED: now reaches U15.16 (PC4)
- net LED_RED: now also R25.2
- net LED_GREEN: now reaches U15.39 (PC10)
- net LED_GREEN: now also R21.2
- net LED_YELLOW: now reaches U15.40 (PC11)
- net LED_YELLOW: now also R24.2
- new net: D3.2 (A), R21.1
- new net: D5.2 (A), R25.1
- new net: D4.2 (A), R24.1
Other:
- moved on the sheet: J3
