File: hardware/schematic/v1.0/GPSDO_Rev1.0/MCU.kicad_sch (KiCad schematic)
At the start: 27 parts, among them J3 Conn_01x04_Socket, U1 TDC7200PWR, U11 CH340E, U15 STM32G431CBU6

Commit message: sch update
Parts:
- added R38: 0, GPSDO_Rev1.0:R_0402_1005Metric, symbol GPSDO_Rev1.0:R__R_0402_1005Metric
Connections:
- net PULSE_GNSS: now also U15.24 (PB11); no longer U15.29 (PC6)
- net PULSE_MCU: now also R38.1
- net PWM: now also U15.34 (PA12); no longer U15.8 (PA0)
- net TIM2_CH3: now reaches U15.22 (PB10)
- net TIM2_CH3: now also R38.2
- net VCTL: now reaches U15.9 (PA1)
Changed lines of the file:
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@@
 	(text "Microcontroller"
 		(exclude_from_sim no)
-		(at 48.26 26.416 0)
+		(at 35.814 27.432 0)
 		(effects
 			(font
@@
 	(text "32bit TIM"
 		(exclude_from_sim no)
-		(at 116.332 68.834 0)
+		(at 122.428 145.034 0)
 		(effects
 			(font
@@
 	(wire
 		(pts
+			(xy 127 139.7) (xy 125.73 139.7)
+		)
+		(stroke
+			(width 0)
+			(type default)
+		)
+	)
+	(wire
+		(pts
 			(xy 247.65 110.49) (xy 247.65 113.03)
 		)
@@
 	(wire
 		(pts
-			(xy 104.14 106.68) (xy 106.68 106.68)
+			(xy 104.14 106.68) (xy 118.11 106.68)
 		)
 		(stroke
@@
 	(polyline
 		(pts
-			(xy 27.94 21.59) (xy 27.94 176.53)
+			(xy 16.51 21.59) (xy 16.51 176.53)
 		)
 		(stroke
@@
 	(wire
 		(pts
-			(xy 50.8 119.38) (xy 55.88 119.38)
+			(xy 39.37 119.38) (xy 55.88 119.38)
 		)
 		(stroke
@@
 		)
 	)
+	(wire
+		(pts
+			(xy 104.14 142.24) (xy 127 142.24)
+		)
+		(stroke
+			(width 0)
+			(type default)
+		)
+	)
 	(polyline
 		(pts
-			(xy 27.94 176.53) (xy 139.7 176.53)
+			(xy 16.51 176.53) (xy 143.51 176.53)
 		)
 		(stroke
@@
 	(polyline
 		(pts
-			(xy 27.94 21.59) (xy 139.7 21.59)
+			(xy 16.51 21.59) (xy 143.51 21.59)
 		)
 		(stroke
@@
 	(wire
 		(pts
+			(xy 118.11 99.06) (xy 104.14 99.06)
+		)
+		(stroke
+			(width 0)
+			(type default)
+		)
+	)
+	(wire
+		(pts
 			(xy 104.14 104.14) (xy 113.03 104.14)
 		)
@@
 	(wire
 		(pts
+			(xy 118.11 71.12) (xy 104.14 71.12)
+		)
+		(stroke
+			(width 0)
+			(type default)
+		)
+	)
+	(wire
+		(pts
 			(xy 76.2 44.45) (xy 82.55 44.45)
 		)
@@
 	(polyline
 		(pts
-			(xy 139.7 21.59) (xy 139.7 176.53)
+			(xy 143.51 21.59) (xy 143.51 176.53)
 		)
 		(stroke
@@
 		(pts
 			(xy 179.07 100.33) (xy 182.88 100.33)
+		)
+		(stroke
+			(width 0)
+			(type default)
+		)
+	)
+	(wire
+		(pts
+			(xy 104.14 139.7) (xy 118.11 139.7)
 		)
 		(stroke
@@
 		)
 	)
+	(label "TIM2_CH3"
+		(at 105.41 139.7 0)
+		(effects
+			(font
+				(size 1.27 1.27)
+			)
+			(justify left bottom)
+		)
+	)
+	(label "TIM2_CH4"
+		(at 105.41 142.24 0)
+		(effects
+			(font
+				(size 1.27 1.27)
+			)
+			(justify left bottom)
+		)
+	)
 	(label "LED_GREEN"
 		(at 219.71 143.51 0)
@@
 		)
 	)
+	(label "TIM4_CH2"
+		(at 105.41 99.06 0)
+		(effects
+			(font
+				(size 1.27 1.27)
+			)
+			(justify left bottom)
+		)
+	)
 	(label "TDC_SPI1_MOSI"
 		(at 213.36 107.95 0)
@@
 		)
 	)
+	(label "ADC1_IN2"
+		(at 105.41 71.12 0)
+		(effects
+			(font
+				(size 1.27 1.27)
+			)
+			(justify left bottom)
+		)
+	)
 	(label "USB_D-"
 		(at 168.91 44.45 0)
@@
 			)
 			(justify left bottom)
+		)
+	)
+	(hierarchical_label "PULSE_GNSS"
+		(shape input)
+		(at 127 142.24 0)
+		(effects
+			(font
+				(size 1.27 1.27)
+			)
+			(justify left)
 		)
 	)
@@
 		)
 	)
+	(hierarchical_label "VCTL"
+		(shape input)
+		(at 118.11 71.12 0)
+		(effects
+			(font
+				(size 1.27 1.27)
+			)
+			(justify left)
+		)
+	)
 	(hierarchical_label "GNSS_UART_RXD"
 		(shape output)
@@
 	(hierarchical_label "PULSE_MCU"
 		(shape output)
-		(at 152.4 185.42 0)
-		(effects
-			(font
-				(size 1.27 1.27)
-			)
-			(justify left)
-		)
-	)
-	(hierarchical_label "PWM"
-		(shape output)
-		(at 105.41 68.58 0)
+		(at 127 139.7 0)
 		(effects
 			(font
@@
 		)
 	)
-	(hierarchical_label "PULSE_GNSS"
-		(shape input)
-		(at 50.8 119.38 180)
-		(effects
-			(font
-				(size 1.27 1.27)
-			)
-			(justify right)
+	(hierarchical_label "PWM"
+		(shape output)
+		(at 118.11 99.06 0)
+		(effects
+			(font
+				(size 1.27 1.27)
+			)
+			(justify left)
 		)
 	)
 	(hierarchical_label "TMP_SCL"
 		(shape output)
-		(at 106.68 106.68 0)
+		(at 118.11 106.68 0)
 		(effects
 			(font
@@
 					(unit 1)
 				)
+			)
+		)
+	)
+	(symbol
+		(lib_id "GPSDO_Rev1.0:R__R_0402_1005Metric")
+		(at 121.92 139.7 270)
+		(unit 1)
+		(body_style 1)
+		(exclude_from_sim no)
+		(in_bom yes)
+		(on_board yes)
+		(in_pos_files yes)
+		(dnp no)
+		(property "Reference" "R38"
+			(at 117.094 138.176 90)
+			(show_name no)
+			(do_not_autoplace no)
+			(effects
+				(font
+					(size 1.27 1.27)
+				)
+			)
+		)
+		(property "Value" "0"
+			(at 125.476 138.176 90)
+			(show_name no)
+			(do_not_autoplace no)
+			(effects
+				(font
+					(size 1.27 1.27)
+				)
+			)
+		)
+		(property "Footprint" "GPSDO_Rev1.0:R_0402_1005Metric"
+			(at 121.92 137.922 90)
+			(hide yes)
+			(show_name no)
+			(do_not_autoplace no)
+			(effects
+				(font
+					(size 1.27 1.27)
+				)
+			)
+		)
+		(property "Datasheet" ""
+			(at 121.92 139.7 0)
+			(hide yes)
+			(show_name no)
+			(do_not_autoplace no)
+			(effects
+				(font
+					(size 1.27 1.27)
+				)
+			)
+		)
+		(property "Description" "Resistor"
+			(at 121.92 139.7 0)
+			(hide yes)
+			(show_name no)
+			(do_not_autoplace no)
+			(effects
+				(font
+					(size 1.27 1.27)
+				)
+			)
+		)
+		(pin "1"
+		)
+		(pin "2"
+		)
+		(instances
+			(project "GPSDO_Rev1.0"
+				(path "/7fcb1340-2836-48b1-8b47-374fa7e6ca96/a223c499-b8b9-41df-ac1a-b6212c61923a"
+					(reference "R38")
+					(unit 1)
+				)

Commit message: sch update
Connections:
- net VBAT: now also U15.20 (VREF+)
- no-connect marks 11 -> 26
Changed lines of the file:
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@@
+	)
+	(junction
+		(at 55.88 106.68)
+		(diameter 0)
+		(color 0 0 0 0)
 	)
 	(junction
@@
 	)
 	(no_connect
+		(at 104.14 129.54)
+	)
+	(no_connect
+		(at 104.14 152.4)
+	)
+	(no_connect
+		(at 104.14 116.84)
+	)
+	(no_connect
 		(at 55.88 132.08)
 	)
 	(no_connect
+		(at 104.14 144.78)
+	)
+	(no_connect
+		(at 104.14 127)
+	)
+	(no_connect
+		(at 104.14 114.3)
+	)
+	(no_connect
+		(at 55.88 127)
+	)
+	(no_connect
+		(at 104.14 121.92)
+	)
+	(no_connect
 		(at 186.69 110.49)
 	)
@@
 	)
 	(no_connect
+		(at 105.41 68.58)
+	)
+	(no_connect
 		(at 229.87 55.88)
 	)
 	(no_connect
+		(at 104.14 147.32)
+	)
+	(no_connect
 		(at 180.34 39.37)
 	)
@@
 	)
 	(no_connect
+		(at 104.14 88.9)
+	)
+	(no_connect
+		(at 104.14 137.16)
+	)
+	(no_connect
 		(at 55.88 99.06)
 	)
 	(no_connect
+		(at 104.14 124.46)
+	)
+	(no_connect
+		(at 104.14 119.38)
+	)
+	(no_connect
 		(at 255.27 55.88)
 	)
@@
 	)
 	(no_connect
-		(at 55.88 109.22)
+		(at 104.14 149.86)
+	)
+	(no_connect
+		(at 104.14 96.52)
 	)
 	(wire
@@
 		)
 		(stroke
+			(width 0)
+			(type default)
+		)
+	)
+	(wire
+		(pts
+			(xy 55.88 106.68) (xy 55.88 109.22)
+		)
+		(stroke

Commit message: sch update
Connections:
- no-connect marks 26 -> 27
Changed lines of the file:
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@@
+	)
+	(no_connect
+		(at 55.88 119.38)
 	)
 	(no_connect
@@
 		)
 		(stroke
-			(width 0)
-			(type default)
-		)
-	)
-	(wire
-		(pts
-			(xy 39.37 119.38) (xy 55.88 119.38)
-		)
-		(stroke

Commit message: sch update
Connections:
- net TDC_ENABLE: now also U15.30 (PA8)
- no-connect marks 27 -> 26
Changed lines of the file:
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@@
-	)
-	(no_connect
-		(at 104.14 88.9)
 	)
 	(no_connect
@@
 		(pts
 			(xy 257.81 143.51) (xy 266.7 143.51)
+		)
+		(stroke
+			(width 0)
+			(type default)
+		)
+	)
+	(wire
+		(pts
+			(xy 104.14 88.9) (xy 118.11 88.9)
 		)
 		(stroke
@@
 		(effects
 			(font
+				(size 1.27 1.27)
+			)
+			(justify left bottom)
+		)
+	)
+	(label "TDC_ENABLE"
+		(at 105.41 88.9 0)
+		(effects
+			(font

Commit message: sch update
Parts:
- added R48: 10K, GPSDO_Rev1.0:R_0402_1005Metric, symbol GPSDO_Rev1.0:R__R_0402_1005Metric
Connections:
- net GND: now also R48.2; no longer U15.46 (PB8-BOOT0)
- net LED_RED: now also U15.41 (PB3); no longer U15.16 (PC4)
- net BOOST_EN: now reaches U15.17 (PB0)
- net TIM2_CH3: no longer names the net of R38.2, U15.22 (PB10)
- new net: R48.1, U15.46 (PB8-BOOT0)
- no-connect marks 26 -> 24
Other:
- note added: "ADC1_IN2"
- note added: "TIM2_CH3"
- note added: "TIM2_CH4"
- note added: "TIM4_CH2"
- note added: "USART2_RX"
- note added: "USART2_TX"

Commit message: sch update
Parts:
- added C27: 100nF, GPSDO_Rev1.0:C_0402_1005Metric, symbol GPSDO_Rev1.0:C__C_0402_1005Metric
- added C28: 1uF, GPSDO_Rev1.0:C_0603_1608Metric, symbol GPSDO_Rev1.0:C
Connections:
- net GND: now also C27.2, C28.2
- net at FB6.1, U11.10 (V3), U11.7 (VCC): now also C27.1, C28.1
- no-connect marks 24 -> 25
Other:
- moved on the sheet: U11

Commit message: sch update
Changed lines of the file:
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@@
 	(hierarchical_label "10MHZ_TDC"
 		(shape input)
-		(at 170.18 107.95 270)
+		(at 170.18 107.95 180)
 		(effects
 			(font
