File: hardware/schematic/v1.0/GPSDO_Rev1.0/OCXO.kicad_sch (KiCad schematic)
At the start: 2 parts, among them U2 LMK1C1103PWR, U3 TMP117AIDRVR

Commit message: sch update
Parts:
- added C10, C11, C13, C9: 100nF, Capacitor_SMD:C_0402_1005Metric, symbol Device:C
- added C12, C56, C58: 10uF, Capacitor_SMD:C_0603_1608Metric, symbol Device:C
- added C57: 1uF, Capacitor_SMD:C_0603_1608Metric, symbol Device:C
- added R13, R14: 1K, Resistor_SMD:R_0402_1005Metric, symbol Device:R
- added R15: 3296W-1-103_C48997937, Counter:3296W-1-103_C48997937, symbol Counter:3296W-1-103_C48997937
- added R28: 10R, Resistor_SMD:R_0603_1608Metric, symbol Device:R
- added R29: 0R, Resistor_SMD:R_0603_1608Metric, symbol Device:R
- added R30: 0R, Resistor_SMD:R_0402_1005Metric, symbol Device:R
- added R39: 0R, Resistor_SMD:R_0805_2012Metric, symbol Device:R
- added RF10: KH-IPEX-K501-29, JLCImport:KH-IPEX-K501-29, symbol JLCImport:KH-IPEX-K501-29
- added TP1: Volt TestPoint, TestPoint:TestPoint_Pad_D1.0mm, symbol Connector:TestPoint
- added TP2: TestPoint, TestPoint:TestPoint_Pad_D1.0mm, symbol Connector:TestPoint
- added U5: OCXO_20x20mm, JLCImport:OCXO_20x20mm, symbol Counter:OCXO_20x20mm
- added U7: OCXO_25.4x25.4mm, JLCImport:DOPFITKR2-10M, symbol Counter:OCXO_25.4x25.4mm
- added U8: REF5040, JLCImport:REF5040, symbol JLCImport:REF5040
Connections:
- new net: C11.2, C56.1, R28.1, U8.2 (VIN)
- new net: C57.1, U8.5 (TRIM/NR)
- new net: C58.1, R29.1, U8.6 (VOUT)
- new net: R30.2, U5.2 (RF)
- new net: R39.1, U5.1 (VCC)
- new net GND: C10.2, C11.1, C12.1, C13.2, C56.2, C57.2, C58.2, R15.1, RF10.1 (GND), RF10.2 (GND), RF10.3 (GND), TP2.1, U5.3 (GND), U7.2 (GND), U8.4 (GND)
- new net OCXO_MON: C9.2, R13.2
- new net OCXO_MON_RF: C9.1, RF10.4 (SIG)
- new net OCXO_OUT: R13.1, R30.1, U7.1 (RF)
- new net OCXO_VCC: C10.1, C12.2, R28.2, R39.2, TP1.1, U7.5 (VCC)
- new net VCTRL: C13.1, R14.2, U5.4 (VCTRL/NC), U7.3 (VCTRL)
- new net VCTRL_ADJ: R14.1, R15.2
- new net VREF: R15.3, R29.2
- no-connect marks 0 -> 6
Other:
- note added: "50 OHM TRACE"
- note added: "OCXO 20x20mm"
- note added: "OCXO 25.4x25.4mm"
- note added: "OCXO 二选一"
- note added: "VREF"
- moved on the sheet: U2, U3

Commit message: sch update
Parts:
- removed C10: 100nF, Capacitor_SMD:C_0402_1005Metric, symbol Device:C
- removed C12: 10uF, Capacitor_SMD:C_0603_1608Metric, symbol Device:C
- removed R30: 0R, Resistor_SMD:R_0402_1005Metric, symbol Device:R
- removed R39: 0R, Resistor_SMD:R_0805_2012Metric, symbol Device:R
- removed U5: OCXO_20x20mm, JLCImport:OCXO_20x20mm, symbol Counter:OCXO_20x20mm
- removed U7: OCXO_25.4x25.4mm, JLCImport:DOPFITKR2-10M, symbol Counter:OCXO_25.4x25.4mm
- added C1: 100nF, GPSDO_Rev1.0:C_0402_1005Metric, symbol GPSDO_Rev1.0:C
- added C2: 10uF, GPSDO_Rev1.0:C_0603_1608Metric, symbol GPSDO_Rev1.0:C
- added R4: 0R, GPSDO_Rev1.0:R_0402_1005Metric, symbol GPSDO_Rev1.0:R
- added R5: 0R, GPSDO_Rev1.0:R_0805_2012Metric, symbol GPSDO_Rev1.0:R
- added U5: OCXO_20x20mm, GPSDO_Rev1.0:OCXO_20x20mm, symbol GPSDO_Rev1.0:OCXO_20x20mm
- added U7: OCXO_25.4x25.4mm, GPSDO_Rev1.0:DOPFITKR2-10M, symbol GPSDO_Rev1.0:OCXO_25.4x25.4mm
Connections:
- net GND: now also C1.1, C2.1, U5.3 (GND), U7.2 (GND)
- net OCXO_OUT: now also R4.2, U7.1 (RF)
- net OCXO_VCC: now also C1.2, C2.2, R5.1, U7.5 (VCC)
- net VCTRL: now also U5.4 (VCTRL/NC), U7.3 (VCTRL)
- new net: R5.2, U5.1 (VCC)
- new net: R4.1, U5.2 (RF)

Commit message: sch update
Parts:
- removed C9: 100nF, Capacitor_SMD:C_0402_1005Metric, symbol Device:C
- removed RF10: KH-IPEX-K501-29, JLCImport:KH-IPEX-K501-29, symbol JLCImport:KH-IPEX-K501-29
- added C3: 1uF, GPSDO_Rev1.0:C_0603_1608Metric, symbol GPSDO_Rev1.0:C
- added C4, C5: 100nF, GPSDO_Rev1.0:C_0402_1005Metric, symbol GPSDO_Rev1.0:C
- added R6: 0, GPSDO_Rev1.0:C_0603_1608Metric, symbol GPSDO_Rev1.0:R
- added R7: 0, GPSDO_Rev1.0:R_0603_1608Metric, symbol GPSDO_Rev1.0:R
- added RF2: KH-IPEX-K501-29, GPSDO_Rev1.0:KH-IPEX-K501-29, symbol GPSDO_Rev1.0:KH-IPEX-K501-29
- R4, R5: value 0R -> 0
Connections:
- net GND: now also U2.4 (GND), C3.2, C4.2, RF2.1 (GND), RF2.2 (GND), RF2.3 (GND)
- net OCXO_MON: now also C5.2
- net OCXO_MON_RF: now also C5.1, RF2.4 (SIG)
- net OCXO_OUT: now also U2.1 (CLKIN)
- net VCTRL: no longer C13.1, R14.2
- net +3.3V: now reaches U2.2 (1G)
- net +3.3V: now also U2.6 (VDD), C3.1, C4.1
- net 10MHZ_OUT: now reaches U2.3 (Y0)
- net at U2.5 (Y2): now also R7.1
- net at U2.8 (Y1): now also R6.1
- new net: C13.1, R14.2
- new net 10MHZ_MCU: R6.2
- new net 10MHZ_TDC: R7.2
- no-connect marks 6 -> 7
Other:
- moved on the sheet: C1, C11, C2, C56, C57, C58, R13, R28, R29, R4, R5, TP1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

Commit message: sch update
Parts:
- removed C13: 100nF, Capacitor_SMD:C_0402_1005Metric, symbol Device:C
- removed R14: 1K, Resistor_SMD:R_0402_1005Metric, symbol Device:R
- removed R15: 3296W-1-103_C48997937, Counter:3296W-1-103_C48997937, symbol Counter:3296W-1-103_C48997937
Other:
- note added: "Fanout Buffer"

Commit message: sch update
Other:
- moved on the sheet: C3, C4, R6, R7, U2

Commit message: pdf and sch update
Other:
- moved on the sheet: U3
Changed lines of the file:
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@@
 	(symbol
 		(lib_id "GPSDO_Rev1.0:TMP117AIDRVR")
-		(at 148.59 181.61 0)
+		(at 142.24 173.99 0)
 		(unit 1)
 		(body_style 1)
@@
 		(fields_autoplaced yes)
 		(property "Reference" "U3"
-			(at 148.59 170.18 0)
+			(at 142.24 162.56 0)
 			(show_name no)
 			(do_not_autoplace no)
@@
 		)
 		(property "Value" "TMP117AIDRVR"
-			(at 148.59 172.72 0)
+			(at 142.24 165.1 0)
 			(show_name no)
 			(do_not_autoplace no)
@@
 		)
 		(property "Footprint" "GPSDO_Rev1.0:TMP117AIDRVR"
-			(at 148.59 181.61 0)
+			(at 142.24 173.99 0)
 			(hide yes)
 			(show_name no)
@@
 		)
 		(property "Datasheet" "https://www.lcsc.com/datasheet/lcsc_datasheet_2309221403_Texas-Instruments-TMP117AIDRVR_C699536.pdf"
-			(at 148.59 181.61 0)
+			(at 142.24 173.99 0)
 			(hide yes)
 			(show_name no)
@@
 		)
 		(property "Description" "-55℃~+150℃ 1.7V~5.5V 15.5ms 16bit 3.1uA Factory temperature calibration、Temperature threshold monitoring、Low-power standby、On-chip non-volatile parameter storage、On-chip digital filtering/averaging I2C、SMBus ±0.1℃ WDFN-6-EP(2x2) Temperature Sensors ROHS"
-			(at 148.59 181.61 0)
+			(at 142.24 173.99 0)
 			(hide yes)
 			(show_name no)
@@
 		)
 		(property "LCSC" "C699536"
-			(at 148.59 181.61 0)
+			(at 142.24 173.99 0)
 			(hide yes)
 			(show_name no)
@@
 		)
 		(property "Manufacturer" "Texas Instruments"
-			(at 148.59 181.61 0)
+			(at 142.24 173.99 0)
 			(hide yes)
 			(show_name no)
@@
 		)
 		(property "Manufacturer Part" "TMP117AIDRVR"
-			(at 148.59 181.61 0)
+			(at 142.24 173.99 0)
 			(hide yes)
 			(show_name no)
