File: hardware/schematic/v1.0/GPSDO_Rev1.0/OCXO.kicad_sch (KiCad schematic)
At the start: 24 parts, among them U2 LMK1C1103PWR, U3 TMP117AIDRVR, U5 OCXO_20x20mm, U7 OCXO_25.4x25.4mm, U8 REF5040

Commit message: sch update
Parts:
- added C16: 100nF, GPSDO_Rev1.0:C_0402_1005Metric, symbol GPSDO_Rev1.0:C
- added FB3: 100R, GPSDO_Rev1.0:L_0603_1608Metric, symbol GPSDO_Rev1.0:FerriteBead_Small
- added R12, R15, R16: 4K7, GPSDO_Rev1.0:R_0402_1005Metric, symbol GPSDO_Rev1.0:R
Connections:
- net +3.3V: now also U3.5 (V+), C16.1, FB3.2, R12.1, R15.1, R16.1; no longer C3.1, C4.1, U2.2 (1G), U2.6 (VDD)
- net GND: now also U3.4 (ADD0), U3.7 (EP), C16.2
- net TMP_SCL: now reaches U3.1 (SCL)
- net TMP_SCL: now also R16.2
- net at U3.3 (ALERT): now also R15.2
- net TMP_SDA: now reaches U3.6 (SDA)
- net TMP_SDA: now also R12.2
- new net: C3.1, C4.1, FB3.1, U2.2 (1G), U2.6 (VDD)
Other:
- note added: "Temperature Sensor"
- moved on the sheet: R4, R5, U3, U5

Commit message: sch update
Parts:
- added FB4, FB5: 100R, GPSDO_Rev1.0:L_0603_1608Metric, symbol GPSDO_Rev1.0:FerriteBead_Small
Connections:
- net OCXO_VCC: now also FB4.1, FB4.2, FB5.1, FB5.2

Commit message: sch update
Parts:
- removed R13: 1K, Resistor_SMD:R_0402_1005Metric, symbol Device:R
- added C17: 1uF, GPSDO_Rev1.0:C_0603_1608Metric, symbol GPSDO_Rev1.0:C
- added C18: 100nF, GPSDO_Rev1.0:C_0402_1005Metric, symbol GPSDO_Rev1.0:C
- added FB7: 600R, GPSDO_Rev1.0:L_0603_1608Metric, symbol GPSDO_Rev1.0:FerriteBead_Small
- added R13: 1K, GPSDO_Rev1.0:R_0402_1005Metric, symbol GPSDO_Rev1.0:R
- added U10: OPA189IDR, GPSDO_Rev1.0:OPA189IDR, symbol GPSDO_Rev1.0:OPA189IDR
Connections:
- net GND: now also C17.2, C18.2, U10.4 (V-)
- net OCXO_MON: now also R13.1
- net OCXO_OUT: now also R13.2
- new net: C17.1, C18.1, FB7.1, U10.7 (V+)
- new net +5V: FB7.2
- no-connect marks 7 -> 10
Other:
- moved on the sheet: C3, C4, FB3, R6, R7, TP2, U2

Commit message: sch update
Parts:
- added C19: 10uF, GPSDO_Rev1.0:C_0603_1608Metric, symbol GPSDO_Rev1.0:C
- added C20: 1uF, GPSDO_Rev1.0:C_0603_1608Metric, symbol GPSDO_Rev1.0:C
- added C21: 2.2uF, GPSDO_Rev1.0:C_0603_1608Metric, symbol GPSDO_Rev1.0:C
- added R17: 100R, GPSDO_Rev1.0:R_0603_1608Metric, symbol GPSDO_Rev1.0:R
- added R18: 15K, GPSDO_Rev1.0:R_0603_1608Metric, symbol GPSDO_Rev1.0:R
- added R19: 8.2K, GPSDO_Rev1.0:R_0603_1608Metric, symbol GPSDO_Rev1.0:R
Connections:
- net GND: now also C19.2, C20.2
- net VCTRL: now also C19.1, R17.2
- net at U10.2 (-IN): now also U10.6 (OUT), C21.2, R17.1
- net at U10.3 (+IN): now also C20.1, R18.2
- new net: C21.1, R18.1, R19.2
- new net PWM: R19.1
Other:
- note added: "Active Low-pass Filter for Tuning Voltage"
- note added: "Passive LPF to compensate attenuation reversal of active LPF."
- moved on the sheet: C17, C18, FB7, U10

Commit message: sch update
Changed lines of the file:
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@@
 	(text "Passive LPF to compensate\nattenuation reversal of \nactive LPF."
 		(exclude_from_sim no)
-		(at 128.27 166.116 0)
+		(at 128.524 164.846 0)
 		(effects
 			(font
@@
 	(polyline
 		(pts
-			(xy 127 161.29) (xy 127 194.31)
+			(xy 127 160.02) (xy 127 194.31)
 		)
 		(stroke
@@
 	(polyline
 		(pts
-			(xy 46.99 161.29) (xy 46.99 194.31)
+			(xy 46.99 160.02) (xy 46.99 194.31)
 		)
 		(stroke
@@
 	(polyline
 		(pts
-			(xy 46.99 161.29) (xy 127 161.29)
+			(xy 46.99 160.02) (xy 127 160.02)
 		)
 		(stroke
@@
 	(polyline
 		(pts
-			(xy 127 161.29) (xy 160.02 161.29)
-		)
-		(stroke
+			(xy 127 160.02) (xy 160.02 160.02)
+		)
+		(stroke

Commit message: sch update
Changed lines of the file:
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@@
 	(wire
 		(pts
-			(xy 158.75 50.8) (xy 161.29 50.8)
+			(xy 158.75 50.8) (xy 168.91 50.8)
 		)
 		(stroke
@@
 	(label "VCTRL"
 		(at 91.44 119.38 0)
+		(effects
+			(font
+				(size 1.27 1.27)
+			)
+			(justify left bottom)
+		)
+	)
+	(label "VCTRL"
+		(at 162.56 50.8 0)
 		(effects
 			(font
@@
 			)
 		)
-	)
-	(global_label "VCTRL"
-		(shape input)
-		(at 161.29 50.8 0)
-		(fields_autoplaced yes)
-		(effects
-			(font
-				(size 1.27 1.27)
-			)
-			(justify left)
-		)
-		(property "Intersheetrefs" "${INTERSHEET_REFS}"
-			(at 169.8995 50.8 0)
-			(hide yes)
-			(show_name no)
-			(do_not_autoplace no)
-			(effects
-				(font
-					(size 1.27 1.27)
-				)
-				(justify left)
-			)
-		)

Commit message: sch update
Connections:
- net +5V: now also R28.2
- net OCXO_VCC: no longer R28.2
Changed lines of the file:
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@@
 		)
 	)
-	(hierarchical_label "OCXO_VCC"
-		(shape bidirectional)
-		(at 198.12 34.29 90)
-		(effects
-			(font
-				(size 1.27 1.27)
-			)
-			(justify left)
-		)
-	)
 	(hierarchical_label "PWM"
 		(shape input)
@@
 					(unit 1)
 				)
+			)
+		)
+	)
+	(symbol
+		(lib_id "power:+5V")
+		(at 198.12 34.29 0)
+		(unit 1)
+		(body_style 1)
+		(exclude_from_sim no)
+		(in_bom yes)
+		(on_board yes)
+		(in_pos_files yes)
+		(dnp no)
+		(fields_autoplaced yes)
+		(property "Reference" "#PWR043"
+			(at 198.12 38.1 0)
+			(hide yes)
+			(show_name no)
+			(do_not_autoplace no)
+			(effects
+				(font
+					(size 1.27 1.27)
+				)
+			)
+		)
+		(property "Value" "+5V"
+			(at 198.12 29.21 0)
+			(show_name no)
+			(do_not_autoplace no)
+			(effects
+				(font
+					(size 1.27 1.27)
+				)
+			)
+		)
+		(property "Footprint" ""
+			(at 198.12 34.29 0)
+			(hide yes)
+			(show_name no)
+			(do_not_autoplace no)
+			(effects
+				(font
+					(size 1.27 1.27)
+				)
+			)
+		)
+		(property "Datasheet" ""
+			(at 198.12 34.29 0)
+			(hide yes)
+			(show_name no)
+			(do_not_autoplace no)
+			(effects
+				(font
+					(size 1.27 1.27)
+				)
+			)
+		)
+		(property "Description" "Power symbol creates a global label with name \"+5V\""
+			(at 198.12 34.29 0)
+			(hide yes)
+			(show_name no)
+			(do_not_autoplace no)
+			(effects
+				(font
+					(size 1.27 1.27)
+				)
+			)
+		)
+		(pin "1"
+		)
+		(instances
+			(project "GPSDO_Rev1.0"
+				(path "/7fcb1340-2836-48b1-8b47-374fa7e6ca96/40d668d4-3bfe-4d48-b2dd-b6741ecb73a3"
+					(reference "#PWR043")
+					(unit 1)
+				)

Commit message: sch update
Connections:
- net OCXO_OUT renamed OCXO_RF
Changed lines of the file:
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@@
 		)
 	)
-	(global_label "OCXO_OUT"
+	(global_label "OCXO_RF"
 		(shape input)
 		(at 92.71 101.6 90)
@@
 		)
 		(property "Intersheetrefs" "${INTERSHEET_REFS}"
-			(at 92.71 96.2562 90)
+			(at 92.71 90.1481 90)
 			(hide yes)
 			(show_name no)
@@
 		)
 	)
-	(global_label "OCXO_OUT"
+	(global_label "OCXO_RF"
 		(shape output)
 		(at 130.81 55.88 270)
@@
 		)
 		(property "Intersheetrefs" "${INTERSHEET_REFS}"
-			(at 130.81 68.6019 90)
+			(at 130.81 67.3319 90)
 			(hide yes)
 			(show_name no)
