File: hardware/schematic/v1.0/GPSDO_Rev1.0/OCXO.kicad_sch (KiCad schematic)
At the start: 41 parts, among them U10 OPA189IDR, U2 LMK1C1103PWR, U3 TMP117AIDRVR, U5 OCXO_20x20mm, U7 OCXO_25.4x25.4mm, U8 REF5040

Commit message: sch update
Parts:
- removed U10: OPA189IDR, GPSDO_Rev1.0:OPA189IDR, symbol GPSDO_Rev1.0:OPA189IDR
- added U9: OPA388IDR, GPSDO_Rev1.0:OPA388IDR, symbol GPSDO_Rev1.0:OPA388IDR
Connections:
- net GND: now also U9.4 (V-)
- net at C21.2, R17.1: now also U9.2 (-IN), U9.6 (OUT)
- net at C20.1, R18.2: now also U9.3 (+IN)
- net at C17.1, C18.1, FB7.1: now also U9.7 (V+)
Changed lines of the file:
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@@
 	)
 	(symbol
+		(lib_id "GPSDO_Rev1.0:OPA388IDR")
+		(at 102.87 172.72 0)
+		(unit 1)
+		(body_style 1)
+		(exclude_from_sim no)
+		(in_bom yes)
+		(on_board yes)
+		(in_pos_files yes)
+		(dnp no)
+		(property "Reference" "U9"
+			(at 102.616 180.594 0)
+			(show_name no)
+			(do_not_autoplace no)
+			(effects
+				(font
+					(size 1.27 1.27)
+				)
+			)
+		)
+		(property "Value" "OPA388IDR"
+			(at 102.616 183.134 0)
+			(show_name no)
+			(do_not_autoplace no)
+			(effects
+				(font
+					(size 1.27 1.27)
+				)
+			)
+		)
+		(property "Footprint" "GPSDO_Rev1.0:OPA388IDR"
+			(at 102.87 172.72 0)
+			(hide yes)
+			(show_name no)
+			(do_not_autoplace no)
+			(effects
+				(font
+					(size 1.27 1.27)
+				)
+			)
+		)
+		(property "Datasheet" "https://www.lcsc.com/datasheet/lcsc_datasheet_1809141431_Texas-Instruments-OPA388IDR_C154118.pdf"
+			(at 102.87 172.72 0)
+			(hide yes)
+			(show_name no)
+			(do_not_autoplace no)
+			(effects
+				(font
+					(size 1.27 1.27)
+				)
+			)
+		)
+		(property "Description" "-2.75V~-1.25V、1.25V~2.75V -40℃~+125℃ 1 10MHz 140dB 2.4mA 2.5V~5.5V 250nV 30pA 5V/us 5nV/℃ 60mA 60pA 7nV/√Hz@1kHz EMI filtering/RF suppression、Zero drift / auto-zero、Built-in compensation Rail-to-Rail Input, Rail-to-Rail Output SOIC-8 Precision Op Amps ROHS"
+			(at 102.87 172.72 0)
+			(hide yes)
+			(show_name no)
+			(do_not_autoplace no)
+			(effects
+				(font
+					(size 1.27 1.27)
+				)
+			)
+		)
+		(property "LCSC" "C154118"
+			(at 102.87 172.72 0)
+			(hide yes)
+			(show_name no)
+			(do_not_autoplace no)
+			(effects
+				(font
+					(size 1.27 1.27)
+				)
+			)
+		)
+		(property "Manufacturer" "Texas Instruments"
+			(at 102.87 172.72 0)
+			(hide yes)
+			(show_name no)
+			(do_not_autoplace no)
+			(effects
+				(font
+					(size 1.27 1.27)
+				)
+			)
+		)
+		(property "Manufacturer Part" "OPA388IDR"
+			(at 102.87 172.72 0)
+			(hide yes)
+			(show_name no)
+			(do_not_autoplace no)
+			(effects
+				(font
+					(size 1.27 1.27)
+				)
+			)
+		)
+		(pin "4"
+		)
+		(pin "2"
+		)
+		(pin "5"
+		)
+		(pin "7"
+		)
+		(pin "1"
+		)
+		(pin "8"
+		)
+		(pin "6"
+		)
+		(pin "3"
+		)
+		(instances
+			(project "GPSDO_Rev1.0"
+				(path "/7fcb1340-2836-48b1-8b47-374fa7e6ca96/40d668d4-3bfe-4d48-b2dd-b6741ecb73a3"
+					(reference "U9")
+					(unit 1)
+				)
+			)
+		)
+	)
+	(symbol
 		(lib_id "GPSDO_Rev1.0:R")
 		(at 73.66 173.99 90)
@@
 					(unit 1)
 				)
-			)
-		)
-	)
-	(symbol
-		(lib_id "GPSDO_Rev1.0:OPA189IDR")
-		(at 102.87 172.72 0)
-		(unit 1)
-		(body_style 1)
-		(exclude_from_sim no)
-		(in_bom yes)
-		(on_board yes)
-		(in_pos_files yes)
-		(dnp no)
-		(property "Reference" "U10"
-			(at 102.87 164.592 0)
-			(show_name no)
-			(do_not_autoplace no)
-			(effects
-				(font
-					(size 1.27 1.27)
-				)
-			)
-		)
-		(property "Value" "OPA189IDR"
-			(at 102.87 182.118 0)
-			(show_name no)
-			(do_not_autoplace no)
-			(effects
-				(font
-					(size 1.27 1.27)
-				)
-			)
-		)
-		(property "Footprint" "GPSDO_Rev1.0:OPA189IDR"
-			(at 102.87 172.72 0)
-			(hide yes)
-			(show_name no)
-			(do_not_autoplace no)
-			(effects
-				(font
-					(size 1.27 1.27)
-				)
-			)
-		)
-		(property "Datasheet" "https://www.lcsc.com/datasheet/lcsc_datasheet_2304140030_Texas-Instruments-OPA189IDR_C781811.pdf"
-			(at 102.87 172.72 0)
-			(hide yes)
-			(show_name no)
-			(do_not_autoplace no)
-			(effects
-				(font
-					(size 1.27 1.27)
-				)
-			)
-		)
-		(property "Description" "-18V~-2.25V、2.25V~18V -40℃~+125℃ 1 1.7mA 140pA 14MHz 168dB 20V/us 3uV 4.5V~36V 5.2nV/√Hz@1kHz 5nV/℃ 65mA 70pA EMI filtering/RF suppression、Zero drift / auto-zero、ESD protection、Reverse-phase input protection Rail-to-rail output SOP-8 Precision Op Amps ROHS"
-			(at 102.87 172.72 0)
-			(hide yes)
-			(show_name no)
-			(do_not_autoplace no)
-			(effects
-				(font
-					(size 1.27 1.27)
-				)
-			)
-		)
-		(property "LCSC" "C781811"
-			(at 102.87 172.72 0)
-			(hide yes)
-			(show_name no)
-			(do_not_autoplace no)
-			(effects
-				(font
-					(size 1.27 1.27)
-				)
-			)
-		)
-		(property "Manufacturer" "Texas Instruments"
-			(at 102.87 172.72 0)
-			(hide yes)
-			(show_name no)
-			(do_not_autoplace no)
-			(effects
-				(font
-					(size 1.27 1.27)
-				)
-			)
-		)
-		(property "Manufacturer Part" "OPA189IDR"
-			(at 102.87 172.72 0)
-			(hide yes)
-			(show_name no)
-			(do_not_autoplace no)
-			(effects
-				(font
-					(size 1.27 1.27)
-				)
-			)
-		)
-		(pin "1"
-		)
-		(pin "2"
-		)
-		(pin "8"
-		)
-		(pin "4"
-		)
-		(pin "3"
-		)
-		(pin "7"
-		)
-		(pin "5"
-		)
-		(pin "6"
-		)
-		(instances
-			(project "GPSDO_Rev1.0"
-				(path "/7fcb1340-2836-48b1-8b47-374fa7e6ca96/40d668d4-3bfe-4d48-b2dd-b6741ecb73a3"
-					(reference "U10")
-					(unit 1)
-				)

Commit message: pdf and sch update
Parts:
- added C22, C24: 100nF, GPSDO_Rev1.0:C_0402_1005Metric, symbol GPSDO_Rev1.0:C
- added R35: 100K, GPSDO_Rev1.0:R_0402_1005Metric, symbol GPSDO_Rev1.0:R
- added U10: SN74LVC1T45DBVR, GPSDO_Rev1.0:SN74LVC1T45DBVR, symbol GPSDO_Rev1.0:SN74LVC1T45DBVR
Connections:
- net +3.3V: now also C22.1, U10.1 (VCCA), U10.5 (DIR)
- net GND: now also C22.2, C24.2, R35.2, U10.2 (GND)
- net PWM: now also R35.1, U10.3 (A); no longer R19.1
- net VREF: now also C24.1, U10.6 (VCCB)
- new net: R19.1, U10.4 (B)
Other:
- moved on the sheet: C17, C18, C19, C20, C21, FB7, R17, R18, R19, U9

Commit message: sch update
Parts:
- added R36: 0, GPSDO_Rev1.0:R_0603_1608Metric, symbol GPSDO_Rev1.0:R
- added R37: 0, GPSDO_Rev1.0:R_0402_1005Metric, symbol GPSDO_Rev1.0:R
Connections:
- net GND: now also R37.2
- net OCXO_RF: now also R36.2; no longer U2.1 (CLKIN)
- new net OCXO_OUT: R36.1, R37.1, U2.1 (CLKIN)

Commit message: sch update
Parts:
- C1, C16, C18, C22, C24, C4, C5: symbol GPSDO_Rev1.0:C -> GPSDO_Rev1.0:C__C_0402_1005Metric
- C11: footprint Capacitor_SMD:C_0402_1005Metric -> GPSDO_Rev1.0:C_0402_1005Metric; symbol Device:C -> GPSDO_Rev1.0:C__C_0402_1005Metric
- C56, C57, C58: footprint Capacitor_SMD:C_0603_1608Metric -> GPSDO_Rev1.0:C_0603_1608Metric; symbol Device:C -> GPSDO_Rev1.0:C
- R12, R13, R15, R16, R35, R37, R4: symbol GPSDO_Rev1.0:R -> GPSDO_Rev1.0:R__R_0402_1005Metric
- R28, R29: footprint Resistor_SMD:R_0603_1608Metric -> GPSDO_Rev1.0:R_0603_1608Metric; symbol Device:R -> GPSDO_Rev1.0:R
- R5: symbol GPSDO_Rev1.0:R -> GPSDO_Rev1.0:R__R_0805_2012Metric
- R6: symbol GPSDO_Rev1.0:R -> GPSDO_Rev1.0:R__C_0603_1608Metric
- TP1, TP2: footprint TestPoint:TestPoint_Pad_D1.0mm -> GPSDO_Rev1.0:TestPoint_Pad_D1.0mm; symbol Connector:TestPoint -> GPSDO_Rev1.0:TestPoint
- U8: footprint JLCImport:REF5040 -> GPSDO_Rev1.0:REF5040; symbol JLCImport:REF5040 -> GPSDO_Rev1.0:REF5040

Commit message: sch update
Connections:
- net VCTRL renamed VCTL
Changed lines of the file:
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@@
+	)
+	(junction
+		(at 246.38 35.56)
+		(diameter 0)
+		(color 0 0 0 0)
+	)
+	(junction
+		(at 78.74 111.76)
+		(diameter 0)
+		(color 0 0 0 0)
+	)
+	(junction
+		(at 67.31 111.76)
+		(diameter 0)
+		(color 0 0 0 0)
+	)
+	(junction
+		(at 205.74 44.45)
+		(diameter 0)
+		(color 0 0 0 0)
+	)
+	(junction
+		(at 72.39 173.99)
+		(diameter 0)
+		(color 0 0 0 0)
+	)
+	(junction
+		(at 120.65 173.99)
+		(diameter 0)
+		(color 0 0 0 0)
+	)
+	(junction
+		(at 201.93 57.15)
+		(diameter 0)
+		(color 0 0 0 0)
+	)
+	(junction
+		(at 83.82 50.8)
+		(diameter 0)
+		(color 0 0 0 0)
+	)
+	(junction
+		(at 142.24 111.76)
+		(diameter 0)
+		(color 0 0 0 0)
+	)
+	(junction
+		(at 92.71 111.76)
+		(diameter 0)
+		(color 0 0 0 0)
+	)
+	(junction
+		(at 165.1 173.99)
+		(diameter 0)
+		(color 0 0 0 0)
+	)
+	(junction
+		(at 87.63 173.99)
+		(diameter 0)
+		(color 0 0 0 0)
+	)
+	(junction
+		(at 110.49 152.4)
+		(diameter 0)
+		(color 0 0 0 0)
+	)
+	(junction
+		(at 246.38 46.99)
+		(diameter 0)
+		(color 0 0 0 0)
+	)
+	(junction
+		(at 46.99 50.8)
+		(diameter 0)
+		(color 0 0 0 0)
+	)
+	(junction
+		(at 138.43 102.87)
+		(diameter 0)
+		(color 0 0 0 0)
+	)
+	(junction
+		(at 129.54 111.76)
+		(diameter 0)
+		(color 0 0 0 0)
+	)
+	(junction
+		(at 157.48 97.79)
+		(diameter 0)
+		(color 0 0 0 0)
+	)
+	(junction
+		(at 134.62 111.76)
+		(diameter 0)
+		(color 0 0 0 0)
+	)
+	(junction
+		(at 125.73 173.99)
+		(diameter 0)
+		(color 0 0 0 0)
+	)
+	(junction
+		(at 198.12 44.45)
+		(diameter 0)
+		(color 0 0 0 0)
+	)
+	(junction
+		(at 25.4 173.99)
+		(diameter 0)
+		(color 0 0 0 0)
+	)
+	(junction
+		(at 157.48 106.68)
+		(diameter 0)
+		(color 0 0 0 0)
+	)
+	(junction
+		(at 49.53 151.13)
+		(diameter 0)
+		(color 0 0 0 0)
+	)
+	(junction
+		(at 205.74 57.15)
+		(diameter 0)
+		(color 0 0 0 0)
 	)
 	(junction
 		(at 147.32 173.99)
-		(diameter 0)
-		(color 0 0 0 0)
-	)
-	(junction
-		(at 246.38 35.56)
-		(diameter 0)
-		(color 0 0 0 0)
-	)
-	(junction
-		(at 78.74 111.76)
-		(diameter 0)
-		(color 0 0 0 0)
-	)
-	(junction
-		(at 67.31 111.76)
-		(diameter 0)
-		(color 0 0 0 0)
-	)
-	(junction
-		(at 205.74 44.45)
-		(diameter 0)
-		(color 0 0 0 0)
-	)
-	(junction
-		(at 72.39 173.99)
-		(diameter 0)
-		(color 0 0 0 0)
-	)
-	(junction
-		(at 120.65 173.99)
-		(diameter 0)
-		(color 0 0 0 0)
-	)
-	(junction
-		(at 201.93 57.15)
-		(diameter 0)
-		(color 0 0 0 0)
-	)
-	(junction
-		(at 83.82 50.8)
-		(diameter 0)
-		(color 0 0 0 0)
-	)
-	(junction
-		(at 142.24 111.76)
-		(diameter 0)
-		(color 0 0 0 0)
-	)
-	(junction
-		(at 92.71 111.76)
-		(diameter 0)
-		(color 0 0 0 0)
-	)
-	(junction
-		(at 87.63 173.99)
-		(diameter 0)
-		(color 0 0 0 0)
-	)
-	(junction
-		(at 110.49 152.4)
-		(diameter 0)
-		(color 0 0 0 0)
-	)
-	(junction
-		(at 246.38 46.99)
-		(diameter 0)
-		(color 0 0 0 0)
-	)
-	(junction
-		(at 46.99 50.8)
-		(diameter 0)
-		(color 0 0 0 0)
-	)
-	(junction
-		(at 138.43 102.87)
-		(diameter 0)
-		(color 0 0 0 0)
-	)
-	(junction
-		(at 129.54 111.76)
-		(diameter 0)
-		(color 0 0 0 0)
-	)
-	(junction
-		(at 157.48 97.79)
-		(diameter 0)
-		(color 0 0 0 0)
-	)
-	(junction
-		(at 134.62 111.76)
-		(diameter 0)
-		(color 0 0 0 0)
-	)
-	(junction
-		(at 125.73 173.99)
-		(diameter 0)
-		(color 0 0 0 0)
-	)
-	(junction
-		(at 198.12 44.45)
-		(diameter 0)
-		(color 0 0 0 0)
-	)
-	(junction
-		(at 25.4 173.99)
-		(diameter 0)
-		(color 0 0 0 0)
-	)
-	(junction
-		(at 157.48 106.68)
-		(diameter 0)
-		(color 0 0 0 0)
-	)
-	(junction
-		(at 49.53 151.13)
-		(diameter 0)
-		(color 0 0 0 0)
-	)
-	(junction
-		(at 205.74 57.15)
 		(diameter 0)
 		(color 0 0 0 0)
@@
 		)
 	)
-	(polyline
-		(pts
-			(xy 132.08 194.31) (xy 165.1 194.31)
+	(wire
+		(pts
+			(xy 165.1 166.37) (xy 165.1 173.99)
+		)
+		(stroke
+			(width 0)
+			(type default)
+		)
+	)
+	(polyline
+		(pts
+			(xy 132.08 194.31) (xy 161.29 194.31)
 		)
 		(stroke
@@
 	(wire
 		(pts
+			(xy 165.1 173.99) (xy 167.64 173.99)
+		)
+		(stroke
+			(width 0)
+			(type default)
+		)
+	)
+	(wire
+		(pts
 			(xy 201.93 116.84) (xy 219.71 116.84)
 		)
@@
 	(polyline
 		(pts
-			(xy 132.08 160.02) (xy 165.1 160.02)
+			(xy 132.08 160.02) (xy 161.29 160.02)
 		)
 		(stroke
@@
 	(polyline
 		(pts
-			(xy 165.1 161.29) (xy 165.1 194.31)
+			(xy 161.29 160.02) (xy 161.29 194.31)
 		)
 		(stroke
@@
 	(wire
 		(pts
-			(xy 147.32 173.99) (xy 166.37 173.99)
+			(xy 147.32 173.99) (xy 165.1 173.99)
 		)
 		(stroke
@@
 	)
 	(label "VCTRL"
-		(at 166.37 173.99 0)
+		(at 167.64 173.99 0)
 		(effects
 			(font
@@
 		(effects
 			(font
+				(size 1.27 1.27)
+			)
+			(justify left)
+		)
+	)
+	(hierarchical_label "VCTL"
+		(shape output)
+		(at 165.1 166.37 90)
+		(effects
+			(font

Commit message: sch update
Parts:
- added C26: 100nF, GPSDO_Rev1.0:C_0402_1005Metric, symbol GPSDO_Rev1.0:C__C_0402_1005Metric
- added R39, R40: 100K, GPSDO_Rev1.0:R_0402_1005Metric, symbol GPSDO_Rev1.0:R__R_0402_1005Metric
- added R41: 1K, GPSDO_Rev1.0:R_0402_1005Metric, symbol GPSDO_Rev1.0:R__R_0402_1005Metric
Connections:
- net GND: now also C26.2, R40.1
- net VCTL: now also C26.1, R41.1; no longer C19.1, R17.2, U5.4 (VCTRL/NC), U7.3 (VCTRL)
- new net: R39.1, R40.2, R41.2
- new net VCTRL: C19.1, R17.2, R39.2, U5.4 (VCTRL/NC), U7.3 (VCTRL)

Commit message: sch update
Connections:
- net GND: now also U3.2 (GND)
Changed lines of the file:
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@@
 		)
 	)
-	(hierarchical_label "OCXO_VCC"
-		(shape bidirectional)
-		(at 157.48 96.52 90)
-		(effects
-			(font
-				(size 1.27 1.27)
-			)
-			(justify left)
-		)
-	)
 	(hierarchical_label "VCTL"
 		(shape output)
@@
 	)
 	(symbol
+		(lib_id "GPSDO_Rev1.0:GND")
+		(at 49.53 53.34 270)
+		(unit 1)
+		(body_style 1)
+		(exclude_from_sim no)
+		(in_bom yes)
+		(on_board yes)
+		(in_pos_files yes)
+		(dnp no)
+		(fields_autoplaced yes)
+		(property "Reference" "#PWR046"
+			(at 43.18 53.34 0)
+			(hide yes)
+			(show_name no)
+			(do_not_autoplace no)
+			(effects
+				(font
+					(size 1.27 1.27)
+				)
+			)
+		)
+		(property "Value" "GND"
+			(at 44.45 53.34 0)
+			(hide yes)
+			(show_name no)
+			(do_not_autoplace no)
+			(effects
+				(font
+					(size 1.27 1.27)
+				)
+			)
+		)
+		(property "Footprint" ""
+			(at 49.53 53.34 0)
+			(hide yes)
+			(show_name no)
+			(do_not_autoplace no)
+			(effects
+				(font
+					(size 1.27 1.27)
+				)
+			)
+		)
+		(property "Datasheet" ""
+			(at 49.53 53.34 0)
+			(hide yes)
+			(show_name no)
+			(do_not_autoplace no)
+			(effects
+				(font
+					(size 1.27 1.27)
+				)
+			)
+		)
+		(property "Description" "Power symbol creates a global label with name \"GND\" , ground"
+			(at 49.53 53.34 0)
+			(hide yes)
+			(show_name no)
+			(do_not_autoplace no)
+			(effects
+				(font
+					(size 1.27 1.27)
+				)
+			)
+		)
+		(pin "1"
+		)
+		(instances
+			(project "GPSDO_Rev1.0"
+				(path "/7fcb1340-2836-48b1-8b47-374fa7e6ca96/40d668d4-3bfe-4d48-b2dd-b6741ecb73a3"
+					(reference "#PWR046")
+					(unit 1)
+				)
+			)
+		)
+	)
+	(symbol
 		(lib_id "GPSDO_Rev1.0:C__C_0402_1005Metric")
 		(at 119.38 156.21 0)
@@
 					(unit 1)
 				)
+			)
+		)
+	)
+	(symbol
+		(lib_id "GPSDO_Rev1.0:VDDA")
+		(at 157.48 96.52 0)
+		(unit 1)
+		(body_style 1)
+		(exclude_from_sim no)
+		(in_bom yes)
+		(on_board yes)
+		(in_pos_files yes)
+		(dnp no)
+		(fields_autoplaced yes)
+		(property "Reference" "#PWR056"
+			(at 157.48 100.33 0)
+			(hide yes)
+			(show_name no)
+			(do_not_autoplace no)
+			(effects
+				(font
+					(size 1.27 1.27)
+				)
+			)
+		)
+		(property "Value" "OCXO_VCC"
+			(at 157.48 91.44 0)
+			(show_name no)
+			(do_not_autoplace no)
+			(effects
+				(font
+					(size 1.27 1.27)
+				)
+			)
+		)
+		(property "Footprint" ""
+			(at 157.48 96.52 0)
+			(hide yes)
+			(show_name no)
+			(do_not_autoplace no)
+			(effects
+				(font
+					(size 1.27 1.27)
+				)
+			)
+		)
+		(property "Datasheet" ""
+			(at 157.48 96.52 0)
+			(hide yes)
+			(show_name no)
+			(do_not_autoplace no)
+			(effects
+				(font
+					(size 1.27 1.27)
+				)
+			)
+		)
+		(property "Description" "Power symbol creates a global label with name \"VDDA\""
+			(at 157.48 96.52 0)
+			(hide yes)
+			(show_name no)
+			(do_not_autoplace no)
+			(effects
+				(font
+					(size 1.27 1.27)
+				)
+			)
+		)
+		(pin "1"
+		)
+		(instances
+			(project "GPSDO_Rev1.0"
+				(path "/7fcb1340-2836-48b1-8b47-374fa7e6ca96/40d668d4-3bfe-4d48-b2dd-b6741ecb73a3"
+					(reference "#PWR056")
+					(unit 1)
+				)
