File: hardware/schematic/v1.0/GPSDO_Rev1.0/EXT.kicad_sch (KiCad schematic)
At the start: 1 part, among them U4 BUF602IDBVT

Commit message: sch update
Parts:
- added C30: 100nF, GPSDO_Rev1.0:C_0402_1005Metric, symbol GPSDO_Rev1.0:C
- added C31: 4.7uF, GPSDO_Rev1.0:C_0603_1608Metric, symbol GPSDO_Rev1.0:C
Connections:
- net GND: now reaches U4.2 (−VCC)
- net GND: now also C30.2, C31.2
- net 10MHZ_OUT: now reaches U4.4 (In)
- net +5V: now reaches U4.5 (+VCC)
- net +5V: now also C30.1, C31.1
- no-connect marks 0 -> 1

Commit message: sch update
Parts:
- added J1: Conn_Coaxial, Connector_Coaxial:SMA_Amphenol_132134-11_Vertical, symbol Connector:Conn_Coaxial
Connections:
- net GND: now also J1.2 (Ext)
Changed lines of the file:
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@@
+	)
+	(symbol
+		(lib_id "Connector:Conn_Coaxial")
+		(at 119.38 78.74 0)
+		(unit 1)
+		(body_style 1)
+		(exclude_from_sim no)
+		(in_bom yes)
+		(on_board yes)
+		(in_pos_files yes)
+		(dnp no)
+		(property "Reference" "J1"
+			(at 120.396 70.866 0)
+			(show_name no)
+			(do_not_autoplace no)
+			(effects
+				(font
+					(size 1.27 1.27)
+				)
+				(justify right)
+			)
+		)
+		(property "Value" "Conn_Coaxial"
+			(at 125.984 73.914 0)
+			(show_name no)
+			(do_not_autoplace no)
+			(effects
+				(font
+					(size 1.27 1.27)
+				)
+				(justify right)
+			)
+		)
+		(property "Footprint" "Connector_Coaxial:SMA_Amphenol_132134-11_Vertical"
+			(at 119.38 78.74 0)
+			(hide yes)
+			(show_name no)
+			(do_not_autoplace no)
+			(effects
+				(font
+					(size 1.27 1.27)
+				)
+			)
+		)
+		(property "Datasheet" ""
+			(at 119.38 78.74 0)
+			(hide yes)
+			(show_name no)
+			(do_not_autoplace no)
+			(effects
+				(font
+					(size 1.27 1.27)
+				)
+			)
+		)
+		(property "Description" "coaxial connector (BNC, SMA, SMB, SMC, Cinch/RCA, LEMO, ...)"
+			(at 119.38 78.74 0)
+			(hide yes)
+			(show_name no)
+			(do_not_autoplace no)
+			(effects
+				(font
+					(size 1.27 1.27)
+				)
+			)
+		)
+		(pin "1"
+		)
+		(pin "2"
+		)
+		(instances
+			(project "GPSDO_Rev1.0"
+				(path "/7fcb1340-2836-48b1-8b47-374fa7e6ca96/1e6d2fc9-653e-45d2-a1bc-ab2903490aa7"
+					(reference "J1")
+					(unit 1)
+				)
+			)
+		)
 	)
 	(symbol
@@
 					(unit 1)
 				)
+			)
+		)
+	)
+	(symbol
+		(lib_id "power:GND")
+		(at 119.38 83.82 0)
+		(unit 1)
+		(body_style 1)
+		(exclude_from_sim no)
+		(in_bom yes)
+		(on_board yes)
+		(in_pos_files yes)
+		(dnp no)
+		(property "Reference" "#PWR0163"
+			(at 119.38 90.17 0)
+			(hide yes)
+			(show_name no)
+			(do_not_autoplace no)
+			(effects
+				(font
+					(size 1.27 1.27)
+				)
+			)
+		)
+		(property "Value" "GND"
+			(at 119.38 86.868 90)
+			(hide yes)
+			(show_name no)
+			(do_not_autoplace no)
+			(effects
+				(font
+					(size 1.27 1.27)
+				)
+				(justify right)
+			)
+		)
+		(property "Footprint" ""
+			(at 119.38 83.82 0)
+			(hide yes)
+			(show_name no)
+			(do_not_autoplace no)
+			(effects
+				(font
+					(size 1.27 1.27)
+				)
+			)
+		)
+		(property "Datasheet" ""
+			(at 119.38 83.82 0)
+			(hide yes)
+			(show_name no)
+			(do_not_autoplace no)
+			(effects
+				(font
+					(size 1.27 1.27)
+				)
+			)
+		)
+		(property "Description" "Power symbol creates a global label with name \"GND\" , ground"
+			(at 119.38 83.82 0)
+			(hide yes)
+			(show_name no)
+			(do_not_autoplace no)
+			(effects
+				(font
+					(size 1.27 1.27)
+				)
+			)
+		)
+		(pin "1"
+		)
+		(instances
+			(project "GPSDO_Rev1.0"
+				(path "/7fcb1340-2836-48b1-8b47-374fa7e6ca96/1e6d2fc9-653e-45d2-a1bc-ab2903490aa7"
+					(reference "#PWR0163")
+					(unit 1)
+				)

Commit message: sch update
Parts:
- added R20: 49.9, GPSDO_Rev1.0:C_0603_1608Metric, symbol GPSDO_Rev1.0:R
- J1: footprint Connector_Coaxial:SMA_Amphenol_132134-11_Vertical -> Connector_Coaxial:SMA_Amphenol_132289_EdgeMount
Connections:
- net at J1.1 (In): now also R20.2
- net at U4.1 (Out): now also R20.1
Other:
- moved on the sheet: J1
Changed lines of the file:
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@@
+	(wire
+		(pts
+			(xy 110.49 78.74) (xy 115.57 78.74)
+		)
+		(stroke
+			(width 0)
+			(type default)
+		)
+	)
 	(wire
 		(pts
 			(xy 68.58 53.34) (xy 68.58 78.74)
+		)
+		(stroke
+			(width 0)
+			(type default)
+		)
+	)
+	(wire
+		(pts
+			(xy 95.25 78.74) (xy 102.87 78.74)
 		)
 		(stroke
@@
 	(symbol
 		(lib_id "Connector:Conn_Coaxial")
-		(at 119.38 78.74 0)
+		(at 120.65 78.74 0)
 		(unit 1)
 		(body_style 1)
@@
 		(dnp no)
 		(property "Reference" "J1"
-			(at 120.396 70.866 0)
+			(at 121.666 70.866 0)
 			(show_name no)
 			(do_not_autoplace no)
@@
 		)
 		(property "Value" "Conn_Coaxial"
-			(at 125.984 73.914 0)
+			(at 127.254 73.914 0)
 			(show_name no)
 			(do_not_autoplace no)
@@
 			)
 		)
-		(property "Footprint" "Connector_Coaxial:SMA_Amphenol_132134-11_Vertical"
-			(at 119.38 78.74 0)
-			(hide yes)
-			(show_name no)
-			(do_not_autoplace no)
-			(effects
-				(font
-					(size 1.27 1.27)
-				)
-			)
-		)
-		(property "Datasheet" ""
-			(at 119.38 78.74 0)
+		(property "Footprint" "Connector_Coaxial:SMA_Amphenol_132289_EdgeMount"
+			(at 120.65 78.74 0)
+			(hide yes)
+			(show_name no)
+			(do_not_autoplace no)
+			(effects
+				(font
+					(size 1.27 1.27)
+				)
+			)
+		)
+		(property "Datasheet" ""
+			(at 120.65 78.74 0)
 			(hide yes)
 			(show_name no)
@@
 		)
 		(property "Description" "coaxial connector (BNC, SMA, SMB, SMC, Cinch/RCA, LEMO, ...)"
-			(at 119.38 78.74 0)
+			(at 120.65 78.74 0)
 			(hide yes)
 			(show_name no)
@@
 	(symbol
 		(lib_id "power:GND")
-		(at 119.38 83.82 0)
+		(at 120.65 83.82 0)
 		(unit 1)
 		(body_style 1)
@@
 		(dnp no)
 		(property "Reference" "#PWR0163"
-			(at 119.38 90.17 0)
+			(at 120.65 90.17 0)
 			(hide yes)
 			(show_name no)
@@
 		)
 		(property "Value" "GND"
-			(at 119.38 86.868 90)
+			(at 120.65 86.868 90)
 			(hide yes)
 			(show_name no)
@@
 		)
 		(property "Footprint" ""
-			(at 119.38 83.82 0)
-			(hide yes)
-			(show_name no)
-			(do_not_autoplace no)
-			(effects
-				(font
-					(size 1.27 1.27)
-				)
-			)
-		)
-		(property "Datasheet" ""
-			(at 119.38 83.82 0)
+			(at 120.65 83.82 0)
+			(hide yes)
+			(show_name no)
+			(do_not_autoplace no)
+			(effects
+				(font
+					(size 1.27 1.27)
+				)
+			)
+		)
+		(property "Datasheet" ""
+			(at 120.65 83.82 0)
 			(hide yes)
 			(show_name no)
@@
 		)
 		(property "Description" "Power symbol creates a global label with name \"GND\" , ground"
-			(at 119.38 83.82 0)
+			(at 120.65 83.82 0)
 			(hide yes)
 			(show_name no)
@@
 					(unit 1)
 				)
+			)
+		)
+	)
+	(symbol
+		(lib_id "GPSDO_Rev1.0:R")
+		(at 106.68 78.74 90)
+		(unit 1)
+		(body_style 1)
+		(exclude_from_sim no)
+		(in_bom yes)
+		(on_board yes)
+		(in_pos_files yes)
+		(dnp no)
+		(property "Reference" "R20"
+			(at 101.6 77.47 90)
+			(show_name no)
+			(do_not_autoplace no)
+			(effects
+				(font
+					(size 1.27 1.27)
+				)
+			)
+		)
+		(property "Value" "49.9"
+			(at 112.014 77.47 90)
+			(show_name no)
+			(do_not_autoplace no)
+			(effects
+				(font
+					(size 1.27 1.27)
+				)
+			)
+		)
+		(property "Footprint" "GPSDO_Rev1.0:C_0603_1608Metric"
+			(at 106.68 80.518 90)
+			(hide yes)
+			(show_name no)
+			(do_not_autoplace no)
+			(effects
+				(font
+					(size 1.27 1.27)
+				)
+			)
+		)
+		(property "Datasheet" ""
+			(at 106.68 78.74 0)
+			(hide yes)
+			(show_name no)
+			(do_not_autoplace no)
+			(effects
+				(font
+					(size 1.27 1.27)
+				)
+			)
+		)
+		(property "Description" "Resistor"
+			(at 106.68 78.74 0)
+			(hide yes)
+			(show_name no)
+			(do_not_autoplace no)
+			(effects
+				(font
+					(size 1.27 1.27)
+				)
+			)
+		)
+		(pin "1"
+		)
+		(pin "2"
+		)
+		(instances
+			(project "GPSDO_Rev1.0"
+				(path "/7fcb1340-2836-48b1-8b47-374fa7e6ca96/1e6d2fc9-653e-45d2-a1bc-ab2903490aa7"
+					(reference "R20")
+					(unit 1)
+				)

Commit message: sch update
Other:
- note added: "10 MHz Outputs"
- note added: "Pulse Outputs"
Changed lines of the file:
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@@
 	(generator_version "10.0")
 	(paper "A4")
+	(text "10 MHz Outputs"
+		(exclude_from_sim no)
+		(at 37.846 41.656 0)
+		(effects
+			(font
+				(size 2.54 2.54)
+				(thickness 0.508)
+				(bold yes)
+			)
+			(justify left)
+		)
+	)
+	(text "Pulse Outputs"
+		(exclude_from_sim no)
+		(at 37.592 104.14 0)
+		(effects
+			(font
+				(size 2.54 2.54)
+				(thickness 0.508)
+				(bold yes)
+			)
+			(justify left)
+		)
+	)
 	(junction
 		(at 77.47 53.34)
@@
 		(at 95.25 73.66)
 	)
+	(polyline
+		(pts
+			(xy 38.1 106.68) (xy 38.1 160.02)
+		)
+		(stroke
+			(width 0)
+			(type dash)
+		)
+	)
 	(wire
 		(pts
@@
 			(width 0)
 			(type default)
+		)
+	)
+	(polyline
+		(pts
+			(xy 38.1 160.02) (xy 171.45 160.02)
+		)
+		(stroke
+			(width 0)
+			(type dash)
 		)
 	)
@@
 		)
 	)
+	(polyline
+		(pts
+			(xy 171.45 44.45) (xy 171.45 97.79)
+		)
+		(stroke
+			(width 0)
+			(type dash)
+		)
+	)
+	(polyline
+		(pts
+			(xy 38.1 44.45) (xy 171.45 44.45)
+		)
+		(stroke
+			(width 0)
+			(type dash)
+		)
+	)
+	(polyline
+		(pts
+			(xy 38.1 97.79) (xy 171.45 97.79)
+		)
+		(stroke
+			(width 0)
+			(type dash)
+		)
+	)
+	(polyline
+		(pts
+			(xy 38.1 106.68) (xy 171.45 106.68)
+		)
+		(stroke
+			(width 0)
+			(type dash)
+		)
+	)
+	(polyline
+		(pts
+			(xy 171.45 106.68) (xy 171.45 160.02)
+		)
+		(stroke
+			(width 0)
+			(type dash)
+		)
+	)
 	(wire
 		(pts
@@
 		)
 	)
+	(polyline
+		(pts
+			(xy 38.1 44.45) (xy 38.1 97.79)
+		)
+		(stroke
+			(width 0)
+			(type dash)
+		)
+	)

Commit message: sch update
Parts:
- added C44: 100nF, GPSDO_Rev1.0:C_0402_1005Metric, symbol GPSDO_Rev1.0:C
- added C45: 4.7uF, GPSDO_Rev1.0:C_0603_1608Metric, symbol GPSDO_Rev1.0:C
- added D6, D7: TPD1E10B06DPYR, GPSDO_Rev1.0:TPD1E10B06DPYR, symbol GPSDO_Rev1.0:TPD1E10B06DPYR
- added J2: Conn_Coaxial, Connector_Coaxial:SMA_Amphenol_132289_EdgeMount, symbol Connector:Conn_Coaxial
- added R34: 49.9, GPSDO_Rev1.0:C_0603_1608Metric, symbol GPSDO_Rev1.0:R
- added U12: BUF602IDBVT, GPSDO_Rev1.0:BUF602IDBVT, symbol GPSDO_Rev1.0:BUF602IDBVT
Connections:
- net +5V: now also C44.1, C45.1, U12.5 (+VCC)
- net GND: now also C44.2, C45.2, D6.2, D7.2, J2.2 (Ext), U12.2 (−VCC)
- net at J1.1 (In), R20.2: now also D6.1
- new net: R34.1, U12.1 (Out)
- new net: D7.1, J2.1 (In), R34.2
- new net PULSE_OUT: U12.4 (In)
- no-connect marks 1 -> 2
Other:
- moved on the sheet: C30, C31, J1, R20, U4

Commit message: sch update
Changed lines of the file:
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@@
-	)
-	(symbol
-		(lib_id "power:GND")
-		(at 80.01 26.67 180)
-		(unit 1)
-		(body_style 1)
-		(exclude_from_sim no)
-		(in_bom yes)
-		(on_board yes)
-		(in_pos_files yes)
-		(dnp no)
-		(property "Reference" "#PWR0168"
-			(at 80.01 20.32 0)
-			(hide yes)
-			(show_name no)
-			(do_not_autoplace no)
-			(effects
-				(font
-					(size 1.27 1.27)
-				)
-			)
-		)
-		(property "Value" "GND"
-			(at 80.01 23.622 90)
-			(hide yes)
-			(show_name no)
-			(do_not_autoplace no)
-			(effects
-				(font
-					(size 1.27 1.27)
-				)
-				(justify right)
-			)
-		)
-		(property "Footprint" ""
-			(at 80.01 26.67 0)
-			(hide yes)
-			(show_name no)
-			(do_not_autoplace no)
-			(effects
-				(font
-					(size 1.27 1.27)
-				)
-			)
-		)
-		(property "Datasheet" ""
-			(at 80.01 26.67 0)
-			(hide yes)
-			(show_name no)
-			(do_not_autoplace no)
-			(effects
-				(font
-					(size 1.27 1.27)
-				)
-			)
-		)
-		(property "Description" "Power symbol creates a global label with name \"GND\" , ground"
-			(at 80.01 26.67 0)
-			(hide yes)
-			(show_name no)
-			(do_not_autoplace no)
-			(effects
-				(font
-					(size 1.27 1.27)
-				)
-			)
-		)
-		(pin "1"
-		)
-		(instances
-			(project "GPSDO_Rev1.0"
-				(path "/7fcb1340-2836-48b1-8b47-374fa7e6ca96/1e6d2fc9-653e-45d2-a1bc-ab2903490aa7"
-					(reference "#PWR0168")
-					(unit 1)
-				)
-			)
-		)
 	)
 	(symbol

Commit message: sch update
Parts:
- added C47, C49: 100nF, GPSDO_Rev1.0:C_0402_1005Metric, symbol GPSDO_Rev1.0:C
- added C48, C50: 4.7uF, GPSDO_Rev1.0:C_0603_1608Metric, symbol GPSDO_Rev1.0:C
Connections:
- net GND: now also C47.2, C48.2, C49.2, C50.2; no longer U12.2 (−VCC), U4.2 (−VCC)
- new net -5V: C47.1, C48.1, C49.1, C50.1, U12.2 (−VCC), U4.2 (−VCC)

Commit message: sch update
Parts:
- removed C47, C49: 100nF, GPSDO_Rev1.0:C_0402_1005Metric, symbol GPSDO_Rev1.0:C
- removed C48, C50: 4.7uF, GPSDO_Rev1.0:C_0603_1608Metric, symbol GPSDO_Rev1.0:C
- C30, C44: symbol GPSDO_Rev1.0:C -> GPSDO_Rev1.0:C__C_0402_1005Metric
- J1, J2: footprint Connector_Coaxial:SMA_Amphenol_132289_EdgeMount -> GPSDO_Rev1.0:SMA_Amphenol_132289_EdgeMount; symbol Connector:Conn_Coaxial -> GPSDO_Rev1.0:Conn_Coaxial
- R20, R34: symbol GPSDO_Rev1.0:R -> GPSDO_Rev1.0:R__C_0603_1608Metric
Connections:
- net -5V: no longer names the net of U12.2 (−VCC)
- net -5V: no longer U4.2 (−VCC)
- no-connect marks 2 -> 4
Other:
- note added: "TODO: -5V source removed. U4 / U12 still use BUF602. Replace drivers or redesign supplies before operating outputs."
