File: hardware/schematic/v1.0/GPSDO_Rev1.0/EXT.kicad_sch (KiCad schematic)
At the start: 12 parts, among them J1 Conn_Coaxial, J2 Conn_Coaxial, U12 BUF602IDBVT, U4 BUF602IDBVT

Commit message: sch update
Parts:
- removed C30, C44: 100nF, GPSDO_Rev1.0:C_0402_1005Metric, symbol GPSDO_Rev1.0:C__C_0402_1005Metric
- removed C31, C45: 4.7uF, GPSDO_Rev1.0:C_0603_1608Metric, symbol GPSDO_Rev1.0:C
- removed D7: TPD1E10B06DPYR, GPSDO_Rev1.0:TPD1E10B06DPYR, symbol GPSDO_Rev1.0:TPD1E10B06DPYR
- removed J2: Conn_Coaxial, GPSDO_Rev1.0:SMA_Amphenol_132289_EdgeMount, symbol GPSDO_Rev1.0:Conn_Coaxial
- removed R34: 49.9, GPSDO_Rev1.0:C_0603_1608Metric, symbol GPSDO_Rev1.0:R__C_0603_1608Metric
- removed U12, U4: BUF602IDBVT, GPSDO_Rev1.0:BUF602IDBVT, symbol GPSDO_Rev1.0:BUF602IDBVT
- added C46, C48: 100nF, GPSDO_Rev1.0:C_0402_1005Metric, symbol GPSDO_Rev1.0:C__C_0402_1005Metric
- added C47, C49: 4.7uF, GPSDO_Rev1.0:C_0603_1608Metric, symbol GPSDO_Rev1.0:C
- added D9: TPD1E10B06DPYR, GPSDO_Rev1.0:TPD1E10B06DPYR, symbol GPSDO_Rev1.0:TPD1E10B06DPYR
- added J4: Conn_Coaxial, GPSDO_Rev1.0:SMA_Amphenol_132289_EdgeMount, symbol GPSDO_Rev1.0:Conn_Coaxial
- added R42, R46: 10K, GPSDO_Rev1.0:R_0402_1005Metric, symbol GPSDO_Rev1.0:R__R_0402_1005Metric
- added R47: 49.9, GPSDO_Rev1.0:C_0603_1608Metric, symbol GPSDO_Rev1.0:R__C_0603_1608Metric
- added U13: ISL55110IRZ-T, GPSDO_Rev1.0:ISL55110IRZ-T, symbol GPSDO_Rev1.0:ISL55110IRZ-T
Connections:
- net +5V: now also C48.1, C49.1, U13.10 (VH)
- net 10MHZ_OUT: now also R42.1, U13.5 (IN-A)
- net GND: now also C46.2, C47.2, C48.2, C49.2, D9.2, J4.2 (Ext), R42.2, R46.1, U13.11 (GND), U13.17 (EP), U13.2 (ENABLE#), U13.3 (PD)
- net PULSE_OUT: now also R46.2, U13.4 (IN-B)
- net at R20.1: now also U13.9 (OA)
- new net: R47.1, U13.12 (OB)
- new net: D9.1, J4.1 (In), R47.2
- new net +3.3V: C46.1, C47.1, U13.1 (VDD)
- no-connect marks 4 -> 7

Commit message: sch update
Other:
- note removed: "TODO: -5V source removed. U4 / U12 still use BUF602. Replace drivers or redesign supplies before operating outputs."
Changed lines of the file:
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@@
-		)
-	)
-	(text "TODO: -5V source removed. U4 / U12 still use BUF602.\nReplace drivers or redesign supplies before operating outputs."
-		(exclude_from_sim no)
-		(at 61.976 155.702 0)
-		(effects
-			(font
-				(size 1.27 1.27)
-			)
-			(justify left)
 		)
 	)

Commit message: sch update
Parts:
- R20, R47: footprint GPSDO_Rev1.0:C_0603_1608Metric -> GPSDO_Rev1.0:R_0805_2012Metric; symbol GPSDO_Rev1.0:R__C_0603_1608Metric -> GPSDO_Rev1.0:R__R_0805_2012Metric
Connections:
- net +5V renamed +5V2
Changed lines of the file:
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@@
 	(text "Pulse Outputs"
 		(exclude_from_sim no)
-		(at 109.22 43.434 0)
+		(at 110.998 44.45 0)
 		(effects
 			(font
@@
 	)
 	(junction
-		(at 93.98 127)
+		(at 165.1 115.57)
 		(diameter 0)
 		(color 0 0 0 0)
 	)
 	(junction
-		(at 165.1 115.57)
+		(at 93.98 127)
 		(diameter 0)
 		(color 0 0 0 0)
@@
 	)
 	(symbol
-		(lib_id "GPSDO_Rev1.0:R__C_0603_1608Metric")
+		(lib_id "GPSDO_Rev1.0:R__R_0805_2012Metric")
 		(at 179.07 102.87 90)
 		(unit 1)
@@
 			)
 		)
-		(property "Footprint" "GPSDO_Rev1.0:C_0603_1608Metric"
+		(property "Footprint" "GPSDO_Rev1.0:R_0805_2012Metric"
 			(at 179.07 104.648 90)
 			(hide yes)
@@
 			)
 		)
-		(property "Description" "Resistor"
+		(property "Description" "49.9 ohm source series resistor; select 0805 >=0.25W and verify temperature derating / load duty cycle"
 			(at 179.07 102.87 0)
 			(hide yes)
@@
 				(path "/7fcb1340-2836-48b1-8b47-374fa7e6ca96/1e6d2fc9-653e-45d2-a1bc-ab2903490aa7"
 					(reference "R42")
+					(unit 1)
+				)
+			)
+		)
+	)
+	(symbol
+		(lib_id "GPSDO_Rev1.0:+5V")
+		(at 171.45 115.57 0)
+		(unit 1)
+		(body_style 1)
+		(exclude_from_sim no)
+		(in_bom no)
+		(on_board yes)
+		(in_pos_files yes)
+		(dnp no)
+		(property "Reference" "#PWR0202"
+			(at 173.45 114.07 0)
+			(hide yes)
+			(show_name no)
+			(do_not_autoplace no)
+			(effects
+				(font
+					(size 1 1)
+				)
+				(justify left)
+			)
+		)
+		(property "Value" "+5V2"
+			(at 171.45 112.014 0)
+			(show_name no)
+			(do_not_autoplace no)
+			(effects
+				(font
+					(size 1 1)
+				)
+			)
+		)
+		(property "Footprint" ""
+			(at 171.45 115.57 0)
+			(hide yes)
+			(show_name no)
+			(do_not_autoplace no)
+			(effects
+				(font
+					(size 1 1)
+				)
+			)
+		)
+		(property "Datasheet" ""
+			(at 171.45 115.57 0)
+			(hide yes)
+			(show_name no)
+			(do_not_autoplace no)
+			(effects
+				(font
+					(size 1 1)
+				)
+			)
+		)
+		(property "Description" ""
+			(at 171.45 115.57 0)
+			(hide yes)
+			(show_name no)
+			(do_not_autoplace no)
+			(effects
+				(font
+					(size 1 1)
+				)
+			)
+		)
+		(pin "1"
+		)
+		(instances
+			(project "GPSDO_Rev1.0"
+				(path "/7fcb1340-2836-48b1-8b47-374fa7e6ca96/1e6d2fc9-653e-45d2-a1bc-ab2903490aa7"
+					(reference "#PWR0202")
 					(unit 1)
 				)
@@
 	)
 	(symbol
-		(lib_id "GPSDO_Rev1.0:R__C_0603_1608Metric")
+		(lib_id "GPSDO_Rev1.0:R__R_0805_2012Metric")
 		(at 107.95 113.03 270)
 		(mirror x)
@@
 			)
 		)
-		(property "Footprint" "GPSDO_Rev1.0:C_0603_1608Metric"
+		(property "Footprint" "GPSDO_Rev1.0:R_0805_2012Metric"
 			(at 107.95 114.808 90)
 			(hide yes)
@@
 			)
 		)
-		(property "Description" "Resistor"
+		(property "Description" "49.9 ohm source series resistor; select 0805 >=0.25W and verify temperature derating / load duty cycle"
 			(at 107.95 113.03 0)
 			(hide yes)
@@
 					(unit 1)
 				)
-			)
-		)
-	)
-	(symbol
-		(lib_id "GPSDO_Rev1.0:+5V")
-		(at 171.45 115.57 0)
-		(unit 1)
-		(body_style 1)
-		(exclude_from_sim no)
-		(in_bom yes)
-		(on_board yes)
-		(in_pos_files yes)
-		(dnp no)
-		(fields_autoplaced yes)
-		(property "Reference" "#PWR058"
-			(at 171.45 119.38 0)
-			(hide yes)
-			(show_name no)
-			(do_not_autoplace no)
-			(effects
-				(font
-					(size 1.27 1.27)
-				)
-			)
-		)
-		(property "Value" "+5V"
-			(at 171.45 110.49 0)
-			(show_name no)
-			(do_not_autoplace no)
-			(effects
-				(font
-					(size 1.27 1.27)
-				)
-			)
-		)
-		(property "Footprint" ""
-			(at 171.45 115.57 0)
-			(hide yes)
-			(show_name no)
-			(do_not_autoplace no)
-			(effects
-				(font
-					(size 1.27 1.27)
-				)
-			)
-		)
-		(property "Datasheet" ""
-			(at 171.45 115.57 0)
-			(hide yes)
-			(show_name no)
-			(do_not_autoplace no)
-			(effects
-				(font
-					(size 1.27 1.27)
-				)
-			)
-		)
-		(property "Description" "Power symbol creates a global label with name \"+5V\""
-			(at 171.45 115.57 0)
-			(hide yes)
-			(show_name no)
-			(do_not_autoplace no)
-			(effects
-				(font
-					(size 1.27 1.27)
-				)
-			)
-		)
-		(pin "1"
-		)
-		(instances
-			(project "GPSDO_Rev1.0"
-				(path "/7fcb1340-2836-48b1-8b47-374fa7e6ca96/1e6d2fc9-653e-45d2-a1bc-ab2903490aa7"
-					(reference "#PWR058")
-					(unit 1)
-				)
