File: hardware/schematic/v1.0/GPSDO_Rev1.0/GPSDO_Rev1.0.kicad_sch (KiCad schematic)
At the start: 3 parts, among them U1 TDC7200PWR, U2 LMK1C1103PWR, U3 TMP117AIDRVR

Commit message: add pdf and sch
Parts:
- removed U2: LMK1C1103PWR, GPSDO_Rev1.0:LMK1C1103PWR, symbol GPSDO_Rev1.0:LMK1C1103PWR
- removed U3: TMP117AIDRVR, GPSDO_Rev1.0:TMP117AIDRVR, symbol GPSDO_Rev1.0:TMP117AIDRVR
Other:
- added sheet EXT (EXT.kicad_sch)
- added sheet MCU (MCU.kicad_sch)
- added sheet OCXO (OCXO.kicad_sch)
Changed lines of the file:
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@@
 		)
 	)
-	(symbol
-		(lib_id "GPSDO_Rev1.0:LMK1C1103PWR")
-		(at 114.3 154.94 0)
-		(unit 1)
-		(body_style 1)
+	(sheet
+		(at 113.03 143.51)
+		(size 17.78 29.21)
 		(exclude_from_sim no)
 		(in_bom yes)
 		(on_board yes)
-		(in_pos_files yes)
 		(dnp no)
 		(fields_autoplaced yes)
-		(property "Reference" "U2"
-			(at 116.4433 143.51 0)
+		(stroke
+			(width 0.1524)
+			(type solid)
+		)
+		(fill
+			(color 0 0 0 0)
+		)
+		(property "Sheetname" "EXT"
+			(at 113.03 142.7984 0)
 			(show_name no)
 			(do_not_autoplace no)
@@
 					(size 1.27 1.27)
 				)
-				(justify left)
+				(justify left bottom)
 			)
 		)
-		(property "Value" "LMK1C1103PWR"
-			(at 116.4433 146.05 0)
+		(property "Sheetfile" "EXT.kicad_sch"
+			(at 113.03 173.3046 0)
 			(show_name no)
 			(do_not_autoplace no)
@@
 					(size 1.27 1.27)
 				)
-				(justify left)
+				(justify left top)
 			)
 		)
-		(property "Footprint" "GPSDO_Rev1.0:LMK1C1103PWR"
-			(at 114.3 153.67 0)
-			(hide yes)
+		(instances
+			(project "GPSDO_Rev1.0"
+				(path "/7fcb1340-2836-48b1-8b47-374fa7e6ca96"
+					(page "4")
+				)
+			)
+		)
+	)
+	(sheet
+		(at 62.23 132.08)
+		(size 26.67 30.48)
+		(exclude_from_sim no)
+		(in_bom yes)
+		(on_board yes)
+		(dnp no)
+		(fields_autoplaced yes)
+		(stroke
+			(width 0.1524)
+			(type solid)
+		)
+		(fill
+			(color 0 0 0 0)
+		)
+		(property "Sheetname" "OCXO"
+			(at 62.23 131.3684 0)
 			(show_name no)
 			(do_not_autoplace no)
@@
 					(size 1.27 1.27)
 				)
+				(justify left bottom)
 			)
 		)
-		(property "Datasheet" "https://wmsc.lcsc.com/wmsc/upload/file/pdf/v2/lcsc/2303010130_Texas-Instruments-LMK1C1103PWR_C2873274.pdf"
-			(at 114.3 153.67 0)
-			(hide yes)
+		(property "Sheetfile" "OCXO.kicad_sch"
+			(at 62.23 163.1446 0)
 			(show_name no)
 			(do_not_autoplace no)
@@
 					(size 1.27 1.27)
 				)
+				(justify left top)
 			)
 		)
-		(property "Description" "-40℃~+125℃ 1 1.71V~1.89V、2.375V~2.625V、3.135V~3.465V 250MHz 3 TSSOP-8 Clock Buffers, Drivers, Distributors ROHS"
-			(at 114.3 153.67 0)
-			(hide yes)
+		(instances
+			(project "GPSDO_Rev1.0"
+				(path "/7fcb1340-2836-48b1-8b47-374fa7e6ca96"
+					(page "3")
+				)
+			)
+		)
+	)
+	(sheet
+		(at 62.23 77.47)
+		(size 30.48 40.64)
+		(exclude_from_sim no)
+		(in_bom yes)
+		(on_board yes)
+		(dnp no)
+		(fields_autoplaced yes)
+		(stroke
+			(width 0.1524)
+			(type solid)
+		)
+		(fill
+			(color 0 0 0 0)
+		)
+		(property "Sheetname" "MCU"
+			(at 62.23 76.7584 0)
 			(show_name no)
 			(do_not_autoplace no)
@@
 					(size 1.27 1.27)
 				)
+				(justify left bottom)
 			)
 		)
-		(property "LCSC" "C2873274"
-			(at 114.3 154.94 0)
-			(hide yes)
+		(property "Sheetfile" "MCU.kicad_sch"
+			(at 62.23 118.6946 0)
 			(show_name no)
 			(do_not_autoplace no)
@@
 					(size 1.27 1.27)
 				)
+				(justify left top)
 			)
-		)
-		(property "Manufacturer" "Texas Instruments"
-			(at 114.3 154.94 0)
-			(hide yes)
-			(show_name no)
-			(do_not_autoplace no)
-			(effects
-				(font
-					(size 1.27 1.27)
-				)
-			)
-		)
-		(property "Manufacturer Part" "LMK1C1103PWR"
-			(at 114.3 154.94 0)
-			(hide yes)
-			(show_name no)
-			(do_not_autoplace no)
-			(effects
-				(font
-					(size 1.27 1.27)
-				)
-			)
-		)
-		(pin "7"
-		)
-		(pin "5"
-		)
-		(pin "1"
-		)
-		(pin "3"
-		)
-		(pin "8"
-		)
-		(pin "2"
-		)
-		(pin "4"
-		)
-		(pin "6"
 		)
 		(instances
 			(project "GPSDO_Rev1.0"
 				(path "/7fcb1340-2836-48b1-8b47-374fa7e6ca96"
-					(reference "U2")
-					(unit 1)
+					(page "2")
 				)
 			)
-		)
-	)
-	(symbol
-		(lib_id "GPSDO_Rev1.0:TMP117AIDRVR")
-		(at 209.55 149.86 0)
-		(unit 1)
-		(body_style 1)
-		(exclude_from_sim no)
-		(in_bom yes)
-		(on_board yes)
-		(in_pos_files yes)
-		(dnp no)
-		(fields_autoplaced yes)
-		(property "Reference" "U3"
-			(at 209.55 138.43 0)
-			(show_name no)
-			(do_not_autoplace no)
-			(effects
-				(font
-					(size 1.27 1.27)
-				)
-			)
-		)
-		(property "Value" "TMP117AIDRVR"
-			(at 209.55 140.97 0)
-			(show_name no)
-			(do_not_autoplace no)
-			(effects
-				(font
-					(size 1.27 1.27)
-				)
-			)
-		)
-		(property "Footprint" "GPSDO_Rev1.0:TMP117AIDRVR"
-			(at 209.55 149.86 0)
-			(hide yes)
-			(show_name no)
-			(do_not_autoplace no)
-			(effects
-				(font
-					(size 1.27 1.27)
-				)
-			)
-		)
-		(property "Datasheet" "https://www.lcsc.com/datasheet/lcsc_datasheet_2309221403_Texas-Instruments-TMP117AIDRVR_C699536.pdf"
-			(at 209.55 149.86 0)
-			(hide yes)
-			(show_name no)
-			(do_not_autoplace no)
-			(effects
-				(font
-					(size 1.27 1.27)
-				)
-			)
-		)
-		(property "Description" "-55℃~+150℃ 1.7V~5.5V 15.5ms 16bit 3.1uA Factory temperature calibration、Temperature threshold monitoring、Low-power standby、On-chip non-volatile parameter storage、On-chip digital filtering/averaging I2C、SMBus ±0.1℃ WDFN-6-EP(2x2) Temperature Sensors ROHS"
-			(at 209.55 149.86 0)
-			(hide yes)
-			(show_name no)
-			(do_not_autoplace no)
-			(effects
-				(font
-					(size 1.27 1.27)
-				)
-			)
-		)
-		(property "LCSC" "C699536"
-			(at 209.55 149.86 0)
-			(hide yes)
-			(show_name no)
-			(do_not_autoplace no)
-			(effects
-				(font
-					(size 1.27 1.27)
-				)
-			)
-		)
-		(property "Manufacturer" "Texas Instruments"
-			(at 209.55 149.86 0)
-			(hide yes)
-			(show_name no)
-			(do_not_autoplace no)
-			(effects
-				(font
-					(size 1.27 1.27)
-				)
-			)
-		)
-		(property "Manufacturer Part" "TMP117AIDRVR"
-			(at 209.55 149.86 0)
-			(hide yes)
-			(show_name no)
-			(do_not_autoplace no)
-			(effects
-				(font
-					(size 1.27 1.27)
-				)
-			)
-		)
-		(pin "3"
-		)
-		(pin "5"
-		)
-		(pin "7"
-		)
-		(pin "4"
-		)
-		(pin "6"
-		)
-		(pin "1"
-		)
-		(pin "2"
-		)
-		(instances
-			(project "GPSDO_Rev1.0"
-				(path "/7fcb1340-2836-48b1-8b47-374fa7e6ca96"
-					(reference "U3")
-					(unit 1)
-				)
-			)

Commit message: sch update
Parts:
- removed U1: TDC7200PWR, GPSDO_Rev1.0:TDC7200PWR, symbol GPSDO_Rev1.0:TDC7200PWR
Other:
- added sheet GNSS (GNSS.kicad_sch)
Changed lines of the file:
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@@
 	(generator_version "10.0")
 	(paper "A4")
-	(symbol
-		(lib_id "GPSDO_Rev1.0:TDC7200PWR")
-		(at 163.83 121.92 0)
-		(unit 1)
-		(body_style 1)
-		(exclude_from_sim no)
-		(in_bom yes)
-		(on_board yes)
-		(in_pos_files yes)
-		(dnp no)
-		(fields_autoplaced yes)
-		(property "Reference" "U1"
-			(at 163.83 106.68 0)
-			(show_name no)
-			(do_not_autoplace no)
-			(effects
-				(font
-					(size 1.27 1.27)
-				)
-			)
-		)
-		(property "Value" "TDC7200PWR"
-			(at 163.83 109.22 0)
-			(show_name no)
-			(do_not_autoplace no)
-			(effects
-				(font
-					(size 1.27 1.27)
-				)
-			)
-		)
-		(property "Footprint" "GPSDO_Rev1.0:TDC7200PWR"
-			(at 163.83 121.92 0)
-			(hide yes)
-			(show_name no)
-			(do_not_autoplace no)
-			(effects
-				(font
-					(size 1.27 1.27)
-				)
-			)
-		)
-		(property "Datasheet" "https://www.lcsc.com/datasheet/lcsc_datasheet_2303011701_Texas-Instruments-TDC7200PWR_C2653139.pdf"
-			(at 163.83 121.92 0)
-			(hide yes)
-			(show_name no)
-			(do_not_autoplace no)
-			(effects
-				(font
-					(size 1.27 1.27)
-				)
-			)
-		)
-		(property "Description" "-40℃~+85℃ 0.5uA 20MHz 2V~3.6V SPI TSSOP-14 ADCs/DACs - Special Purpose ROHS"
-			(at 163.83 121.92 0)
-			(hide yes)
-			(show_name no)
-			(do_not_autoplace no)
-			(effects
-				(font
-					(size 1.27 1.27)
-				)
-			)
-		)
-		(property "LCSC" "C2653139"
-			(at 163.83 121.92 0)
-			(hide yes)
-			(show_name no)
-			(do_not_autoplace no)
-			(effects
-				(font
-					(size 1.27 1.27)
-				)
-			)
-		)
-		(property "Manufacturer" "Texas Instruments"
-			(at 163.83 121.92 0)
-			(hide yes)
-			(show_name no)
-			(do_not_autoplace no)
-			(effects
-				(font
-					(size 1.27 1.27)
-				)
-			)
-		)
-		(property "Manufacturer Part" "TDC7200PWR"
-			(at 163.83 121.92 0)
-			(hide yes)
-			(show_name no)
-			(do_not_autoplace no)
-			(effects
-				(font
-					(size 1.27 1.27)
-				)
-			)
-		)
-		(pin "5"
-		)
-		(pin "6"
-		)
-		(pin "10"
-		)
-		(pin "13"
-		)
-		(pin "9"
-		)
-		(pin "1"
-		)
-		(pin "2"
-		)
-		(pin "3"
-		)
-		(pin "4"
-		)
-		(pin "7"
-		)
-		(pin "8"
-		)
-		(pin "11"
-		)
-		(pin "12"
-		)
-		(pin "14"
-		)
-		(instances
-			(project "GPSDO_Rev1.0"
-				(path "/7fcb1340-2836-48b1-8b47-374fa7e6ca96"
-					(reference "U1")
-					(unit 1)
-				)
-			)
-		)
-	)
 	(sheet
 		(at 113.03 143.51)
@@
 				)
 			)
+		)
+	)
+	(sheet
+		(at 115.57 92.71)
+		(size 13.97 27.94)
+		(exclude_from_sim no)
+		(in_bom yes)
+		(on_board yes)
+		(dnp no)
+		(fields_autoplaced yes)
+		(stroke
+			(width 0.1524)
+			(type solid)
+		)
+		(fill
+			(color 0 0 0 0)
+		)
+		(property "Sheetname" "GNSS"
+			(at 115.57 91.9984 0)
+			(show_name no)
+			(do_not_autoplace no)
+			(effects
+				(font
+					(size 1.27 1.27)
+				)
+				(justify left bottom)
+			)
+		)
+		(property "Sheetfile" "GNSS.kicad_sch"
+			(at 115.57 121.2346 0)
+			(show_name no)
+			(do_not_autoplace no)
+			(effects
+				(font
+					(size 1.27 1.27)
+				)
+				(justify left top)
+			)
+		)
+		(instances
+			(project "GPSDO_Rev1.0"
+				(path "/7fcb1340-2836-48b1-8b47-374fa7e6ca96"
+					(page "5")
+				)
+			)

Commit message: sch update
Other:
- added sheet POWER (POWER.kicad_sch)
Changed lines of the file:
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@@
+		)
+	)
+	(sheet
+		(at 167.64 99.06)
+		(size 24.13 29.21)
+		(exclude_from_sim no)
+		(in_bom yes)
+		(on_board yes)
+		(dnp no)
+		(fields_autoplaced yes)
+		(stroke
+			(width 0.1524)
+			(type solid)
+		)
+		(fill
+			(color 0 0 0 0)
+		)
+		(property "Sheetname" "POWER"
+			(at 167.64 98.3484 0)
+			(show_name no)
+			(do_not_autoplace no)
+			(effects
+				(font
+					(size 1.27 1.27)
+				)
+				(justify left bottom)
+			)
+		)
+		(property "Sheetfile" "POWER.kicad_sch"
+			(at 167.64 128.8546 0)
+			(show_name no)
+			(do_not_autoplace no)
+			(effects
+				(font
+					(size 1.27 1.27)
+				)
+				(justify left top)
+			)
+		)
+		(instances
+			(project "GPSDO_Rev1.0"
+				(path "/7fcb1340-2836-48b1-8b47-374fa7e6ca96"
+					(page "6")
+				)
+			)
 		)
 	)

Commit message: sch update
Parts:
- added H1, H2, H3, H4: MountingHole_Pad, MountingHole:MountingHole_3.2mm_M3_Pad, symbol Mechanical:MountingHole_Pad
Connections:
- new net GND: H1.1, H2.1, H3.1, H4.1
Other:
- note added: "HOLE"

Commit message: sch update
Parts:
- H1, H2, H3, H4: footprint MountingHole:MountingHole_3.2mm_M3_Pad -> GPSDO_Rev1.0:MountingHole_3.2mm_M3_Pad; symbol Mechanical:MountingHole_Pad -> GPSDO_Rev1.0:MountingHole_Pad
Changed lines of the file:
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@@
 	)
 	(symbol
-		(lib_id "Mechanical:MountingHole_Pad")
+		(lib_id "GPSDO_Rev1.0:MountingHole_Pad")
 		(at 219.71 151.13 0)
 		(unit 1)
@@
 			)
 		)
-		(property "Footprint" "MountingHole:MountingHole_3.2mm_M3_Pad"
+		(property "Footprint" "GPSDO_Rev1.0:MountingHole_3.2mm_M3_Pad"
 			(at 219.71 151.13 0)
 			(hide yes)
@@
 	)
 	(symbol
-		(lib_id "Mechanical:MountingHole_Pad")
+		(lib_id "GPSDO_Rev1.0:MountingHole_Pad")
 		(at 219.71 135.89 0)
 		(unit 1)
@@
 			)
 		)
-		(property "Footprint" "MountingHole:MountingHole_3.2mm_M3_Pad"
+		(property "Footprint" "GPSDO_Rev1.0:MountingHole_3.2mm_M3_Pad"
 			(at 219.71 135.89 0)
 			(hide yes)
@@
 	)
 	(symbol
-		(lib_id "power:GND")
+		(lib_id "GPSDO_Rev1.0:GND")
 		(at 219.71 153.67 0)
 		(unit 1)
@@
 	)
 	(symbol
-		(lib_id "power:GND")
+		(lib_id "GPSDO_Rev1.0:GND")
 		(at 252.73 138.43 0)
 		(unit 1)
@@
 	)
 	(symbol
-		(lib_id "power:GND")
+		(lib_id "GPSDO_Rev1.0:GND")
 		(at 252.73 153.67 0)
 		(unit 1)
@@
 	)
 	(symbol
-		(lib_id "power:GND")
+		(lib_id "GPSDO_Rev1.0:GND")
 		(at 219.71 138.43 0)
 		(unit 1)
@@
 	)
 	(symbol
-		(lib_id "Mechanical:MountingHole_Pad")
+		(lib_id "GPSDO_Rev1.0:MountingHole_Pad")
 		(at 252.73 151.13 0)
 		(unit 1)
@@
 			)
 		)
-		(property "Footprint" "MountingHole:MountingHole_3.2mm_M3_Pad"
+		(property "Footprint" "GPSDO_Rev1.0:MountingHole_3.2mm_M3_Pad"
 			(at 252.73 151.13 0)
 			(hide yes)
@@
 	)
 	(symbol
-		(lib_id "Mechanical:MountingHole_Pad")
+		(lib_id "GPSDO_Rev1.0:MountingHole_Pad")
 		(at 252.73 135.89 0)
 		(unit 1)
@@
 			)
 		)
-		(property "Footprint" "MountingHole:MountingHole_3.2mm_M3_Pad"
+		(property "Footprint" "GPSDO_Rev1.0:MountingHole_3.2mm_M3_Pad"
 			(at 252.73 135.89 0)
 			(hide yes)

Commit message: sch update
Other:
- sheet EXT ports: added 10MHZ_OUT, PULSE_OUT; removed none
- sheet GNSS ports: added GNSS_UART_RXD, GNSS_UART_TXD, PULSE_GNSS; removed none
- sheet MCU ports: added 10MHZ_MCU, 10MHZ_TDC, GNSS_UART_RXD, GNSS_UART_TXD, PULSE_GNSS, PWM, TMP_SCL, TMP_SDA; removed none
Changed lines of the file:
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@@
+			)
+		)
+		(pin "PULSE_OUT" input
+			(at 106.68 110.49 180)
+			(effects
+				(font
+					(size 1.27 1.27)
+				)
+				(justify left)
+			)
+		)
+		(pin "10MHZ_OUT" input
+			(at 106.68 123.19 180)
+			(effects
+				(font
+					(size 1.27 1.27)
+				)
+				(justify left)
 			)
 		)
@@
 	(sheet
 		(at 109.22 52.07)
-		(size 13.97 27.94)
+		(size 21.59 27.94)
 		(exclude_from_sim no)
 		(in_bom yes)
@@
 				)
 				(justify left top)
+			)
+		)
+		(pin "GNSS_UART_RXD" input
+			(at 109.22 60.96 180)
+			(effects
+				(font
+					(size 1.27 1.27)
+				)
+				(justify left)
+			)
+		)
+		(pin "GNSS_UART_TXD" output
+			(at 109.22 63.5 180)
+			(effects
+				(font
+					(size 1.27 1.27)
+				)
+				(justify left)
+			)
+		)
+		(pin "PULSE_GNSS" output
+			(at 109.22 67.31 180)
+			(effects
+				(font
+					(size 1.27 1.27)
+				)
+				(justify left)
 			)
 		)
@@
 			)
 		)
+		(pin "10MHZ_TDC" input
+			(at 86.36 50.8 0)
+			(effects
+				(font
+					(size 1.27 1.27)
+				)
+				(justify right)
+			)
+		)
+		(pin "TMP_SDA" bidirectional
+			(at 86.36 64.77 0)
+			(effects
+				(font
+					(size 1.27 1.27)
+				)
+				(justify right)
+			)
+		)
+		(pin "PULSE_GNSS" input
+			(at 86.36 72.39 0)
+			(effects
+				(font
+					(size 1.27 1.27)
+				)
+				(justify right)
+			)
+		)
+		(pin "10MHZ_MCU" input
+			(at 86.36 68.58 0)
+			(effects
+				(font
+					(size 1.27 1.27)
+				)
+				(justify right)
+			)
+		)
+		(pin "PWM" output
+			(at 86.36 43.18 0)
+			(effects
+				(font
+					(size 1.27 1.27)
+				)
+				(justify right)
+			)
+		)
+		(pin "GNSS_UART_RXD" output
+			(at 86.36 57.15 0)
+			(effects
+				(font
+					(size 1.27 1.27)
+				)
+				(justify right)
+			)
+		)
+		(pin "GNSS_UART_TXD" input
+			(at 86.36 59.69 0)
+			(effects
+				(font
+					(size 1.27 1.27)
+				)
+				(justify right)
+			)
+		)
+		(pin "TMP_SCL" output
+			(at 86.36 62.23 0)
+			(effects
+				(font
+					(size 1.27 1.27)
+				)
+				(justify right)
+			)
+		)

Commit message: pdf update
Other:
- sheet OCXO ports: added 10MHZ_MCU, 10MHZ_OUT, 10MHZ_TDC, OCXO_VCC, PWM, TMP_SCL, TMP_SDA; removed none
- sheet POWER ports: added OCXO_VCC, PDN; removed none
Changed lines of the file:
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@@
 	)
 	(sheet
-		(at 106.68 102.87)
+		(at 156.21 99.06)
 		(size 17.78 29.21)
 		(exclude_from_sim no)
@@
 		)
 		(property "Sheetname" "EXT"
-			(at 106.68 102.1584 0)
+			(at 156.21 98.3484 0)
 			(show_name no)
 			(do_not_autoplace no)
@@
 		)
 		(property "Sheetfile" "EXT.kicad_sch"
-			(at 106.68 132.6646 0)
+			(at 156.21 128.8546 0)
 			(show_name no)
 			(do_not_autoplace no)
@@
 		)
 		(pin "PULSE_OUT" input
-			(at 106.68 110.49 180)
+			(at 156.21 106.68 180)
 			(effects
 				(font
@@
 		)
 		(pin "10MHZ_OUT" input
-			(at 106.68 123.19 180)
+			(at 156.21 119.38 180)
 			(effects
 				(font
@@
 			)
 		)
+		(pin "10MHZ_OUT" output
+			(at 82.55 97.79 0)
+			(effects
+				(font
+					(size 1.27 1.27)
+				)
+				(justify right)
+			)
+		)
+		(pin "OCXO_VCC" bidirectional
+			(at 82.55 118.11 0)
+			(effects
+				(font
+					(size 1.27 1.27)
+				)
+				(justify right)
+			)
+		)
+		(pin "TMP_SCL" input
+			(at 82.55 114.3 0)
+			(effects
+				(font
+					(size 1.27 1.27)
+				)
+				(justify right)
+			)
+		)
+		(pin "10MHZ_MCU" output
+			(at 82.55 100.33 0)
+			(effects
+				(font
+					(size 1.27 1.27)
+				)
+				(justify right)
+			)
+		)
+		(pin "TMP_SDA" bidirectional
+			(at 82.55 111.76 0)
+			(effects
+				(font
+					(size 1.27 1.27)
+				)
+				(justify right)
+			)
+		)
+		(pin "PWM" input
+			(at 82.55 106.68 0)
+			(effects
+				(font
+					(size 1.27 1.27)
+				)
+				(justify right)
+			)
+		)
+		(pin "10MHZ_TDC" output
+			(at 82.55 102.87 0)
+			(effects
+				(font
+					(size 1.27 1.27)
+				)
+				(justify right)
+			)
+		)
 		(instances
 			(project "GPSDO_Rev1.0"
@@
 	)
 	(sheet
-		(at 55.88 36.83)
-		(size 30.48 40.64)
+		(at 105.41 91.44)
+		(size 35.56 40.64)
 		(exclude_from_sim no)
 		(in_bom yes)
@@
 		)
 		(property "Sheetname" "MCU"
-			(at 55.88 36.1184 0)
+			(at 105.41 90.7284 0)
 			(show_name no)
 			(do_not_autoplace no)
@@
 		)
 		(property "Sheetfile" "MCU.kicad_sch"
-			(at 55.88 78.0546 0)
+			(at 105.41 132.6646 0)
 			(show_name no)
 			(do_not_autoplace no)
@@
 		)
 		(pin "10MHZ_TDC" input
-			(at 86.36 50.8 0)
-			(effects
-				(font
-					(size 1.27 1.27)
-				)
-				(justify right)
+			(at 105.41 102.87 180)
+			(effects
+				(font
+					(size 1.27 1.27)
+				)
+				(justify left)
 			)
 		)
 		(pin "TMP_SDA" bidirectional
-			(at 86.36 64.77 0)
-			(effects
-				(font
-					(size 1.27 1.27)
-				)
-				(justify right)
+			(at 105.41 111.76 180)
+			(effects
+				(font
+					(size 1.27 1.27)
+				)
+				(justify left)
 			)
 		)
 		(pin "PULSE_GNSS" input
-			(at 86.36 72.39 0)
+			(at 140.97 127 0)
 			(effects
 				(font
@@
 		)
 		(pin "10MHZ_MCU" input
-			(at 86.36 68.58 0)
-			(effects
-				(font
-					(size 1.27 1.27)
-				)
-				(justify right)
+			(at 105.41 100.33 180)
+			(effects
+				(font
+					(size 1.27 1.27)
+				)
+				(justify left)
 			)
 		)
 		(pin "PWM" output
-			(at 86.36 43.18 0)
-			(effects
-				(font
-					(size 1.27 1.27)
-				)
-				(justify right)
+			(at 105.41 106.68 180)
+			(effects
+				(font
+					(size 1.27 1.27)
+				)
+				(justify left)
 			)
 		)
 		(pin "GNSS_UART_RXD" output
-			(at 86.36 57.15 0)
+			(at 140.97 111.76 0)
 			(effects
 				(font
@@
 		)
 		(pin "GNSS_UART_TXD" input
-			(at 86.36 59.69 0)
+			(at 140.97 114.3 0)
 			(effects
 				(font
@@
 		)
 		(pin "TMP_SCL" output
-			(at 86.36 62.23 0)
-			(effects
-				(font
-					(size 1.27 1.27)
-				)
-				(justify right)
+			(at 105.41 114.3 180)
+			(effects
+				(font
+					(size 1.27 1.27)
+				)
+				(justify left)
 			)
 		)
@@
 			)
 		)
+		(pin "OCXO_VCC" output
+			(at 161.29 68.58 180)
+			(effects
+				(font
+					(size 1.27 1.27)
+				)
+				(justify left)
+			)
+		)
+		(pin "PDN" output
+			(at 161.29 73.66 180)
+			(effects
+				(font
+					(size 1.27 1.27)
+				)
+				(justify left)
+			)
+		)
