File: hardware/schematic/v1.0/GPSDO_Rev1.0/GPSDO_Rev1.0.kicad_sch (KiCad schematic)
At the start: 4 parts

Commit message: sch update
Other:
- sheet MCU ports: added PULSE_MCU, VCTL; removed none
- sheet OCXO ports: added VCTL; removed none
Changed lines of the file:
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@@
+		)
+	)
+	(wire
+		(pts
+			(xy 118.11 120.65) (xy 130.81 120.65)
+		)
+		(stroke
+			(width 0)
+			(type default)
 		)
 	)
@@
 			(width 0)
 			(type dash)
+		)
+	)
+	(wire
+		(pts
+			(xy 118.11 105.41) (xy 130.81 105.41)
+		)
+		(stroke
+			(width 0)
+			(type default)
+		)
+	)
+	(wire
+		(pts
+			(xy 118.11 107.95) (xy 130.81 107.95)
+		)
+		(stroke
+			(width 0)
+			(type default)
+		)
+	)
+	(wire
+		(pts
+			(xy 76.2 119.38) (xy 82.55 119.38)
+		)
+		(stroke
+			(width 0)
+			(type default)
+		)
+	)
+	(wire
+		(pts
+			(xy 118.11 118.11) (xy 130.81 118.11)
+		)
+		(stroke
+			(width 0)
+			(type default)
+		)
+	)
+	(wire
+		(pts
+			(xy 124.46 91.44) (xy 172.72 91.44)
+		)
+		(stroke
+			(width 0)
+			(type default)
+		)
+	)
+	(wire
+		(pts
+			(xy 118.11 111.76) (xy 130.81 111.76)
+		)
+		(stroke
+			(width 0)
+			(type default)
+		)
+	)
+	(wire
+		(pts
+			(xy 76.2 116.84) (xy 82.55 116.84)
+		)
+		(stroke
+			(width 0)
+			(type default)
+		)
+	)
+	(wire
+		(pts
+			(xy 76.2 113.03) (xy 82.55 113.03)
+		)
+		(stroke
+			(width 0)
+			(type default)
+		)
+	)
+	(wire
+		(pts
+			(xy 124.46 91.44) (xy 124.46 99.06)
+		)
+		(stroke
+			(width 0)
+			(type default)
+		)
+	)
+	(wire
+		(pts
+			(xy 118.11 99.06) (xy 124.46 99.06)
+		)
+		(stroke
+			(width 0)
+			(type default)
+		)
+	)
+	(wire
+		(pts
+			(xy 166.37 111.76) (xy 179.07 111.76)
+		)
+		(stroke
+			(width 0)
+			(type default)
+		)
+	)
+	(wire
+		(pts
+			(xy 172.72 91.44) (xy 172.72 105.41)
+		)
+		(stroke
+			(width 0)
+			(type default)
+		)
+	)
+	(wire
+		(pts
+			(xy 118.11 114.3) (xy 130.81 114.3)
+		)
+		(stroke
+			(width 0)
+			(type default)
+		)
+	)
+	(wire
+		(pts
+			(xy 172.72 105.41) (xy 179.07 105.41)
+		)
+		(stroke
+			(width 0)
+			(type default)
 		)
 	)
@@
 	)
 	(sheet
-		(at 151.13 87.63)
+		(at 179.07 100.33)
 		(size 17.78 16.51)
 		(exclude_from_sim no)
@@
 		)
 		(property "Sheetname" "EXT"
-			(at 151.13 86.9184 0)
+			(at 179.07 99.6184 0)
 			(show_name no)
 			(do_not_autoplace no)
@@
 		)
 		(property "Sheetfile" "EXT.kicad_sch"
-			(at 151.13 104.7246 0)
+			(at 179.07 117.4246 0)
 			(show_name no)
 			(do_not_autoplace no)
@@
 		)
 		(pin "PULSE_OUT" input
-			(at 151.13 92.71 180)
+			(at 179.07 105.41 180)
 			(effects
 				(font
@@
 		)
 		(pin "10MHZ_OUT" input
-			(at 151.13 99.06 180)
+			(at 179.07 111.76 180)
 			(effects
 				(font
@@
 	)
 	(sheet
-		(at 97.79 92.71)
-		(size 35.56 30.48)
+		(at 130.81 97.79)
+		(size 35.56 33.02)
 		(exclude_from_sim no)
 		(in_bom yes)
@@
 		)
 		(property "Sheetname" "OCXO"
-			(at 97.79 91.9984 0)
+			(at 130.81 97.0784 0)
 			(show_name no)
 			(do_not_autoplace no)
@@
 		)
 		(property "Sheetfile" "OCXO.kicad_sch"
-			(at 97.79 123.7746 0)
+			(at 130.81 131.3946 0)
 			(show_name no)
 			(do_not_autoplace no)
@@
 		)
 		(pin "10MHZ_OUT" output
-			(at 133.35 99.06 0)
+			(at 166.37 111.76 0)
 			(effects
 				(font
@@
 		)
 		(pin "OCXO_VCC" bidirectional
-			(at 97.79 119.38 180)
+			(at 130.81 124.46 180)
 			(effects
 				(font
@@
 		)
 		(pin "TMP_SCL" input
-			(at 97.79 115.57 180)
+			(at 130.81 120.65 180)
 			(effects
 				(font
@@
 		)
 		(pin "10MHZ_MCU" output
-			(at 97.79 100.33 180)
+			(at 130.81 105.41 180)
 			(effects
 				(font
@@
 		)
 		(pin "TMP_SDA" bidirectional
-			(at 97.79 113.03 180)
+			(at 130.81 118.11 180)
 			(effects
 				(font
@@
 		)
 		(pin "PWM" input
-			(at 97.79 109.22 180)
+			(at 130.81 111.76 180)
 			(effects
 				(font
@@
 		)
 		(pin "10MHZ_TDC" output
-			(at 97.79 102.87 180)
+			(at 130.81 107.95 180)
+			(effects
+				(font
+					(size 1.27 1.27)
+				)
+				(justify left)
+			)
+		)
+		(pin "VCTL" output
+			(at 130.81 114.3 180)
 			(effects
 				(font
@@
 	)
 	(sheet
-		(at 179.07 132.08)
-		(size 21.59 27.94)
+		(at 54.61 109.22)
+		(size 21.59 13.97)
 		(exclude_from_sim no)
 		(in_bom yes)
@@
 		)
 		(property "Sheetname" "GNSS"
-			(at 179.07 131.3684 0)
+			(at 54.61 108.5084 0)
 			(show_name no)
 			(do_not_autoplace no)
@@
 		)
 		(property "Sheetfile" "GNSS.kicad_sch"
-			(at 179.07 160.6046 0)
+			(at 54.61 123.7746 0)
 			(show_name no)
 			(do_not_autoplace no)
@@
 		)
 		(pin "GNSS_UART_RXD" input
-			(at 179.07 140.97 180)
-			(effects
-				(font
-					(size 1.27 1.27)
-				)
-				(justify left)
+			(at 76.2 119.38 0)
+			(effects
+				(font
+					(size 1.27 1.27)
+				)
+				(justify right)
 			)
 		)
 		(pin "GNSS_UART_TXD" output
-			(at 179.07 143.51 180)
-			(effects
-				(font
-					(size 1.27 1.27)
-				)
-				(justify left)
+			(at 76.2 116.84 0)
+			(effects
+				(font
+					(size 1.27 1.27)
+				)
+				(justify right)
 			)
 		)
 		(pin "PULSE_GNSS" output
-			(at 179.07 147.32 180)
-			(effects
-				(font
-					(size 1.27 1.27)
-				)
-				(justify left)
+			(at 76.2 113.03 0)
+			(effects
+				(font
+					(size 1.27 1.27)
+				)
+				(justify right)
 			)
 		)
@@
 	)
 	(sheet
-		(at 49.53 85.09)
-		(size 35.56 44.45)
+		(at 82.55 95.25)
+		(size 35.56 31.75)
 		(exclude_from_sim no)
 		(in_bom yes)
@@
 		)
 		(property "Sheetname" "MCU"
-			(at 49.53 84.3784 0)
+			(at 82.55 94.5384 0)
 			(show_name no)
 			(do_not_autoplace no)
@@
 		)
 		(property "Sheetfile" "MCU.kicad_sch"
-			(at 49.53 130.1246 0)
+			(at 82.55 127.5846 0)
 			(show_name no)
 			(do_not_autoplace no)
@@
 		)
 		(pin "10MHZ_TDC" input
-			(at 49.53 96.52 180)
-			(effects
-				(font
-					(size 1.27 1.27)
-				)
-				(justify left)
+			(at 118.11 107.95 0)
+			(effects
+				(font
+					(size 1.27 1.27)
+				)
+				(justify right)
 			)
 		)
 		(pin "TMP_SDA" bidirectional
-			(at 49.53 106.68 180)
-			(effects
-				(font
-					(size 1.27 1.27)
-				)
-				(justify left)
+			(at 118.11 118.11 0)
+			(effects
+				(font
+					(size 1.27 1.27)
+				)
+				(justify right)
 			)
 		)
 		(pin "PULSE_GNSS" input
-			(at 85.09 100.33 0)
+			(at 82.55 113.03 180)
+			(effects
+				(font
+					(size 1.27 1.27)
+				)
+				(justify left)
+			)
+		)
+		(pin "10MHZ_MCU" input
+			(at 118.11 105.41 0)
 			(effects
 				(font
@@
 			)
 		)
-		(pin "10MHZ_MCU" input
-			(at 49.53 93.98 180)
-			(effects
-				(font
-					(size 1.27 1.27)
-				)
-				(justify left)
-			)
-		)
 		(pin "PWM" output
-			(at 49.53 100.33 180)
-			(effects
-				(font
-					(size 1.27 1.27)
-				)
-				(justify left)
+			(at 118.11 111.76 0)
+			(effects
+				(font
+					(size 1.27 1.27)
+				)
+				(justify right)
 			)
 		)
 		(pin "GNSS_UART_RXD" output
-			(at 85.09 93.98 0)
+			(at 82.55 119.38 180)
+			(effects
+				(font
+					(size 1.27 1.27)
+				)
+				(justify left)
+			)
+		)
+		(pin "GNSS_UART_TXD" input
+			(at 82.55 116.84 180)
+			(effects
+				(font
+					(size 1.27 1.27)
+				)
+				(justify left)
+			)
+		)
+		(pin "TMP_SCL" output
+			(at 118.11 120.65 0)
 			(effects
 				(font
@@
 			)
 		)
-		(pin "GNSS_UART_TXD" input
-			(at 85.09 96.52 0)
+		(pin "PULSE_MCU" output
+			(at 118.11 99.06 0)
 			(effects
 				(font
@@
 			)
 		)
-		(pin "TMP_SCL" output
-			(at 49.53 109.22 180)
-			(effects
-				(font
-					(size 1.27 1.27)
-				)
-				(justify left)
-			)
-		)
+		(pin "VCTL" input
+			(at 118.11 114.3 0)
+			(effects
+				(font
+					(size 1.27 1.27)
+				)
+				(justify right)
+			)
+		)

Commit message: sch update
Other:
- sheet OCXO ports: added none; removed OCXO_VCC
- sheet POWER ports: added none; removed OCXO_VCC, PDN
Changed lines of the file:
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@@
-			)
-		)
-		(pin "OCXO_VCC" bidirectional
-			(at 130.81 124.46 180)
-			(effects
-				(font
-					(size 1.27 1.27)
-				)
-				(justify left)
 			)
 		)
@@
 	)
 	(sheet
-		(at 200.66 58.42)
+		(at 214.63 77.47)
 		(size 24.13 29.21)
 		(exclude_from_sim no)
@@
 		)
 		(property "Sheetname" "POWER"
-			(at 200.66 57.7084 0)
+			(at 214.63 76.7584 0)
 			(show_name no)
 			(do_not_autoplace no)
@@
 		)
 		(property "Sheetfile" "POWER.kicad_sch"
-			(at 200.66 88.2146 0)
+			(at 214.63 107.2646 0)
 			(show_name no)
 			(do_not_autoplace no)
@@
 			)
 		)
-		(pin "OCXO_VCC" output
-			(at 200.66 68.58 180)
-			(effects
-				(font
-					(size 1.27 1.27)
-				)
-				(justify left)
-			)
-		)
-		(pin "PDN" output
-			(at 200.66 73.66 180)
-			(effects
-				(font
-					(size 1.27 1.27)
-				)
-				(justify left)
-			)
-		)

Commit message: sch update
Other:
- sheet MCU ports: added BOOST_EN; removed none
- sheet POWER ports: added BOOST_EN; removed none
