File: hardware/schematic/v1.0/GPSDO_Rev1.0/POWER.kicad_sch (KiCad schematic)
At the start: 18 parts, among them CN1 LAIL-PHC2_54-2P-01-XH-L, U12 TPS7A5201RPSR, U13 TPS7A5201RPSR

Commit message: sch update
Parts:
- removed C22, C23, C28, C29: 22uF, Capacitor_SMD:C_0805_2012Metric, symbol Device:C
- removed C24, C26: 100nF, Capacitor_SMD:C_0402_1005Metric, symbol Device:C
- removed C25, C27: 10nF, Capacitor_SMD:C_0402_1005Metric, symbol Device:C
- removed R20, R23: 100K, Resistor_SMD:R_0402_1005Metric, symbol Device:R
- removed R21, R22: 12.1K, Resistor_SMD:R_0402_1005Metric, symbol Device:R
- removed R24, R25: 3.87K, Resistor_SMD:R_0402_1005Metric, symbol Device:R
- removed U12, U13: TPS7A5201RPSR, JLCImport:TPS7A5201RPSR, symbol JLCImport:TPS7A5201RPSR
- added C34, C37, C38, C41: 22uF, GPSDO_Rev1.0:C_0805_2012Metric, symbol GPSDO_Rev1.0:C
- added C35, C39: 100nF, GPSDO_Rev1.0:C_0402_1005Metric, symbol GPSDO_Rev1.0:C
- added C36, C40: 10nF, GPSDO_Rev1.0:C_0402_1005Metric, symbol GPSDO_Rev1.0:C
- added R26, R32: 12.1K, GPSDO_Rev1.0:R_0402_1005Metric, symbol GPSDO_Rev1.0:R
- added R27, R31: 100K, GPSDO_Rev1.0:R_0402_1005Metric, symbol GPSDO_Rev1.0:R
- added R30, R33: 3.87K, GPSDO_Rev1.0:R_0402_1005Metric, symbol GPSDO_Rev1.0:R
- added U14, U16: TPS7A5201RPSR, GPSDO_Rev1.0:TPS7A5201RPSR, symbol GPSDO_Rev1.0:TPS7A5201RPSR
- CN1: footprint JLCImport:LAIL-PHC2_54-2P-01-XH-L -> GPSDO_Rev1.0:LAIL-PHC2_54-2P-01-XH-L
Connections:
- net +3.3V: now also C36.1, C37.1, R26.1, R27.1, U14.10 (OUT), U14.11 (OUT)
- net +5V: now also C34.1, C38.1, U14.1 (IN), U14.2 (IN), U14.3 (EN), U16.1 (IN), U16.2 (IN), U16.3 (EN)
- net 3.3V_OCXO: now also C40.1, C41.1, R31.1, R32.1, U16.10 (OUT), U16.11 (OUT)
- net GND: now also C34.2, C35.2, C37.2, C38.2, C39.2, C41.2, R30.2, R33.2, U14.12 (GND), U14.5 (BIAS), U14.6 (GND), U14.7 (GND), U16.12 (GND), U16.5 (BIAS), U16.6 (GND), U16.7 (GND)
- net LDO_3V3_FB: now also C36.2, R26.2, R30.1, U14.9 (FB)
- net LDO_3V3_NR: now also C35.1, U14.4 (NR/SS)
- net LDO_OCXO_FB: now also C40.2, R32.2, R33.1, U16.9 (FB)
- net LDO_OCXO_NR: now also C39.1, U16.4 (NR/SS)
- net LDO_OCXO_PG: now also R31.2, U16.8 (PG)
- net PDN: now also R27.2, U14.8 (PG)
Other:
- note added: "U3 TPS7A52 5V -> 3.3V 给整体供电"
- note removed: "U3 TPS7A52 5V -> 3.3V 给LMK5B12204供电"

Commit message: sch update
Parts:
- removed D5: LED, LED_SMD:LED_0603_1608Metric, symbol Device:LED
- added C23: TAJB107M010RNJ, JLCImport:TAJB107M010RNJ, symbol JLCImport:TAJB107M010RNJ
- added C25: 10uF, GPSDO_Rev1.0:C_0603_1608Metric, symbol GPSDO_Rev1.0:C
- added C43: 100nF, GPSDO_Rev1.0:C_0402_1005Metric, symbol GPSDO_Rev1.0:C
- added D1, D2: LED, GPSDO_Rev1.0:LED_0603_1608Metric, symbol GPSDO_Rev1.0:LED
- added R22, R23: 0, GPSDO_Rev1.0:R_0805_2012Metric, symbol GPSDO_Rev1.0:R
Connections:
- net +3.3V: now also D1.2 (A)
- net +5V: now also C25.1, C43.1, R22.2
- net 3.3V_OCXO: now also R23.1
- net GND: now also C23.2, C25.2, C43.2, D1.1 (K), D2.1 (K)
- new net OCXO_VCC: C23.1, D2.2 (A), R22.1, R23.2
Other:
- note added: "OCXO 供电选配 (二者互斥, 严禁同装):"
- note added: "装 R19 = 5V OCXO 直供 / 装 R20 = 3.3V OCXO 经 U4 稳压"
- moved on the sheet: C34, C35, C36, C37, C38, C39, C40, C41, R26, R27, R30, R31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

Commit message: sch update
Other:
- moved on the sheet: CN1
Changed lines of the file:
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@@
 	(text "装 R19 = 5V OCXO 直供   /   装 R20 = 3.3V OCXO 经 U4 稳压"
 		(exclude_from_sim no)
-		(at 209.55 51.44 0)
+		(at 211.328 54.356 0)
 		(effects
 			(font
@@
 	(text "OCXO 供电选配 (二者互斥, 严禁同装):"
 		(exclude_from_sim no)
-		(at 209.55 48.26 0)
+		(at 211.328 51.176 0)
 		(effects
 			(font
@@
 	(symbol
 		(lib_id "GPSDO_Rev1.0:LAIL-PHC2_54-2P-01-XH-L")
-		(at 52.07 85.09 0)
+		(at 44.45 64.77 0)
 		(mirror y)
 		(unit 1)
@@
 		(dnp no)
 		(property "Reference" "CN1"
-			(at 53.594 78.74 0)
+			(at 45.974 58.42 0)
 			(show_name no)
 			(do_not_autoplace no)
@@
 		)
 		(property "Value" "LAIL-PHC2_54-2P-01-XH-L"
-			(at 59.944 92.964 0)
+			(at 52.324 72.644 0)
 			(show_name no)
 			(do_not_autoplace no)
@@
 		)
 		(property "Footprint" "GPSDO_Rev1.0:LAIL-PHC2_54-2P-01-XH-L"
-			(at 52.07 85.09 0)
+			(at 44.45 64.77 0)
 			(hide yes)
 			(show_name no)
@@
 		)
 		(property "Datasheet" "https://atta.szlcsc.com/upload/public/pdf/source/20230105/4FFD2EFD3DA44AA828171A44400F3EDE.pdf"
-			(at 52.07 85.09 0)
+			(at 44.45 64.77 0)
 			(hide yes)
 			(show_name no)
@@
 		)
 		(property "Description" "-25℃~+85℃ 1 1x2P 2 2.54mm 250V 2P 3A 5.8mm 7.1mm 7.5mm Brass PA66 Through Hole Tin UL94V-0 White XH Plugin,P=2.5mm Wire To Board Connector ROHS"
-			(at 52.07 85.09 0)
+			(at 44.45 64.77 0)
 			(hide yes)
 			(show_name no)
@@
 		)
 		(property "LCSC" "C54905973"
-			(at 52.07 85.09 0)
+			(at 44.45 64.77 0)
 			(hide yes)
 			(show_name no)
@@
 		)
 		(property "Manufacturer" "LAILAN"
-			(at 52.07 85.09 0)
+			(at 44.45 64.77 0)
 			(hide yes)
 			(show_name no)
@@
 		)
 		(property "Manufacturer Part" "LAIL-PHC2.54-2P-01-XH-L"
-			(at 52.07 85.09 0)
+			(at 44.45 64.77 0)
 			(hide yes)
 			(show_name no)

Commit message: sch update
Parts:
- added C26: 10uF, GPSDO_Rev1.0:C_0603_1608Metric, symbol GPSDO_Rev1.0:C
- added C46: 100nF, GPSDO_Rev1.0:C_0402_1005Metric, symbol GPSDO_Rev1.0:C
- added D8: LED, GPSDO_Rev1.0:LED_0603_1608Metric, symbol GPSDO_Rev1.0:LED
- added F1: BSMD1206C-1300T, JLCImport:BSMD1206C-1300T, symbol JLCImport:BSMD1206C-1300T
Connections:
- net +5V: now also C26.1, C46.1, D8.2 (A), F1.2
- net GND: now also CN1.2, C26.2, C46.2, D8.1 (K)
- net +5V_IN: now reaches CN1.1
- net +5V_IN: now also F1.1
Other:
- moved on the sheet: CN1

Commit message: sch update
Parts:
- added C59, C64, C65: 10uF / 16V, Capacitor_SMD:C_0805_2012Metric, symbol GPSDO_Rev1.0:C
- added C60: 100nF, Capacitor_SMD:C_0603_1608Metric, symbol GPSDO_Rev1.0:C
- added C61: 4.7nF, Capacitor_SMD:C_0603_1608Metric, symbol GPSDO_Rev1.0:C
- added C62: 22uF / 16V, Capacitor_SMD:C_1210_3225Metric, symbol GPSDO_Rev1.0:C
- added C63: 220nF, Capacitor_SMD:C_0603_1608Metric, symbol GPSDO_Rev1.0:C
- added C66, C67: 10nF, Capacitor_SMD:C_0603_1608Metric, symbol GPSDO_Rev1.0:C
- added D9: SS14, Diode_SMD:D_SMA, symbol GPSDO_Rev1.0:D_Schottky
- added L2: 4.7uH, Inductor_SMD:L_Coilcraft_LPS4018, symbol GPSDO_Rev1.0:L
- added R38: 10R, Resistor_SMD:R_0603_1608Metric, symbol GPSDO_Rev1.0:R
- added R39: 715K, Resistor_SMD:R_0603_1608Metric, symbol GPSDO_Rev1.0:R
- added R40: 150K, Resistor_SMD:R_0603_1608Metric, symbol GPSDO_Rev1.0:R
- added R41: 32.4K, Resistor_SMD:R_0603_1608Metric, symbol GPSDO_Rev1.0:R
- added R42: 10K, Resistor_SMD:R_0603_1608Metric, symbol GPSDO_Rev1.0:R
- added U13: TPS7A3001DGNR, GPSDO_Rev1.0:TPS7A3001DGNR, symbol GPSDO_Rev1.0:TPS7A3001DGNR
- added U17: TPS63700, GPSDO_Rev1.0:TPS63700, symbol GPSDO_Rev1.0:TPS63700
Connections:
- net +5V: now also C59.1, R38.1, U17.4 (EN), U17.5 (IN)
- net GND: now also C59.2, C60.2, C61.2, C62.2, C63.1, C64.2, C65.2, C67.2, L2.1, R42.2, U13.4 (GND), U13.9 (EP), U17.11 (PP), U17.2 (GND), U17.7 (PS_GND)
- new net: D9.1 (K), L2.2, U17.6 (SW)
- new net: C61.1, U17.1 (COMP)
- new net: C66.2, R41.2, R42.1, U13.2 (FB)
- new net: C67.1, U13.6 (NRSS)
- new net -5V: C65.1, C66.1, R41.1, U13.1 (OUT)
- new net -5V8_RAW: C62.1, C64.1, D9.2 (A), R39.1, U13.5 (EN), U13.8 (IN), U17.8 (OUT)
- new net N5_FB: R39.2, R40.1, U17.9 (FB)
- new net N5_REF1V213: C63.2, R40.2, U17.10 (VREF)
- new net N5_VIN_RC: C60.1, R38.2, U17.3 (VIN)
- no-connect marks 0 -> 2
Other:
- note added: "D: cathode (bar) -> SW; anode -> RAW"
- note added: "Design target: 100mA; verify ripple / load transient on prototype."
- note added: "EN -> IN; DNC open; EP -> GND"
- note added: "LDO divider: 32.4K / 10K -> approx. -5V"
- note added: "Negative supply for 2 x BUF602: +5V -> -5.8V RAW -> -5V"
- moved on the sheet: C23, C25, C26, C34, C35, C36, C37, C38, C39, C40, C41, C43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

Commit message: sch update
Parts:
- removed C59, C64, C65: 10uF / 16V, Capacitor_SMD:C_0805_2012Metric, symbol GPSDO_Rev1.0:C
- removed C60: 100nF, Capacitor_SMD:C_0603_1608Metric, symbol GPSDO_Rev1.0:C
- removed C61: 4.7nF, Capacitor_SMD:C_0603_1608Metric, symbol GPSDO_Rev1.0:C
- removed C62: 22uF / 16V, Capacitor_SMD:C_1210_3225Metric, symbol GPSDO_Rev1.0:C
- removed C63: 220nF, Capacitor_SMD:C_0603_1608Metric, symbol GPSDO_Rev1.0:C
- removed C66, C67: 10nF, Capacitor_SMD:C_0603_1608Metric, symbol GPSDO_Rev1.0:C
- removed D9: SS14, Diode_SMD:D_SMA, symbol GPSDO_Rev1.0:D_Schottky
- removed L2: 4.7uH, Inductor_SMD:L_Coilcraft_LPS4018, symbol GPSDO_Rev1.0:L
- removed R38: 10R, Resistor_SMD:R_0603_1608Metric, symbol GPSDO_Rev1.0:R
- removed R39: 715K, Resistor_SMD:R_0603_1608Metric, symbol GPSDO_Rev1.0:R
- removed R40: 150K, Resistor_SMD:R_0603_1608Metric, symbol GPSDO_Rev1.0:R
- removed R41: 32.4K, Resistor_SMD:R_0603_1608Metric, symbol GPSDO_Rev1.0:R
- removed R42: 10K, Resistor_SMD:R_0603_1608Metric, symbol GPSDO_Rev1.0:R
- removed U13: TPS7A3001DGNR, GPSDO_Rev1.0:TPS7A3001DGNR, symbol GPSDO_Rev1.0:TPS7A3001DGNR
- removed U17: TPS63700, GPSDO_Rev1.0:TPS63700, symbol GPSDO_Rev1.0:TPS63700
- C23: footprint JLCImport:TAJB107M010RNJ -> GPSDO_Rev1.0:TAJB107M010RNJ; symbol JLCImport:TAJB107M010RNJ -> GPSDO_Rev1.0:TAJB107M010RNJ
- C34, C37, C38, C41: symbol GPSDO_Rev1.0:C -> GPSDO_Rev1.0:C__C_0805_2012Metric
- C35, C36, C39, C40, C43, C46: symbol GPSDO_Rev1.0:C -> GPSDO_Rev1.0:C__C_0402_1005Metric
- F1: footprint JLCImport:BSMD1206C-1300T -> GPSDO_Rev1.0:BSMD1206C-1300T; symbol JLCImport:BSMD1206C-1300T -> GPSDO_Rev1.0:BSMD1206C-1300T
- R22, R23: symbol GPSDO_Rev1.0:R -> GPSDO_Rev1.0:R__R_0805_2012Metric
- R26, R27, R30, R31, R32, R33: symbol GPSDO_Rev1.0:R -> GPSDO_Rev1.0:R__R_0402_1005Metric
Connections:
- no-connect marks 2 -> 0
Other:
- note added: "-5V generator removed. TODO: U4 / U12 (BUF602) need a single-supply driver redesign."
- note removed: "D: cathode (bar) -> SW; anode -> RAW"
- note removed: "Design target: 100mA; verify ripple / load transient on prototype."
- note removed: "EN -> IN; DNC open; EP -> GND"
- note removed: "LDO divider: 32.4K / 10K -> approx. -5V"
- note removed: "Negative supply for 2 x BUF602: +5V -> -5.8V RAW -> -5V"

Commit message: sch update
Parts:
- removed C26: 10uF, GPSDO_Rev1.0:C_0603_1608Metric, symbol GPSDO_Rev1.0:C
- removed C46: 100nF, GPSDO_Rev1.0:C_0402_1005Metric, symbol GPSDO_Rev1.0:C__C_0402_1005Metric
- added C68, C69: 1uF / 16V, GPSDO_Rev1.0:C_0603_1608Metric, symbol GPSDO_Rev1.0:C
- added C70: 100nF / 16V, GPSDO_Rev1.0:C_0402_1005Metric, symbol GPSDO_Rev1.0:C__C_0402_1005Metric
- added C71: 22uF / 10V, GPSDO_Rev1.0:C_0805_2012Metric, symbol GPSDO_Rev1.0:C__C_0805_2012Metric
- added R43: 30.1K 1%, GPSDO_Rev1.0:R_0402_1005Metric, symbol GPSDO_Rev1.0:R__R_0402_1005Metric
- added R44: 10K 1%, GPSDO_Rev1.0:R_0402_1005Metric, symbol GPSDO_Rev1.0:R__R_0402_1005Metric
- added R45: 1K, GPSDO_Rev1.0:R_0402_1005Metric, symbol GPSDO_Rev1.0:R__R_0402_1005Metric
- added U18: TPS2116DRLR, GPSDO_Rev1.0:SOT-583-8, symbol GPSDO_Rev1.0:TPS2116DRL
Connections:
- net +5V: now also C70.1, C71.1, R45.1, U18.2 (VOUT), U18.7 (VOUT); no longer D8.2 (A), F1.2
- net GND: now also C68.2, C69.2, C70.2, C71.2, R44.2, U18.1 (GND)
- new net: D8.2 (A), R45.2
- new net EXT_5V: C68.1, F1.2, R43.1, U18.3 (VIN1), U18.5 (MODE)
- new net MUX_PR1: R43.2, R44.1, U18.4 (PR1)
- new net VBUS: C69.1, U18.6 (VIN2)
- no-connect marks 0 -> 1
Other:
- note added: "5V source selection: CN1 (priority) / USB VBUS -> +5V"
- note added: "CC resistors alone do not authorize high-current draw from a PC."
- note added: "Check 5V dip on source change under maximum load."
- note added: "Inputs: regulated 5V only (max 5.5V). Total mux current <= 2.5A."
- note added: "No over-current limit in U18; upstream source protection required."
- note added: "PR1 threshold: 4.01V typ. (IC reference +/-8%; not precision UVLO)."
- note added: "USB source must cover OCXO warm-up + full board load."
- note added: "VIN1: EXT_5V after F1. VIN2: USB VBUS. MODE -> VIN1."
- moved on the sheet: D8

Commit message: sch update
Connections:
- net PDN: no longer names the net of R27.2, U14.8 (PG)
Changed lines of the file:
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@@
 	)
 	(junction
-		(at 135.89 147.32)
-		(diameter 0)
-		(color 0 0 0 0)
-	)
-	(junction
 		(at 113.03 46.99)
 		(diameter 0)
@@
 	)
 	(junction
-		(at 143.51 62.23)
+		(at 233.68 91.44)
 		(diameter 0)
 		(color 0 0 0 0)
@@
 	)
 	(junction
+		(at 135.89 147.32)
+		(diameter 0)
+		(color 0 0 0 0)
+	)
+	(junction
 		(at 113.03 85.09)
 		(diameter 0)
@@
 	(wire
 		(pts
+			(xy 146.05 147.32) (xy 146.05 144.78)
+		)
+		(stroke
+			(width 0)
+			(type default)
+		)
+	)
+	(wire
+		(pts
 			(xy 234.95 36.83) (xy 241.3 36.83)
 		)
@@
 	(wire
 		(pts
-			(xy 241.3 76.2) (xy 241.3 80.01)
+			(xy 241.3 76.2) (xy 241.3 91.44)
 		)
 		(stroke
@@
 	(wire
 		(pts
+			(xy 233.68 91.44) (xy 241.3 91.44)
+		)
+		(stroke
+			(width 0)
+			(type default)
+		)
+	)
+	(wire
+		(pts
 			(xy 96.52 162.56) (xy 96.52 166.37)
 		)
@@
 	(wire
 		(pts
+			(xy 229.87 91.44) (xy 233.68 91.44)
+		)
+		(stroke
+			(width 0)
+			(type default)
+		)
+	)
+	(wire
+		(pts
 			(xy 138.43 46.99) (xy 140.97 46.99)
 		)
@@
 	(wire
 		(pts
-			(xy 140.97 62.23) (xy 143.51 62.23)
-		)
-		(stroke
-			(width 0)
-			(type default)
-		)
-	)
-	(wire
-		(pts
 			(xy 143.51 87.63) (xy 149.86 87.63)
 		)
@@
 		)
 	)
-	(hierarchical_label "PDN"
-		(shape output)
-		(at 140.97 62.23 180)
-		(effects
-			(font
-				(size 1.27 1.27)
-			)
-			(justify right)
-		)
-	)
-	(hierarchical_label "OCXO_VCC"
-		(shape output)
-		(at 241.3 80.01 270)
-		(effects
-			(font
-				(size 1.27 1.27)
-			)
-			(justify right)
-		)
-	)
 	(symbol
 		(lib_id "GPSDO_Rev1.0:GND")
@@
 	)
 	(symbol
+		(lib_id "GPSDO_Rev1.0:VDDA")
+		(at 233.68 91.44 0)
+		(unit 1)
+		(body_style 1)
+		(exclude_from_sim no)
+		(in_bom yes)
+		(on_board yes)
+		(in_pos_files yes)
+		(dnp no)
+		(fields_autoplaced yes)
+		(property "Reference" "#PWR057"
+			(at 233.68 95.25 0)
+			(hide yes)
+			(show_name no)
+			(do_not_autoplace no)
+			(effects
+				(font
+					(size 1.27 1.27)
+				)
+			)
+		)
+		(property "Value" "OCXO_VCC"
+			(at 233.68 86.36 0)
+			(show_name no)
+			(do_not_autoplace no)
+			(effects
+				(font
+					(size 1.27 1.27)
+				)
+			)
+		)
+		(property "Footprint" ""
+			(at 233.68 91.44 0)
+			(hide yes)
+			(show_name no)
+			(do_not_autoplace no)
+			(effects
+				(font
+					(size 1.27 1.27)
+				)
+			)
+		)
+		(property "Datasheet" ""
+			(at 233.68 91.44 0)
+			(hide yes)
+			(show_name no)
+			(do_not_autoplace no)
+			(effects
+				(font
+					(size 1.27 1.27)
+				)
+			)
+		)
+		(property "Description" "Power symbol creates a global label with name \"VDDA\""
+			(at 233.68 91.44 0)
+			(hide yes)
+			(show_name no)
+			(do_not_autoplace no)
+			(effects
+				(font
+					(size 1.27 1.27)
+				)
+			)
+		)
+		(pin "1"
+		)
+		(instances
+			(project "GPSDO_Rev1.0"
+				(path "/7fcb1340-2836-48b1-8b47-374fa7e6ca96/e383764a-0b62-4980-895b-607aaa53a70d"
+					(reference "#PWR057")
+					(unit 1)
+				)
+			)
+		)
+	)
+	(symbol
 		(lib_id "GPSDO_Rev1.0:GND")
 		(at 120.65 162.56 0)
@@
 	(symbol
 		(lib_id "GPSDO_Rev1.0:+5V")
-		(at 146.05 147.32 0)
+		(at 146.05 144.78 0)
 		(unit 1)
 		(body_style 1)
@@
 		(dnp no)
 		(property "Reference" "#PWR174"
-			(at 148.05 145.82 0)
+			(at 148.05 143.28 0)
 			(hide yes)
 			(show_name no)
@@
 		)
 		(property "Value" "+5V"
-			(at 146.05 144.32 0)
+			(at 146.05 141.224 0)
 			(show_name no)
 			(do_not_autoplace no)
@@
 		)
 		(property "Footprint" ""
-			(at 146.05 147.32 0)
+			(at 146.05 144.78 0)
 			(hide yes)
 			(show_name no)
@@
 		)
 		(property "Datasheet" ""
-			(at 146.05 147.32 0)
+			(at 146.05 144.78 0)
 			(hide yes)
 			(show_name no)
@@
 		)
 		(property "Description" ""
-			(at 146.05 147.32 0)
+			(at 146.05 144.78 0)
 			(hide yes)
 			(show_name no)
@@
 					(unit 1)
 				)
+			)
+		)
+	)
+	(symbol
+		(lib_id "power:PWR_FLAG")
+		(at 229.87 91.44 90)
+		(unit 1)
+		(body_style 1)
+		(exclude_from_sim no)
+		(in_bom yes)
+		(on_board yes)
+		(in_pos_files yes)
+		(dnp no)
+		(fields_autoplaced yes)
+		(property "Reference" "#FLG04"
+			(at 227.965 91.44 0)
+			(hide yes)
+			(show_name no)
+			(do_not_autoplace no)
+			(effects
+				(font
+					(size 1.27 1.27)
+				)
+			)
+		)
+		(property "Value" "PWR_FLAG"
+			(at 226.06 91.4399 90)
+			(show_name no)
+			(do_not_autoplace no)
+			(effects
+				(font
+					(size 1.27 1.27)
+				)
+				(justify left)
+			)
+		)
+		(property "Footprint" ""
+			(at 229.87 91.44 0)
+			(hide yes)
+			(show_name no)
+			(do_not_autoplace no)
+			(effects
+				(font
+					(size 1.27 1.27)
+				)
+			)
+		)
+		(property "Datasheet" ""
+			(at 229.87 91.44 0)
+			(hide yes)
+			(show_name no)
+			(do_not_autoplace no)
+			(effects
+				(font
+					(size 1.27 1.27)
+				)
+			)
+		)
+		(property "Description" "Special symbol for telling ERC where power comes from"
+			(at 229.87 91.44 0)
+			(hide yes)
+			(show_name no)
+			(do_not_autoplace no)
+			(effects
+				(font
+					(size 1.27 1.27)
+				)
+			)
+		)
+		(pin "1"
+		)
+		(instances
+			(project "GPSDO_Rev1.0"
+				(path "/7fcb1340-2836-48b1-8b47-374fa7e6ca96/e383764a-0b62-4980-895b-607aaa53a70d"
+					(reference "#FLG04")
+					(unit 1)
+				)
