File: hardware/schematic/v1.0/GPSDO_Rev1.0/POWER.kicad_sch (KiCad schematic)
At the start: 34 parts, among them CN1 LAIL-PHC2_54-2P-01-XH-L, U14 TPS7A5201RPSR, U16 TPS7A5201RPSR, U18 TPS2116DRLR

Commit message: sch update
Parts:
- added C72: 10uF / 10V, GPSDO_Rev1.0:C_0603_1608Metric, symbol GPSDO_Rev1.0:C
- added C73: 100nF, GPSDO_Rev1.0:C_0402_1005Metric, symbol GPSDO_Rev1.0:C__C_0402_1005Metric
- added C74, C75: 22uF / 10V, GPSDO_Rev1.0:C_0805_2012Metric, symbol GPSDO_Rev1.0:C__C_0805_2012Metric
- added L2: 1uH / DFE201610P, GPSDO_Rev1.0:L_Murata_DFE201610P, symbol GPSDO_Rev1.0:L__L_Murata_DFE201610P
- added R49: 1K, GPSDO_Rev1.0:R_0402_1005Metric, symbol GPSDO_Rev1.0:R__R_0402_1005Metric
- added R50: 10K, GPSDO_Rev1.0:R_0402_1005Metric, symbol GPSDO_Rev1.0:R__R_0402_1005Metric
- added R51: 77.4K 0.1%, GPSDO_Rev1.0:R_0402_1005Metric, symbol GPSDO_Rev1.0:R__R_0402_1005Metric
- added R52: 10K 0.1%, GPSDO_Rev1.0:R_0402_1005Metric, symbol GPSDO_Rev1.0:R__R_0402_1005Metric
- added U4: TPS61023DRLR, GPSDO_Rev1.0:TPS61023DRLR, symbol GPSDO_Rev1.0:TPS61023DRLR
Connections:
- net +3.3V: now also C72.1, C73.1, L2.1, U4.3 (VIN)
- net GND: now also C72.2, C73.2, C74.2, C75.2, R50.2, R52.2, U4.4 (GND)
- new net: R49.2, R50.1, U4.2 (EN)
- new net: L2.2, U4.5 (SW)
- new net +5V2: C74.1, C75.1, R51.1, U4.6 (VOUT)
- new net BOOST_EN: R49.1
- new net BOOST_FB: R51.2, R52.1, U4.1 (FB)
Other:
- note added: "0.595 x (1 + 77.4K/10K) = 5.200V"
- note added: "3.3V -> 5.2V / ISL55110 VH"
- note added: "EN: PB0; LOW during MCU reset"
- note added: "Target 200mA; check ripple / startup"
- note removed: "-5V generator removed. TODO: U4 / U12 (BUF602) need a single-supply driver redesign."

Commit message: sch update
Parts:
- added R34, R53: 2.2K, GPSDO_Rev1.0:R_0402_1005Metric, symbol GPSDO_Rev1.0:R__R_0402_1005Metric
Connections:
- net +3.3V: now also R53.1; no longer D1.2 (A)
- net OCXO_VCC: now also R34.2; no longer D2.2 (A)
- new net: D1.2 (A), R53.2
- new net: D2.2 (A), R34.1
