File: hardware/schematic/v1.0/GPSDO_Rev1.0/GNSS.kicad_sch (KiCad schematic)
At the start: 5 parts, among them U6 NEO-M8T-0

Commit message: sch update
Connections:
- no-connect marks 11 -> 13
Changed lines of the file:
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@@
+	)
+	(no_connect
+		(at 114.3 82.55)
 	)
 	(no_connect
@@
 	)
 	(no_connect
+		(at 114.3 80.01)
+	)
+	(no_connect

Commit message: sch update
Parts:
- added C6, C8: 1uF, GPSDO_Rev1.0:C_0603_1608Metric, symbol GPSDO_Rev1.0:C
- added C7: 100nF, GPSDO_Rev1.0:C_0402_1005Metric, symbol GPSDO_Rev1.0:C
- added L1: 33nH, GPSDO_Rev1.0:L_0402_1005Metric, symbol GPSDO_Rev1.0:L
- added R8: 100K, GPSDO_Rev1.0:R_0402_1005Metric, symbol GPSDO_Rev1.0:R
- added R9: 470, GPSDO_Rev1.0:R_0402_1005Metric, symbol GPSDO_Rev1.0:R
Connections:
- net GND: now also C6.2, C7.2, C8.2, R8.1
- net VCC_RF: now also L1.2
- net at RF1.4 (SIG), U6.11 (RF_IN): now also L1.1
- net at U6.22 (V_BCKP): now also C8.1, R9.1
- net +3.3V: now reaches U6.23 (VCC)
- net +3.3V: now also C6.1, C7.1, R9.2
- net at U6.7 (VDD_USB): now also R8.2
- no-connect marks 13 -> 12

Commit message: sch update
Parts:
- added FB8: 100R, GPSDO_Rev1.0:L_0603_1608Metric, symbol GPSDO_Rev1.0:FerriteBead_Small
Connections:
- net +3.3V: now also FB8.1; no longer C6.1, C7.1, U6.23 (VCC)
- new net: C6.1, C7.1, FB8.2, U6.23 (VCC)
Changed lines of the file:
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@@
+	(wire
+		(pts
+			(xy 190.5 50.8) (xy 190.5 52.07)
+		)
+		(stroke
+			(width 0)
+			(type default)
+		)
+	)
 	(wire
 		(pts
@@
 	(wire
 		(pts
-			(xy 190.5 55.88) (xy 190.5 59.69)
+			(xy 190.5 57.15) (xy 190.5 59.69)
 		)
 		(stroke
@@
 	(symbol
 		(lib_id "power:+3.3V")
-		(at 190.5 55.88 0)
+		(at 190.5 50.8 0)
 		(unit 1)
 		(body_style 1)
@@
 		(fields_autoplaced yes)
 		(property "Reference" "#PWR012"
-			(at 190.5 59.69 0)
+			(at 190.5 54.61 0)
 			(hide yes)
 			(show_name no)
@@
 		)
 		(property "Value" "+3.3V"
+			(at 190.5 45.72 0)
+			(show_name no)
+			(do_not_autoplace no)
+			(effects
+				(font
+					(size 1.27 1.27)
+				)
+			)
+		)
+		(property "Footprint" ""
 			(at 190.5 50.8 0)
-			(show_name no)
-			(do_not_autoplace no)
-			(effects
-				(font
-					(size 1.27 1.27)
-				)
-			)
-		)
-		(property "Footprint" ""
-			(at 190.5 55.88 0)
 			(hide yes)
 			(show_name no)
@@
 		)
 		(property "Datasheet" ""
-			(at 190.5 55.88 0)
+			(at 190.5 50.8 0)
 			(hide yes)
 			(show_name no)
@@
 		)
 		(property "Description" "Power symbol creates a global label with name \"+3.3V\""
-			(at 190.5 55.88 0)
+			(at 190.5 50.8 0)
 			(hide yes)
 			(show_name no)
@@
 					(unit 1)
 				)
+			)
+		)
+	)
+	(symbol
+		(lib_id "GPSDO_Rev1.0:FerriteBead_Small")
+		(at 190.5 54.61 0)
+		(unit 1)
+		(body_style 1)
+		(exclude_from_sim no)
+		(in_bom yes)
+		(on_board yes)
+		(in_pos_files yes)
+		(dnp no)
+		(property "Reference" "FB8"
+			(at 194.31 53.594 0)
+			(show_name no)
+			(do_not_autoplace no)
+			(effects
+				(font
+					(size 1.27 1.27)
+				)
+			)
+		)
+		(property "Value" "100R"
+			(at 194.818 56.896 0)
+			(show_name no)
+			(do_not_autoplace no)
+			(effects
+				(font
+					(size 1.27 1.27)
+				)
+			)
+		)
+		(property "Footprint" "GPSDO_Rev1.0:L_0603_1608Metric"
+			(at 188.722 54.61 90)
+			(hide yes)
+			(show_name no)
+			(do_not_autoplace no)
+			(effects
+				(font
+					(size 1.27 1.27)
+				)
+			)
+		)
+		(property "Datasheet" ""
+			(at 190.5 54.61 0)
+			(hide yes)
+			(show_name no)
+			(do_not_autoplace no)
+			(effects
+				(font
+					(size 1.27 1.27)
+				)
+			)
+		)
+		(property "Description" "Ferrite bead, small symbol"
+			(at 190.5 54.61 0)
+			(hide yes)
+			(show_name no)
+			(do_not_autoplace no)
+			(effects
+				(font
+					(size 1.27 1.27)
+				)
+			)
+		)
+		(pin "2"
+		)
+		(pin "1"
+		)
+		(instances
+			(project "GPSDO_Rev1.0"
+				(path "/7fcb1340-2836-48b1-8b47-374fa7e6ca96/73734292-4707-44de-b5e5-87f3016d7c18"
+					(reference "FB8")
+					(unit 1)
+				)

Commit message: sch update
Parts:
- R1: value 100 -> 0
Connections:
- net 1PPS renamed PULSE_GNSS
- net RXD renamed GNSS_UART_RXD
- net TXD renamed GNSS_UART_TXD
Changed lines of the file:
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@@
 	(wire
 		(pts
-			(xy 97.79 77.47) (xy 101.6 77.47)
+			(xy 100.33 77.47) (xy 101.6 77.47)
 		)
 		(stroke
@@
 	(wire
 		(pts
-			(xy 97.79 74.93) (xy 101.6 74.93)
+			(xy 100.33 74.93) (xy 101.6 74.93)
 		)
 		(stroke
@@
 		)
 	)
-	(hierarchical_label "RXD"
-		(shape output)
-		(at 97.79 77.47 180)
+	(hierarchical_label "GNSS_UART_RXD"
+		(shape input)
+		(at 100.33 77.47 180)
 		(effects
 			(font
@@
 		)
 	)
-	(hierarchical_label "TXD"
+	(hierarchical_label "GNSS_UART_TXD"
 		(shape output)
-		(at 97.79 74.93 180)
+		(at 100.33 74.93 180)
 		(effects
 			(font
@@
 		)
 	)
-	(hierarchical_label "1PPS"
+	(hierarchical_label "PULSE_GNSS"
 		(shape output)
 		(at 182.88 72.39 0)
@@
 			)
 		)
-		(property "Value" "100"
+		(property "Value" "0"
 			(at 177.038 70.104 90)
 			(show_name no)

Commit message: sch update
Parts:
- C7: symbol GPSDO_Rev1.0:C -> GPSDO_Rev1.0:C__C_0402_1005Metric
- L1: symbol GPSDO_Rev1.0:L -> GPSDO_Rev1.0:L__L_0402_1005Metric
- R1, R2, R3, R8, R9: symbol GPSDO_Rev1.0:R -> GPSDO_Rev1.0:R__R_0402_1005Metric
Changed lines of the file:
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@@
 	)
 	(symbol
-		(lib_id "GPSDO_Rev1.0:R")
+		(lib_id "GPSDO_Rev1.0:R__R_0402_1005Metric")
 		(at 182.88 90.17 90)
 		(unit 1)
@@
 	)
 	(symbol
-		(lib_id "GPSDO_Rev1.0:C")
+		(lib_id "GPSDO_Rev1.0:C__C_0402_1005Metric")
 		(at 175.26 54.61 180)
 		(unit 1)
@@
 	)
 	(symbol
-		(lib_id "power:GND")
+		(lib_id "GPSDO_Rev1.0:GND")
 		(at 167.64 106.68 0)
 		(unit 1)
@@
 	)
 	(symbol
-		(lib_id "GPSDO_Rev1.0:R")
+		(lib_id "GPSDO_Rev1.0:R__R_0402_1005Metric")
 		(at 175.26 64.77 270)
 		(unit 1)
@@
 	)
 	(symbol
-		(lib_id "power:GND")
+		(lib_id "GPSDO_Rev1.0:GND")
 		(at 175.26 50.8 180)
 		(unit 1)
@@
 	)
 	(symbol
-		(lib_id "power:+3.3V")
+		(lib_id "GPSDO_Rev1.0:+3.3V")
 		(at 190.5 86.36 0)
 		(unit 1)
@@
 	)
 	(symbol
-		(lib_id "power:GND")
+		(lib_id "GPSDO_Rev1.0:GND")
 		(at 184.15 50.8 180)
 		(unit 1)
@@
 	)
 	(symbol
-		(lib_id "power:GND")
+		(lib_id "GPSDO_Rev1.0:GND")
 		(at 59.69 82.55 0)
 		(unit 1)
@@
 	)
 	(symbol
-		(lib_id "power:GND")
+		(lib_id "GPSDO_Rev1.0:GND")
 		(at 59.69 57.15 180)
 		(unit 1)
@@
 	)
 	(symbol
-		(lib_id "GPSDO_Rev1.0:R")
+		(lib_id "GPSDO_Rev1.0:R__R_0402_1005Metric")
 		(at 175.26 72.39 90)
 		(unit 1)
@@
 	)
 	(symbol
-		(lib_id "power:+3.3V")
+		(lib_id "GPSDO_Rev1.0:+3.3V")
 		(at 190.5 50.8 0)
 		(unit 1)
@@
 	)
 	(symbol
-		(lib_id "GPSDO_Rev1.0:L")
+		(lib_id "GPSDO_Rev1.0:L__L_0402_1005Metric")
 		(at 74.93 77.47 0)
 		(unit 1)
@@
 	)
 	(symbol
-		(lib_id "GPSDO_Rev1.0:R")
+		(lib_id "GPSDO_Rev1.0:R__R_0402_1005Metric")
 		(at 105.41 74.93 90)
 		(unit 1)
@@
 	)
 	(symbol
-		(lib_id "power:GND")
+		(lib_id "GPSDO_Rev1.0:GND")
 		(at 180.34 64.77 90)
 		(unit 1)
@@
 	)
 	(symbol
-		(lib_id "power:GND")
+		(lib_id "GPSDO_Rev1.0:GND")
 		(at 175.26 99.06 0)
 		(unit 1)
@@
 	)
 	(symbol
-		(lib_id "power:GND")
+		(lib_id "GPSDO_Rev1.0:GND")
 		(at 46.99 69.85 270)
 		(unit 1)
@@
 	)
 	(symbol
-		(lib_id "GPSDO_Rev1.0:R")
+		(lib_id "GPSDO_Rev1.0:R__R_0402_1005Metric")
 		(at 105.41 77.47 270)
 		(unit 1)

Commit message: sch update
Changed lines of the file:
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@@
 	(wire
 		(pts
-			(xy 167.64 62.23) (xy 180.34 62.23)
+			(xy 167.64 62.23) (xy 172.72 62.23)
 		)
 		(stroke
@@
 	(wire
 		(pts
-			(xy 74.93 87.63) (xy 85.09 87.63)
+			(xy 74.93 87.63) (xy 78.74 87.63)
 		)
 		(stroke
