File: hardware/schematic/v1.0/GPSDO_Rev1.0/GPSDO_Rev1.0.kicad_pcb (KiCad board)
At the start: 2 copper layers, 75 x 84.1 mm, 130 parts, among them CN1 LAIL-PHC2_54-2P-01-XH-L, J1 Conn_Coaxial, J2 Conn_Coaxial, J3 Conn_01x04_Socket, U1 TDC7200PWR, U10 SN74LVC1T45DBVR, U11 CH340E, U12 BUF602IDBVT, U14 TPS7A5201RPSR, U15 STM32G431CBU6, U16 TPS7A5201RPSR, U2 LMK1C1103PWR, U3 TMP117AIDRVR, U4 BUF602IDBVT, U5 OCXO_20x20mm, U6 NEO-M8T-0, U7 OCXO_25.4x25.4mm, U8 REF5040, U9 OPA388IDR

Commit message: pcb update
Parts:
- removed C26: 10uF, GPSDO_Rev1.0:C_0603_1608Metric
- removed C46: 100nF, GPSDO_Rev1.0:C_0402_1005Metric
- added C68: 1uF / 16V, GPSDO_Rev1.0:C_0603_1608Metric, F.Cu at (162.8, 119.9)
- added C69: 1uF / 16V, GPSDO_Rev1.0:C_0603_1608Metric, F.Cu at (162.8, 122.4)
- added C70: 100nF / 16V, GPSDO_Rev1.0:C_0402_1005Metric, F.Cu at (155.3, 122.7)
- added C71: 22uF / 10V, GPSDO_Rev1.0:C_0805_2012Metric, F.Cu at (151.7, 118.2)
- added R43: 30.1K 1%, GPSDO_Rev1.0:R_0402_1005Metric, F.Cu at (169.9, 105.7)
- added R44: 10K 1%, GPSDO_Rev1.0:R_0402_1005Metric, F.Cu at (169.9, 107.7)
- added R45: 1K, GPSDO_Rev1.0:R_0402_1005Metric, F.Cu at (90.1, 60.6)
- added U18: TPS2116DRLR, GPSDO_Rev1.0:SOT-583-8, F.Cu at (167.2, 113.8)
- moved C39 106.5 mm to (75.5, 67.7)
- moved C40 106.5 mm to (75.5, 69.7)
- moved D1 106.5 mm to (79.0, 68.4)
- moved D8 106.5 mm to (79.0, 73.6)
- moved C35 106.5 mm to (75.5, 63.8)
- moved U14 106.5 mm to (79.4, 65.0)
- moved U16 106.5 mm to (83.7, 65.0)
- moved C36 106.5 mm to (75.5, 65.7)
- moved R31 105.0 mm to (87.2, 56.6)
- moved R33 105.0 mm to (87.2, 60.6)
- moved R32 105.0 mm to (87.2, 58.6)
- moved C34 104.2 mm to (71.9, 57.1)
- moved C37 104.2 mm to (71.9, 60.2)
- moved C38 104.2 mm to (71.9, 63.2)
- moved C41 104.2 mm to (71.9, 66.2)
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Connections:
- D8 pad 2: +5V -> Net-(D8-A)
- F1 pad 2: +5V -> /POWER/EXT_5V
Other:
- board size 75 x 84.1 mm -> 75 x 75 mm

Commit message: sch update
Parts:
- removed C30, C44: 100nF, GPSDO_Rev1.0:C_0402_1005Metric
- removed C31, C45: 4.7uF, GPSDO_Rev1.0:C_0603_1608Metric
- removed D7: TPD1E10B06DPYR, GPSDO_Rev1.0:TPD1E10B06DPYR
- removed J2: Conn_Coaxial, GPSDO_Rev1.0:SMA_Amphenol_132289_EdgeMount
- removed U12: BUF602IDBVT, GPSDO_Rev1.0:BUF602IDBVT
- added C26: 100nF, GPSDO_Rev1.0:C_0402_1005Metric, F.Cu at (142.0, 81.3)
- added C27: 100nF, GPSDO_Rev1.0:C_0402_1005Metric, F.Cu at (167.5, 76.1)
- added C28: 1uF, GPSDO_Rev1.0:C_0603_1608Metric, F.Cu at (161.2, 73.5)
- added C46: 100nF, GPSDO_Rev1.0:C_0402_1005Metric, F.Cu at (153.7, 129.6)
- added C47: 4.7uF, GPSDO_Rev1.0:C_0603_1608Metric, F.Cu at (154.3, 120.6)
- added C48: 100nF, GPSDO_Rev1.0:C_0402_1005Metric, F.Cu at (153.7, 131.6)
- added C49: 4.7uF, GPSDO_Rev1.0:C_0603_1608Metric, F.Cu at (154.3, 123.1)
- added C72: 10uF / 10V, GPSDO_Rev1.0:C_0603_1608Metric, F.Cu at (123.3, 123.9)
- added C73: 100nF, GPSDO_Rev1.0:C_0402_1005Metric, F.Cu at (109.6, 132.7)
- added C74: 22uF / 10V, GPSDO_Rev1.0:C_0805_2012Metric, F.Cu at (119.1, 124.5)
- added C75: 22uF / 10V, GPSDO_Rev1.0:C_0805_2012Metric, F.Cu at (119.1, 127.5)
- added D9: TPD1E10B06DPYR, GPSDO_Rev1.0:TPD1E10B06DPYR, F.Cu at (153.6, 127.6)
- added J4: Conn_Coaxial, GPSDO_Rev1.0:SMA_Amphenol_132289_EdgeMount, F.Cu at (137.3, 126.3)
- added L2: 1uH / DFE201610P, GPSDO_Rev1.0:L_Murata_DFE201610P, F.Cu at (118.7, 130.6)
- added R38: 0, GPSDO_Rev1.0:R_0402_1005Metric, F.Cu at (164.6, 80.1)
- added R39: 100K, GPSDO_Rev1.0:R_0402_1005Metric, F.Cu at (139.2, 71.4)
- added R40: 100K, GPSDO_Rev1.0:R_0402_1005Metric, F.Cu at (139.2, 73.4)
- added R41: 1K, GPSDO_Rev1.0:R_0402_1005Metric, F.Cu at (139.2, 75.3)
- added R42: 10K, GPSDO_Rev1.0:R_0402_1005Metric, F.Cu at (156.3, 125.3)
- added R46: 10K, GPSDO_Rev1.0:R_0402_1005Metric, F.Cu at (156.3, 127.3)
- added R47: 49.9, GPSDO_Rev1.0:R_0805_2012Metric, F.Cu at (154.5, 112.4)
- added R48: 10K, GPSDO_Rev1.0:R_0402_1005Metric, F.Cu at (164.6, 82.1)
- added R49: 1K, GPSDO_Rev1.0:R_0402_1005Metric, F.Cu at (112.5, 116.9)
- added R50: 10K, GPSDO_Rev1.0:R_0402_1005Metric, F.Cu at (112.5, 118.9)
- added R51: 77.4K 0.1%, GPSDO_Rev1.0:R_0402_1005Metric, F.Cu at (115.4, 108.9)
- added R52: 10K 0.1%, GPSDO_Rev1.0:R_0402_1005Metric, F.Cu at (115.4, 110.9)
- added R53: 2.2K, GPSDO_Rev1.0:R_0402_1005Metric, F.Cu at (115.4, 112.9)
- added U13: ISL55110IRZ-T, GPSDO_Rev1.0:ISL55110IRZ-T, F.Cu at (155.4, 116.6)
- R20: footprint GPSDO_Rev1.0:C_0603_1608Metric -> GPSDO_Rev1.0:R_0805_2012Metric
- R34: value 49.9 -> 2.2K; footprint GPSDO_Rev1.0:C_0603_1608Metric -> GPSDO_Rev1.0:R_0402_1005Metric
- R6: footprint GPSDO_Rev1.0:C_0603_1608Metric -> GPSDO_Rev1.0:R_0603_1608Metric
- U4: value BUF602IDBVT -> TPS61023DRLR; footprint GPSDO_Rev1.0:BUF602IDBVT -> GPSDO_Rev1.0:TPS61023DRLR
- moved U11 93.2 mm to (176.4, 61.6)
- moved U15 78.2 mm to (173.3, 71.6)
- moved U16 76.5 mm to (128.1, 127.3)
- moved U14 76.5 mm to (123.8, 127.3)
- moved USB1 73.0 mm to (164.6, 61.6)
- moved JP1 71.7 mm to (175.7, 86.8)
- moved C38 70.5 mm to (119.1, 115.5)
- moved C34 70.5 mm to (119.1, 109.4)
- moved C37 70.5 mm to (119.1, 112.5)
- moved C41 70.5 mm to (119.1, 118.5)
- moved C35 66.5 mm to (109.6, 120.9)
- moved C36 66.5 mm to (109.6, 122.8)
- moved C39 66.5 mm to (109.6, 124.8)
- moved C40 66.5 mm to (109.6, 126.8)
- moved J3 65.9 mm to (171.2, 78.7)
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Connections:
- net /POWER/PDN renamed Net-(U14-PG)
- C23 pad 1: /POWER/OCXO_VCC -> OCXO_VCC
- D1 pad 2: +3.3V -> Net-(D1-A)
- D2 pad 2: /POWER/OCXO_VCC -> Net-(D2-A)
- R12 pad 2: /OCXO/TMP_SDA -> /MCU/TMP_SDA
- R16 pad 2: /OCXO/TMP_SCL -> /MCU/TMP_SCL
- R20 pad 1: Net-(U4-Out) -> Net-(U13-OA)
- R22 pad 1: /POWER/OCXO_VCC -> OCXO_VCC
- R23 pad 2: /POWER/OCXO_VCC -> OCXO_VCC
- R34 pad 1: Net-(U12-Out) -> Net-(D2-A)
- R34 pad 2: Net-(J2-In) -> OCXO_VCC
- R35 pad 1: /OCXO/PWM -> /MCU/PWM
- R6 pad 2: /OCXO/10MHZ_MCU -> /MCU/10MHZ_MCU
- R7 pad 2: /OCXO/10MHZ_TDC -> /MCU/10MHZ_TDC
- U1 pad 3: /MCU/PULSE_GNSS -> /GNSS/PULSE_GNSS
- U10 pad 3: /OCXO/PWM -> /MCU/PWM
- U15 pad 10: /MCU/USART2_TX -> /GNSS/GNSS_UART_RXD
- U15 pad 11: /MCU/USART2_RX -> /GNSS/GNSS_UART_TXD
- U15 pad 16: /MCU/LED_RED -> unconnected-(U15-PC4-Pad16)
- U15 pad 17: unconnected-(U15-PB0-Pad17) -> /MCU/BOOST_EN
- U15 pad 20: unconnected-(U15-VREF+-Pad20) -> /MCU/VBAT
- U15 pad 22: unconnected-(U15-PB10-Pad22) -> Net-(U15-PB10)
- U15 pad 24: unconnected-(U15-PB11-Pad24) -> /GNSS/PULSE_GNSS
- U15 pad 29: /MCU/PULSE_GNSS -> unconnected-(U15-PC6-Pad29)
- U15 pad 30: unconnected-(U15-PA8-Pad30) -> /MCU/TDC_ENABLE
- U15 pad 34: unconnected-(U15-PA12-Pad34) -> /MCU/PWM
- U15 pad 41: unconnected-(U15-PB3-Pad41) -> /MCU/LED_RED
- U15 pad 46: GND -> Net-(U15-PB8-BOOT0)
- U15 pad 8: /MCU/PWM -> unconnected-(U15-PA0-Pad8)
- U15 pad 9: unconnected-(U15-PA1-Pad9) -> /MCU/VCTL
- U2 pad 3: /OCXO/10MHZ_OUT -> /EXT/10MHZ_OUT
- U3 pad 1: /OCXO/TMP_SCL -> /MCU/TMP_SCL
- U3 pad 2: unconnected-(U3-GND-Pad2) -> GND
- U3 pad 6: /OCXO/TMP_SDA -> /MCU/TMP_SDA
- U4 pad 1: Net-(U4-Out) -> /POWER/BOOST_FB
- U4 pad 2: unconnected-(U4-−VCC-Pad2) -> Net-(U4-EN)
- U4 pad 3: unconnected-(U4-VREF-Pad3) -> +3.3V
- U4 pad 4: /EXT/10MHZ_OUT -> GND
- U4 pad 5: +5V -> Net-(U4-SW)
Other:
- board size 75 x 75 mm -> 77.7 x 81.9 mm

Commit message: sch and pcb update
Parts:
- moved U11 71.5 mm to (118.4, 103.4), turned to 90 degrees
- moved H3 69.4 mm to (111.4, 133.4)
- moved USB1 68.0 mm to (110.9, 103.4), turned to -90 degrees
- moved R14 60.4 mm to (114.7, 106.2), turned to 90 degrees
- moved C27 58.6 mm to (117.2, 106.1)
- moved D5 58.0 mm to (176.9, 122.4)
- moved R11 57.4 mm to (115.1, 99.2), turned to 180 degrees
- moved D4 56.6 mm to (176.9, 118.4)
- moved C28 55.8 mm to (117.1, 107.7)
- moved D3 55.2 mm to (176.9, 114.4)
- moved RF1 53.1 mm to (174.8, 76.1), turned to 90 degrees
- moved C23 52.9 mm to (110.7, 80.4), turned to 90 degrees
- moved H4 52.8 mm to (176.4, 133.4)
- moved R35 48.6 mm to (152.6, 114.1)
- moved FB6 48.4 mm to (117.0, 100.7)
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Other:
- board size 77.7 x 81.9 mm -> 75 x 75 mm
- copper layers 2 -> 4
